File: pcb_top/rev.A/charon386_top.kicad_pcb (KiCad board)
At the start: 2 copper layers, 100 x 100 mm, 59 parts, among them J1 PC104_16, J2 AudioJack3, J3 PC104, J4 Jumper for 8-bit bus, J5 DB15_Female_HighDensity_Mount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, SW1 VGA Config, U1 TVGA9000I, U7 27C040, U8 ES1868F, Y1 12 MHz

Commit message: wip pcb rev.A
Parts:
- removed U7: 27C040, Package_LCC:PLCC-32_THT-Socket
- added U2: 27C512PLCC, my:PLCC-32_11.4x14.0mm_P1.27mm-longpads, F.Cu at (152.1, 136.1)

Commit message: wip pcb rev.A
Parts:
- Y1: footprint Crystal:Crystal_HC49-U_Vertical -> Crystal:Crystal_SMD_SeikoEpson_TSX3225-4Pin_3.2x2.5mm_HandSoldering
- moved R9 126.0 mm to (177.5, 63.1), turned to -90 degrees
- moved SW1 123.5 mm to (166.6, 63.8)
- moved R12 122.8 mm to (176.0, 80.2), turned to 180 degrees
- moved R14 118.1 mm to (176.0, 78.4), turned to 180 degrees
- moved R10 116.3 mm to (177.5, 67.0), turned to 90 degrees
- moved R2 114.1 mm to (154.4, 44.2), turned to 180 degrees
- moved R11 113.5 mm to (153.4, 70.2), turned to -90 degrees
- moved C19 107.1 mm to (176.0, 98.9), turned to 180 degrees
- moved R13 102.7 mm to (150.1, 70.2), turned to -90 degrees
- moved C17 101.9 mm to (135.0, 78.2)
- moved C18 98.5 mm to (135.0, 79.8)
- moved R15 94.2 mm to (138.5, 78.2), turned to 180 degrees
- moved R17 92.0 mm to (179.6, 98.9), turned to 180 degrees
- moved R16 87.0 mm to (138.5, 79.8), turned to 180 degrees
- moved JP1 85.3 mm to (176.0, 86.4), turned to -90 degrees
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Connections:
- U1 pad 133: (no net) -> Net-(U1-Pad133)
- U2 pad 1: unconnected-(U2-Pad1) -> (no net)
- U2 pad 12: unconnected-(U2-Pad12) -> (no net)
- U2 pad 17: unconnected-(U2-Pad17) -> (no net)
- U2 pad 26: unconnected-(U2-Pad26) -> (no net)
- Y1 pad 2: (no net) -> GND

Commit message: wip pcb rev.A
Parts:
- added C21: 10u, Capacitor_SMD:C_0603_1608Metric_Pad1.08x0.95mm_HandSolder, F.Cu at (60.2, 133.6)
- added C22: 100n, Capacitor_SMD:C_0603_1608Metric_Pad1.08x0.95mm_HandSolder, F.Cu at (64.5, 133.6)
- added C23: 10u, Capacitor_SMD:C_0603_1608Metric_Pad1.08x0.95mm_HandSolder, F.Cu at (55.9, 133.6)
- added C24: 100n, Capacitor_SMD:C_0603_1608Metric_Pad1.08x0.95mm_HandSolder, F.Cu at (55.9, 136.1)
- added C25: 10u, Capacitor_SMD:C_0603_1608Metric_Pad1.08x0.95mm_HandSolder, F.Cu at (67.0, 59.6)
- added C26: 100n, Capacitor_SMD:C_0603_1608Metric_Pad1.08x0.95mm_HandSolder, F.Cu at (73.7, 57.4)
- added C27: 220n, Capacitor_SMD:C_0603_1608Metric_Pad1.08x0.95mm_HandSolder, F.Cu at (58.4, 59.6)
- added C28: 220n, Capacitor_SMD:C_0603_1608Metric_Pad1.08x0.95mm_HandSolder, F.Cu at (78.0, 54.9)
- added C29: 220n, Capacitor_SMD:C_0603_1608Metric_Pad1.08x0.95mm_HandSolder, F.Cu at (75.8, 59.9)
- added C30: 220n, Capacitor_SMD:C_0603_1608Metric_Pad1.08x0.95mm_HandSolder, F.Cu at (73.7, 54.9)
- added C31: 220n, Capacitor_SMD:C_0603_1608Metric_Pad1.08x0.95mm_HandSolder, F.Cu at (66.4, 102.4)
- added C32: 220n, Capacitor_SMD:C_0603_1608Metric_Pad1.08x0.95mm_HandSolder, F.Cu at (71.0, 95.7)
- added C33: 220n, Capacitor_SMD:C_0603_1608Metric_Pad1.08x0.95mm_HandSolder, F.Cu at (77.0, 91.5)
- added C34: 220n, Capacitor_SMD:C_0603_1608Metric_Pad1.08x0.95mm_HandSolder, F.Cu at (66.4, 99.9)
- added C35: 100u/16V, Capacitor_Tantalum_SMD:CP_EIA-6032-28_Kemet-C_Pad2.25x2.35mm_HandSolder, F.Cu at (25.9, 92.6)
- added C36: 100n, Capacitor_SMD:C_0603_1608Metric_Pad1.08x0.95mm_HandSolder, F.Cu at (34.0, 100.4)
- added C37: 10n, Capacitor_SMD:C_0603_1608Metric_Pad1.08x0.95mm_HandSolder, F.Cu at (23.6, 105.8)
- added C38: 10u, Capacitor_SMD:C_0603_1608Metric_Pad1.08x0.95mm_HandSolder, F.Cu at (27.9, 105.8)
- added C39: 10u, Capacitor_Tantalum_SMD:CP_EIA-3216-18_Kemet-A_Pad1.58x1.35mm_HandSolder, F.Cu at (24.4, 103.0)
- added C40: 10u, Capacitor_Tantalum_SMD:CP_EIA-3216-18_Kemet-A_Pad1.58x1.35mm_HandSolder, F.Cu at (33.4, 91.8)
- added J6: Wavetable, Connector_PinHeader_2.54mm:PinHeader_2x13_P2.54mm_Vertical, F.Cu at (47.0, 52.4)
- added J7: PJ-322, my:PJ-322, F.Cu at (53.7, 99.0)
- added J8: PJ-322, my:PJ-322, F.Cu at (16.8, 99.0)
- added JP2: SolderJumper_2_Open, Jumper:SolderJumper-2_P1.3mm_Open_RoundedPad1.0x1.5mm, F.Cu at (62.7, 60.1)
- added JP3: SolderJumper_2_Open, Jumper:SolderJumper-2_P1.3mm_Open_RoundedPad1.0x1.5mm, F.Cu at (54.0, 60.4)
- added JP4: SolderJumper_2_Open, Jumper:SolderJumper-2_P1.3mm_Open_RoundedPad1.0x1.5mm, F.Cu at (71.4, 60.4)
- added JP5: SolderJumper_2_Open, Jumper:SolderJumper-2_P1.3mm_Open_RoundedPad1.0x1.5mm, F.Cu at (67.0, 62.6)
- added JP6: WTBL. P20, Jumper:SolderJumper-3_P1.3mm_Open_RoundedPad1.0x1.5mm_NumberLabels, F.Cu at (74.3, 51.8)
- added JP7: WTBL. P24, Jumper:SolderJumper-3_P1.3mm_Open_RoundedPad1.0x1.5mm_NumberLabels, F.Cu at (80.0, 51.8)
- added L2: 5.7u, Inductor_SMD:L_1210_3225Metric_Pad1.42x2.65mm_HandSolder, F.Cu at (44.8, 134.4)
- added L3: 5.7u, Inductor_SMD:L_1210_3225Metric_Pad1.42x2.65mm_HandSolder, F.Cu at (50.7, 134.4)
- added L4: BLM21PG331BH1D, Inductor_SMD:L_1210_3225Metric_Pad1.42x2.65mm_HandSolder, F.Cu at (65.9, 92.3)
- added L5: BLM21PG331BH1D, Inductor_SMD:L_1210_3225Metric_Pad1.42x2.65mm_HandSolder, F.Cu at (65.9, 96.5)
- added L6: BLM21PG331BH1D, Inductor_SMD:L_1210_3225Metric_Pad1.42x2.65mm_HandSolder, F.Cu at (71.8, 92.3)
- added L7: BLM21PG331BH1D, Inductor_SMD:L_1210_3225Metric_Pad1.42x2.65mm_HandSolder, F.Cu at (61.2, 102.0)
- added L8: 5.7u, Inductor_SMD:L_1210_3225Metric_Pad1.42x2.65mm_HandSolder, F.Cu at (32.8, 97.1)
- added R18: 100, Resistor_SMD:R_0603_1608Metric_Pad0.98x0.95mm_HandSolder, F.Cu at (148.2, 69.0)
- added R19: 10k, Resistor_SMD:R_0603_1608Metric_Pad0.98x0.95mm_HandSolder, F.Cu at (78.0, 57.4)
- added R20: 22k, Resistor_SMD:R_0603_1608Metric_Pad0.98x0.95mm_HandSolder, F.Cu at (82.2, 57.6)
- added R21: 15k, Resistor_SMD:R_0603_1608Metric_Pad0.98x0.95mm_HandSolder, F.Cu at (69.2, 104.9)
- added R22: 33k, Resistor_SMD:R_0603_1608Metric_Pad0.98x0.95mm_HandSolder, F.Cu at (64.8, 105.4)
- added R23: 15k, Resistor_SMD:R_0603_1608Metric_Pad0.98x0.95mm_HandSolder, F.Cu at (75.4, 95.7)
- added R24: 33k, Resistor_SMD:R_0603_1608Metric_Pad0.98x0.95mm_HandSolder, F.Cu at (60.5, 105.4)
- added R25: 10k, Resistor_SMD:R_0603_1608Metric_Pad0.98x0.95mm_HandSolder, F.Cu at (71.0, 98.2)
- added R26: 10k, Resistor_SMD:R_0603_1608Metric_Pad0.98x0.95mm_HandSolder, F.Cu at (70.8, 100.7)
- added R27: 1k, Resistor_SMD:R_0603_1608Metric_Pad0.98x0.95mm_HandSolder, F.Cu at (38.0, 94.6)
- added R28: 1k, Resistor_SMD:R_0603_1608Metric_Pad0.98x0.95mm_HandSolder, F.Cu at (29.6, 102.7)
- added R29: 10k, Resistor_SMD:R_0603_1608Metric_Pad0.98x0.95mm_HandSolder, F.Cu at (38.5, 91.5)
- added R30: 10k, Resistor_SMD:R_0603_1608Metric_Pad0.98x0.95mm_HandSolder, F.Cu at (38.0, 97.1)
- added U10: NE5532DR, Package_SO:SOIC-8_3.9x4.9mm_P1.27mm, F.Cu at (25.6, 98.2)
- added U11: 74HCT138, Package_SO:TSSOP-16_4.4x5mm_P0.65mm, F.Cu at (82.2, 36.2)
- added U3: MT4C4256, Package_DIP:DIP-20_W7.62mm, F.Cu at (123.1, 145.6)
- added U4: MT4C4256, Package_DIP:DIP-20_W7.62mm, F.Cu at (123.1, 134.8)
- added U5: MT4C4256, Package_DIP:DIP-20_W7.62mm, F.Cu at (152.2, 145.7)
- added U6: MT4C4256, Package_DIP:DIP-20_W7.62mm, F.Cu at (152.2, 134.8)
- added U7: AMS1117-5.0, Package_TO_SOT_SMD:SOT-223-3_TabPin2, F.Cu at (66.6, 54.2)
- added U9: AMS1117-5.0, Package_TO_SOT_SMD:SOT-223-3_TabPin2, F.Cu at (56.8, 54.2)
- C11: value 47p -> 1u
- J2: value AudioJack3 -> AUX_A; footprint Connector_Audio:Jack_3.5mm_CUI_SJ1-3535NG_Horizontal -> Connector_PinHeader_2.54mm:PinHeader_1x03_P2.54mm_Vertical; moved to F.Cu
- R10, R11, R12, R13, R14, R9: value 1k -> 4.7k
- U1: footprint Package_QFP:PQFP-160_28x28mm_P0.65mm -> my:PQFP-160_28x28mm_P0.65mm_LongPads
- Y1: value 12 MHz -> 40 MHz
- moved SW1 82.4 mm to (180.7, 145.0), turned to 90 degrees
- moved J2 81.2 mm to (60.6, 92.5), turned to 0 degrees
- moved R9 71.0 mm to (180.0, 134.1), turned to 0 degrees
- moved R10 67.4 mm to (183.9, 134.1), turned to 180 degrees
- moved R17 55.9 mm to (126.4, 81.7), turned to 0 degrees
- moved C14 50.1 mm to (142.2, 66.4), turned to 90 degrees
- moved C19 49.1 mm to (130.0, 81.7), turned to 0 degrees
- moved C17 48.3 mm to (177.6, 101.0), turned to 180 degrees
- moved C16 48.0 mm to (169.6, 66.9), turned to -90 degrees
- moved R1 47.9 mm to (130.0, 83.7), turned to 0 degrees
- moved L1 46.4 mm to (167.8, 66.9), turned to 90 degrees
- moved C18 45.6 mm to (177.6, 96.2), turned to 180 degrees
- moved R15 44.4 mm to (177.6, 99.4), turned to 0 degrees
- moved R7 43.9 mm to (142.2, 70.0), turned to 90 degrees
- moved Y1 43.7 mm to (163.8, 66.9), turned to 180 degrees
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Connections:
- C14 pad 1: /~IOW -> Net-(U1-Pad154)
- C15 pad 1: /~MEMR -> Net-(C15-Pad1)
- C20 pad 2: +5VA -> /AVDD1
- J3 pad 13: (no net) -> -12V
- J3 pad 17: (no net) -> +12V
- J3 pad 29: (no net) -> /DACK3
- J3 pad 3: /RESET -> Net-(C19-Pad2)
- J3 pad 31: (no net) -> /DRQ3
- J3 pad 33: (no net) -> /DACK1
- J3 pad 35: (no net) -> /DRQ1
- J3 pad 41: (no net) -> /IRQ7
- J3 pad 45: (no net) -> /IRQ5
- J3 pad 47: (no net) -> /IRQ4
- J3 pad 49: (no net) -> /IRQ3
- J3 pad 51: (no net) -> /DACK2
- J3 pad 7: (no net) -> /IRQ9
- R17 pad 1: /RESET -> Net-(C19-Pad2)
- R17 pad 2: Net-(C19-Pad2) -> /RESET
- R2 pad 1: +5V -> (no net)
- R7 pad 1: Net-(R7-Pad1) -> Net-(U1-Pad154)
- U1 pad 124: +5VA -> /AVDD1
- U1 pad 13: +5VA -> /AVDD2
- U1 pad 154: Net-(R7-Pad1) -> Net-(U1-Pad154)
- U1 pad 155: /~MEMR -> Net-(C15-Pad1)
- U1 pad 5: Net-(C19-Pad2) -> /RESET
- U1 pad 52: (no net) -> /MAA0
- U1 pad 53: (no net) -> /MAA1
- U1 pad 54: (no net) -> /MAA2
- U1 pad 55: (no net) -> /MAA3
- U1 pad 56: (no net) -> /MAA4
- U1 pad 57: (no net) -> /MAA5
- U1 pad 59: (no net) -> /MAA6
- U1 pad 6: +5VA -> /AVDD2
- U1 pad 60: (no net) -> /MAA7
- U1 pad 61: (no net) -> /MAA8
- U1 pad 64: (no net) -> /MD0
- U1 pad 65: (no net) -> /MD1
- U1 pad 68: (no net) -> /MD4
- U1 pad 70: (no net) -> /MD5
- U1 pad 71: (no net) -> /MD6
- U1 pad 73: (no net) -> /MAB0
- U1 pad 74: (no net) -> /MAB1
- U1 pad 75: (no net) -> /MAB2
- U1 pad 76: (no net) -> /MAB3
- U1 pad 77: (no net) -> /MAB4
- U1 pad 78: (no net) -> /MAB5
- U1 pad 82: (no net) -> /MAB6
- U1 pad 83: (no net) -> /MAB7
- U1 pad 84: (no net) -> /MAB8
- U1 pad 87: (no net) -> /~WE2
- U1 pad 88: (no net) -> /~WE0
- U1 pad 89: (no net) -> /MD16
- U1 pad 90: (no net) -> /MD17
- U1 pad 91: (no net) -> /MD18
- U1 pad 92: (no net) -> /MD19
- U1 pad 93: (no net) -> /MD20
- U1 pad 94: (no net) -> /MD21
- U1 pad 95: (no net) -> /MD22
- U1 pad 96: (no net) -> /MD23
- U8 pad 1: (no net) -> /A2
- U8 pad 10: (no net) -> /A9
- U8 pad 100: (no net) -> /A1
- U8 pad 11: (no net) -> Net-(U8-Pad11)
- U8 pad 12: (no net) -> /D0
- U8 pad 13: (no net) -> /D1
- U8 pad 14: (no net) -> /D2
- U8 pad 15: (no net) -> /D3
- U8 pad 16: (no net) -> /D4
- U8 pad 17: (no net) -> /D5
- U8 pad 18: (no net) -> /D6
- U8 pad 19: (no net) -> /D7
- U8 pad 2: (no net) -> /A3
- U8 pad 35: (no net) -> Net-(U8-Pad35)
- U8 pad 36: (no net) -> Net-(U8-Pad36)
- U8 pad 37: (no net) -> Net-(U8-Pad37)
- U8 pad 38: (no net) -> Net-(U8-Pad38)
- U8 pad 4: (no net) -> /A4
- U8 pad 43: (no net) -> /AVDD_ES
- U8 pad 48: (no net) -> Net-(U8-Pad48)
- U8 pad 49: (no net) -> Net-(U8-Pad49)
- U8 pad 5: (no net) -> /A5
- U8 pad 50: (no net) -> Net-(U8-Pad50)
- U8 pad 51: (no net) -> Net-(U8-Pad51)
- U8 pad 58: (no net) -> /MSO
- U8 pad 6: (no net) -> /A6
- U8 pad 63: (no net) -> /DRQ3
- U8 pad 64: (no net) -> /DACK3
- U8 pad 65: (no net) -> /DRQ1
- U8 pad 66: (no net) -> /DACK1
- U8 pad 67: (no net) -> Net-(U8-Pad67)
- U8 pad 68: (no net) -> Net-(U8-Pad68)
- U8 pad 70: (no net) -> Net-(U8-Pad70)
- U8 pad 71: (no net) -> Net-(U8-Pad71)
- U8 pad 72: (no net) -> /IRQ7
- U8 pad 73: (no net) -> /IRQ5
- U8 pad 74: (no net) -> /IRQ9
- U8 pad 75: (no net) -> /~IOR
- U8 pad 76: (no net) -> /~IOW
- U8 pad 78: (no net) -> /OSC
- U8 pad 8: (no net) -> /A7
- U8 pad 81: (no net) -> /RESET
- U8 pad 87: (no net) -> /MSD
- U8 pad 88: (no net) -> /MCLK
- U8 pad 9: (no net) -> /A8
- U8 pad 90: (no net) -> /~RSTB
- U8 pad 92: (no net) -> Net-(U8-Pad92)
- U8 pad 97: (no net) -> /A10
- U8 pad 98: (no net) -> /A11
- U8 pad 99: (no net) -> /A0

Commit message: wip pcb rev.A
Parts:
- removed H1, H2, H3, H4: MountingHole, my:MountingHole_3.2mm_M3_dk5.2mm_Mask
- removed J5: DB15_Female_HighDensity_MountingHoles, Connector_Dsub:DSUB-15-HD_Female_Horizontal_P2.29x1.98mm_EdgePinOffset3.03mm_Housed_MountingHolesOffset4.94mm
- removed J8: PJ-322, my:PJ-322
- removed JP2, JP3, JP4, JP5: SolderJumper_2_Open, Jumper:SolderJumper-2_P1.3mm_Open_RoundedPad1.0x1.5mm
- removed L4: BLM21PG331BH1D, Inductor_SMD:L_1210_3225Metric_Pad1.42x2.65mm_HandSolder
- added C41: 10p, Capacitor_SMD:C_0603_1608Metric_Pad1.08x0.95mm_HandSolder, F.Cu at (103.8, 109.6)
- added C42: 10p, Capacitor_SMD:C_0603_1608Metric_Pad1.08x0.95mm_HandSolder, F.Cu at (103.8, 106.8)
- added C43: 47n, Capacitor_SMD:C_0603_1608Metric_Pad1.08x0.95mm_HandSolder, F.Cu at (130.9, 85.0)
- added C44: 100n, Capacitor_SMD:C_0603_1608Metric_Pad1.08x0.95mm_HandSolder, B.Cu at (172.4, 76.1)
- added C45: 100n, Capacitor_SMD:C_0603_1608Metric_Pad1.08x0.95mm_HandSolder, B.Cu at (165.6, 76.4)
- added C46: 100n, Capacitor_SMD:C_0603_1608Metric_Pad1.08x0.95mm_HandSolder, B.Cu at (162.7, 101.2)
- added C47: 100n, Capacitor_SMD:C_0603_1608Metric_Pad1.08x0.95mm_HandSolder, B.Cu at (134.9, 107.0)
- added C48: 1u, Capacitor_SMD:C_0603_1608Metric_Pad1.08x0.95mm_HandSolder, F.Cu at (175.4, 104.6)
- added C49: 100n, Capacitor_SMD:C_0603_1608Metric_Pad1.08x0.95mm_HandSolder, B.Cu at (147.6, 87.8)
- added C50: 100n, Capacitor_SMD:C_0603_1608Metric_Pad1.08x0.95mm_HandSolder, B.Cu at (115.7, 93.9)
- added C51: 100n, Capacitor_SMD:C_0603_1608Metric_Pad1.08x0.95mm_HandSolder, B.Cu at (147.8, 80.7)
- added C52: 100n, Capacitor_SMD:C_0603_1608Metric_Pad1.08x0.95mm_HandSolder, B.Cu at (126.5, 92.6)
- added C53: 100n, Capacitor_SMD:C_0603_1608Metric_Pad1.08x0.95mm_HandSolder, B.Cu at (126.4, 107.5)
- added C54: 100n, Capacitor_SMD:C_0603_1608Metric_Pad1.08x0.95mm_HandSolder, B.Cu at (115.8, 108.8)
- added C55: 100n, Capacitor_SMD:C_0603_1608Metric_Pad1.08x0.95mm_HandSolder, B.Cu at (174.7, 117.9)
- added C56: 100n, Capacitor_SMD:C_0603_1608Metric_Pad1.08x0.95mm_HandSolder, B.Cu at (146.0, 131.0)
- added C57: 100n, Capacitor_SMD:C_0603_1608Metric_Pad1.08x0.95mm_HandSolder, B.Cu at (146.0, 141.8)
- added C58: 100n, Capacitor_SMD:C_0603_1608Metric_Pad1.08x0.95mm_HandSolder, B.Cu at (175.0, 141.8)
- added C59: 100n, Capacitor_SMD:C_0603_1608Metric_Pad1.08x0.95mm_HandSolder, B.Cu at (175.0, 130.8)
- added C60: 1u, Capacitor_SMD:C_0603_1608Metric_Pad1.08x0.95mm_HandSolder, B.Cu at (108.8, 77.3)
- added C61: 1u, Capacitor_SMD:C_0603_1608Metric_Pad1.08x0.95mm_HandSolder, B.Cu at (183.6, 62.5)
- added J9: Conn_02x07_Odd_Even, Connector_PinHeader_2.54mm:PinHeader_2x08_P2.54mm_Vertical, B.Cu at (140.6, 58.6)
- added JP8: SolderJumper_3_Bridged12, Jumper:SolderJumper-3_P1.3mm_Bridged12_RoundedPad1.0x1.5mm_NumberLabels, B.Cu at (111.5, 107.2)
- added JP9: SolderJumper_2_Open, Jumper:SolderJumper-2_P1.3mm_Open_RoundedPad1.0x1.5mm, B.Cu at (110.9, 109.7)
- added L10: BLM21PG331BH1D, Inductor_SMD:L_0805_2012Metric_Pad1.15x1.40mm_HandSolder, F.Cu at (135.8, 58.6)
- added L9: BLM21PG331BH1D, Inductor_SMD:L_0805_2012Metric_Pad1.15x1.40mm_HandSolder, F.Cu at (135.8, 61.1)
- added R31: 10k, Resistor_SMD:R_0603_1608Metric_Pad0.98x0.95mm_HandSolder, B.Cu at (131.9, 97.7)
- added R32: 2.2k, Resistor_SMD:R_0603_1608Metric_Pad0.98x0.95mm_HandSolder, F.Cu at (130.9, 83.5)
- added R33: 1k, Resistor_SMD:R_0603_1608Metric_Pad0.98x0.95mm_HandSolder, B.Cu at (131.9, 93.2)
- added R34: 1k, Resistor_SMD:R_0603_1608Metric_Pad0.98x0.95mm_HandSolder, B.Cu at (131.9, 94.7)
- added R35: 1k, Resistor_SMD:R_0603_1608Metric_Pad0.98x0.95mm_HandSolder, B.Cu at (131.9, 96.2)
- added Y2: 14.318 MHz, Crystal:Crystal_SMD_SeikoEpson_TSX3225-4Pin_3.2x2.5mm_HandSoldering, F.Cu at (107.9, 108.2)
- C14, C15, C17, C18, C2, C26, C29, C3, C30, C36, J7, JP1, R11, R12, R13, R14, R15, R16, R18, R7: moved to B.Cu
- C21, C23, C25, C38: footprint Capacitor_SMD:C_0603_1608Metric_Pad1.08x0.95mm_HandSolder -> Capacitor_SMD:C_0805_2012Metric_Pad1.18x1.45mm_HandSolder
- C28: value 220n -> 100n; moved to B.Cu
- C39, C40: value 10u -> 47u; footprint Capacitor_Tantalum_SMD:CP_EIA-3216-18_Kemet-A_Pad1.58x1.35mm_HandSolder -> Capacitor_Tantalum_SMD:CP_EIA-3528-21_Kemet-B_Pad1.50x2.35mm_HandSolder
- J1: footprint Connector_PinSocket_2.54mm:PinSocket_2x20_P2.54mm_Vertical -> Connector_PinHeader_2.54mm:PinHeader_2x20_P2.54mm_Vertical; moved to B.Cu
- J2: value AUX_A -> Vol. Btns; footprint Connector_PinHeader_2.54mm:PinHeader_1x03_P2.54mm_Vertical -> Connector_PinHeader_2.54mm:PinHeader_2x03_P2.54mm_Vertical
- J3: footprint Connector_PinSocket_2.54mm:PinSocket_2x32_P2.54mm_Vertical -> Connector_PinHeader_2.54mm:PinHeader_2x32_P2.54mm_Vertical; moved to B.Cu
- J6: footprint Connector_PinHeader_2.54mm:PinHeader_2x13_P2.54mm_Vertical -> Connector_PinHeader_2.54mm:PinHeader_2x13_P2.54mm_Horizontal
- JP6, JP7: footprint Jumper:SolderJumper-3_P1.3mm_Open_RoundedPad1.0x1.5mm_NumberLabels -> Jumper:SolderJumper-3_P1.3mm_Bridged12_RoundedPad1.0x1.5mm_NumberLabels; moved to B.Cu
- L5, L6, L7: footprint Inductor_SMD:L_1210_3225Metric_Pad1.42x2.65mm_HandSolder -> Inductor_SMD:L_0805_2012Metric_Pad1.15x1.40mm_HandSolder
- R2: value 0 -> 10k
- R27, R28: value 1k -> 10k
- moved L2 150.6 mm to (181.8, 72.0), turned to 90 degrees
- moved J2 139.9 mm to (193.8, 135.2)
- moved C21 133.6 mm to (178.8, 72.0), turned to 90 degrees
- moved C22 128.2 mm to (176.9, 72.0), turned to -90 degrees
- moved U7 113.3 mm to (179.4, 64.8), turned to 180 degrees
- moved J6 113.0 mm to (111.9, 144.8), turned to 180 degrees
- moved C39 107.8 mm to (124.8, 63.6), turned to 90 degrees
- moved C35 107.4 mm to (131.0, 70.6)
- moved C37 105.4 mm to (124.4, 75.2), turned to 90 degrees
- moved L3 105.0 mm to (138.8, 77.4), turned to -90 degrees
- moved C38 103.0 mm to (126.2, 75.2), turned to 90 degrees
- moved R28 102.9 mm to (129.0, 76.0), turned to 180 degrees
- moved L8 102.7 mm to (133.3, 75.9), turned to 90 degrees
- moved C40 100.6 mm to (129.9, 63.6), turned to 90 degrees
- moved C24 100.0 mm to (139.9, 82.0), turned to -90 degrees
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Connections:
- net /xB renamed /VGA_B
- net /xG renamed /VGA_G
- net /xR renamed /VGA_R
- C1 pad 2: GNDA -> GND
- C10 pad 2: GNDA -> GND
- C11 pad 1: /xMonitor -> /VGA_MON
- C11 pad 2: GNDA -> GND
- C12 pad 1: /xHSYNC -> /VGA_HS
- C12 pad 2: GNDA -> GND
- C13 pad 1: /xVSYNC -> /VGA_VS
- C13 pad 2: GNDA -> GND
- C2 pad 2: GNDA -> GND
- C21 pad 1: GNDA -> GND
- C22 pad 2: GNDA -> GND
- C23 pad 1: GNDA -> GND
- C24 pad 2: GNDA -> GND
- C25 pad 1: GNDA -> GND
- C26 pad 2: GNDA -> GND
- C27 pad 1: Net-(U8-Pad37) -> Net-(C27-Pad1)
- C28 pad 1: Net-(U8-Pad38) -> +5V
- C28 pad 2: Net-(C28-Pad2) -> GND
- C29 pad 2: /AUXBL -> /AUXB_L
- C3 pad 2: GNDA -> GND
- C30 pad 2: /AUXBR -> /AUXB_R
- C35 pad 2: GNDA -> GND
- C36 pad 2: GNDA -> GND
- C37 pad 1: GNDA -> GND
- C38 pad 1: GNDA -> GND
- C39 pad 2: /AOUT_R -> Net-(C39-Pad2)
- C40 pad 2: /AOUT_L -> Net-(C40-Pad2)
- C5 pad 2: GNDA -> GND
- C7 pad 2: GNDA -> GND
- C8 pad 2: GNDA -> GND
- C9 pad 2: GNDA -> GND
- FB3 pad 1: /xMonitor -> /Monitor
- FB3 pad 2: /Monitor -> /VGA_MON
- FB5 pad 1: /xHSYNC -> /HSYNC
- FB5 pad 2: /HSYNC -> /VGA_HS
- FB6 pad 1: /xVSYNC -> /VSYNC
- FB6 pad 2: /VSYNC -> /VGA_VS
- J1 pad 18: (no net) -> /DACK0
- J1 pad 20: (no net) -> /DRQ0
- J1 pad 22: (no net) -> /DACK5
- J1 pad 24: (no net) -> /DRQ5
- J1 pad 8: (no net) -> /IRQ10
- J2 pad 1: /AUXAL -> GND
- J2 pad 2: /AUXAR -> Net-(J2-Pad2)
- J2 pad 3: GNDA -> GND
- J3 pad 47: /IRQ4 -> (no net)
- J3 pad 49: /IRQ3 -> (no net)
- J3 pad 51: /DACK2 -> (no net)
- J6 pad 15: GNDA -> GND
- J6 pad 17: GNDA -> GND
- J6 pad 19: GNDA -> GND
- J6 pad 21: GNDA -> GND
- J6 pad 23: GNDA -> GND
- J6 pad 25: GNDA -> GND
- J7 pad R2: GNDA -> GND
- J7 pad S: GNDA -> GND
- JP6 pad 1: /AUXBR -> /AUXB_L
- JP6 pad 3: /AUXBL -> /AUXB_R
- JP7 pad 1: /AUXBR -> /AUXB_R
- JP7 pad 3: /AUXBL -> /AUXB_L
- L5 pad 1: Net-(C28-Pad2) -> Net-(L5-Pad1)
- L5 pad 2: /AUXAR -> /SPKR
- R2 pad 1: (no net) -> Net-(L5-Pad1)
- R2 pad 2: Net-(J5-Pad9) -> Net-(C27-Pad2)
- R22 pad 1: Net-(R29-Pad2) -> Net-(R22-Pad1)
- R25 pad 2: GNDA -> GND
- R26 pad 2: GNDA -> GND
- R28 pad 1: GNDA -> GND
- R29 pad 2: Net-(R29-Pad2) -> Net-(R22-Pad1)
- R3 pad 2: /xMonitor -> /VGA_MON
- R4 pad 2: GNDA -> GND
- R5 pad 2: GNDA -> GND
- R6 pad 2: GNDA -> GND
- R8 pad 2: GNDA -> GND
- U1 pad 1: GNDA -> GND
- U1 pad 126: GNDA -> GND
- U10 pad 1: Net-(C40-Pad1) -> Net-(C39-Pad1)
- U10 pad 2: Net-(R24-Pad1) -> Net-(R22-Pad1)
- U10 pad 6: Net-(R29-Pad2) -> Net-(R24-Pad1)
- U10 pad 7: Net-(C39-Pad1) -> Net-(C40-Pad1)
- U7 pad 1: GNDA -> GND
- U7 pad 3: +5V -> +12V
- U8 pad 20: (no net) -> Net-(R31-Pad1)
- U8 pad 21: (no net) -> Net-(U8-Pad21)
- U8 pad 22: (no net) -> Net-(U8-Pad22)
- U8 pad 23: (no net) -> Net-(U8-Pad23)
- U8 pad 25: (no net) -> GND
- U8 pad 37: Net-(U8-Pad37) -> Net-(C27-Pad1)
- U8 pad 38: Net-(U8-Pad38) -> Net-(C27-Pad1)
- U8 pad 41: GNDA -> GND
- U8 pad 61: (no net) -> /DRQ5
- U8 pad 62: (no net) -> /DACK5
- U8 pad 67: Net-(U8-Pad67) -> /DRQ0
- U8 pad 68: Net-(U8-Pad68) -> /DACK0
- U8 pad 70: Net-(U8-Pad70) -> (no net)
- U8 pad 71: Net-(U8-Pad71) -> /IRQ10
- U8 pad 78: /OSC -> Net-(JP8-Pad2)
- U8 pad 79: (no net) -> Net-(JP9-Pad2)
- U9 pad 1: GNDA -> GND
- U9 pad 3: +5V -> +12V
Other:
- outline, holes or cut-outs redrawn
- copper layers 2 -> 4

Commit message: wip pcb rev.A
Parts:
- removed JP9: SolderJumper_2_Open, Jumper:SolderJumper-2_P1.3mm_Open_RoundedPad1.0x1.5mm
- added J5: ESP, Connector_PinSocket_2.54mm:PinSocket_2x05_P2.54mm_Vertical, B.Cu at (101.2, 106.9)
- C27: value 220n -> 100n
- C43: value 47n -> 4.7n
- R2: value 10k -> 47k
- R20: moved to B.Cu
- R32: value 2.2k -> 4.7k
- moved C55 51.3 mm to (125.6, 132.6), turned to -90 degrees
- moved U2 50.7 mm to (124.3, 136.3), turned to 0 degrees
- moved U3 26.8 mm to (135.8, 122.0), turned to 0 degrees
- moved U4 26.7 mm to (146.6, 122.0), turned to 0 degrees
- moved U5 24.2 mm to (157.4, 122.0), turned to 0 degrees
- moved U6 20.5 mm to (168.2, 122.0), turned to 0 degrees
- moved C56 14.5 mm to (150.4, 144.9), turned to 0 degrees
- moved C59 14.4 mm to (172.0, 144.9), turned to 0 degrees
- moved C58 14.1 mm to (161.2, 144.9), turned to 0 degrees
- moved R20 8.40 mm to (106.8, 143.6), turned to 90 degrees
- moved C29 8.10 mm to (103.2, 122.6), turned to 0 degrees
- moved C10 7.25 mm to (153.2, 64.8)
- moved FB4 7.25 mm to (153.2, 68.6)
- moved R6 7.25 mm to (155.0, 68.8)
- moved R4 7.20 mm to (147.8, 68.8)
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Connections:
- C41 pad 2: Net-(Y2-Pad1) -> Net-(C41-Pad2)
- U8 pad 79: Net-(JP9-Pad2) -> Net-(C41-Pad2)
- Y2 pad 1: Net-(Y2-Pad1) -> Net-(C41-Pad2)
Routing:
- net GND: track 0.00 -> 340.1 mm, vias 0 -> 13
- net /A0: track 0.00 -> 144.7 mm, vias 0 -> 3
- net /A1: track 0.00 -> 141.1 mm, vias 0 -> 3
- net /A10: track 0.00 -> 139.0 mm, vias 0 -> 3
- net /A2: track 0.00 -> 137.2 mm, vias 0 -> 3
- net /A11: track 0.00 -> 135.1 mm, vias 0 -> 3
- net /A3: track 0.00 -> 134.5 mm, vias 0 -> 3
- net /A4: track 0.00 -> 131.9 mm, vias 0 -> 3
- net /A5: track 0.00 -> 130.5 mm, vias 0 -> 3
- net /A9: track 0.00 -> 128.9 mm, vias 0 -> 3
- net /A6: track 0.00 -> 127.8 mm, vias 0 -> 3
- net /A12: track 0.00 -> 127.7 mm, vias 0 -> 3
- net /A8: track 0.00 -> 127.4 mm, vias 0 -> 3
- net /ROMA0: track 0.00 -> 126.9 mm, vias 0 -> 2
- net /A7: track 0.00 -> 125.4 mm, vias 0 -> 3
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
Commit message: wip pcb rev.A
Parts:
- removed J4: Jumper for 8-bit bus, Connector_PinHeader_2.00mm:PinHeader_2x03_P2.00mm_Vertical
- removed J6: Wavetable, Connector_PinHeader_2.54mm:PinHeader_2x13_P2.54mm_Horizontal
- removed JP6: WTBL. P20, Jumper:SolderJumper-3_P1.3mm_Bridged12_RoundedPad1.0x1.5mm_NumberLabels
- removed JP7: WTBL. P24, Jumper:SolderJumper-3_P1.3mm_Bridged12_RoundedPad1.0x1.5mm_NumberLabels
- removed JP8: SolderJumper_3_Bridged12, Jumper:SolderJumper-3_P1.3mm_Bridged12_RoundedPad1.0x1.5mm_NumberLabels
- added C62: 100n, Capacitor_SMD:C_0603_1608Metric_Pad1.08x0.95mm_HandSolder, B.Cu at (104.8, 134.7)
- added C63: 10u, Capacitor_SMD:C_0805_2012Metric_Pad1.18x1.45mm_HandSolder, B.Cu at (104.7, 136.5)
- added C64: 22p, Capacitor_SMD:C_0603_1608Metric_Pad1.08x0.95mm_HandSolder, F.Cu at (111.2, 141.8)
- added C65: 22p, Capacitor_SMD:C_0603_1608Metric_Pad1.08x0.95mm_HandSolder, F.Cu at (103.5, 141.8)
- added C66: 1u, Capacitor_SMD:C_0603_1608Metric_Pad1.08x0.95mm_HandSolder, B.Cu at (106.2, 131.2)
- added C67: 100n, Capacitor_SMD:C_0603_1608Metric_Pad1.08x0.95mm_HandSolder, B.Cu at (107.7, 137.2)
- added C68: 100n, Capacitor_SMD:C_0603_1608Metric_Pad1.08x0.95mm_HandSolder, B.Cu at (110.6, 131.8)
- added C69: 10u, Capacitor_SMD:C_0805_2012Metric_Pad1.18x1.45mm_HandSolder, B.Cu at (101.2, 122.2)
- added C70: 10u, Capacitor_SMD:C_0805_2012Metric_Pad1.18x1.45mm_HandSolder, B.Cu at (103.5, 122.2)
- added C71: 100n, Capacitor_SMD:C_0603_1608Metric_Pad1.08x0.95mm_HandSolder, B.Cu at (111.5, 126.8)
- added LOGO1: graphic, mygraphic:black-mage-12.5x8.6, F.Cu at (159.4, 93.2)
- added R36: 22, Resistor_SMD:R_0603_1608Metric_Pad0.98x0.95mm_HandSolder, F.Cu at (179.2, 94.8)
- added U12: SAM2695, Package_DFN_QFN:QFN-48-1EP_6x6mm_P0.4mm_EP4.2x4.2mm, F.Cu at (107.7, 134.1)
- added U13: AMS1117-3.3, Package_TO_SOT_SMD:SOT-223-3_TabPin2, F.Cu at (103.5, 123.9)
- added U14: 74HC4050, Package_SO:SO-16_3.9x9.9mm_P1.27mm, F.Cu at (111.6, 123.3)
- C29, C30, C60, C61: moved to F.Cu
- C41: value 10p -> 100n; moved to B.Cu
- C42: value 10p -> 10u; footprint Capacitor_SMD:C_0603_1608Metric_Pad1.08x0.95mm_HandSolder -> Capacitor_SMD:C_0805_2012Metric_Pad1.18x1.45mm_HandSolder; moved to B.Cu
- C48: moved to B.Cu
- R20: value 22k -> 22; moved to F.Cu
- Y2: value 14.318 MHz -> 12 MHz
- moved R20 38.1 mm to (110.0, 105.6)
- moved Y2 33.6 mm to (107.3, 141.8), turned to 180 degrees
- moved C42 31.2 mm to (110.6, 135.7), turned to 0 degrees
- moved C41 22.2 mm to (110.6, 133.9)
- moved C29 15.4 mm to (118.6, 122.3), turned to -90 degrees
- moved C30 13.8 mm to (116.9, 122.3), turned to -90 degrees
- moved L6 8.40 mm to (123.2, 54.8)
- moved L7 8.20 mm to (131.3, 54.8), turned to -90 degrees
- moved R31 5.95 mm to (126.5, 100.2), turned to 180 degrees
- moved R35 5.91 mm to (126.5, 98.6)
- moved R34 5.86 mm to (126.5, 97.0)
- moved R33 5.83 mm to (126.5, 95.4)
- moved C31 4.75 mm to (125.0, 54.8)
- moved C32 4.45 mm to (129.4, 54.8)
- moved U7 3.10 mm to (176.3, 65.8)
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Connections:
- net /~CAS renamed /~{CAS}
- net /~IOR renamed /~{IOR}
- net /~IOW renamed /~{IOW}
- net /~MEMCS16 renamed /~{MEMCS16}
- net /~MEMR renamed /~{MEMR}
- net /~MEMW renamed /~{MEMW}
- net /~NMI renamed /~{NMI}
- net /~RAS renamed /~{RAS}
- net /~REFRESH renamed /~{REFRESH}
- net /~ROMCS renamed /~{ROMCS}
- net /~SBHE renamed /~{SBHE}
- net /~WE0 renamed /~{WE0}
- net /~WE2 renamed /~{WE2}
- C29 pad 2: /AUXB_L -> /MIDI_L
- C30 pad 2: /AUXB_R -> /MIDI_R
- C42 pad 2: Net-(C42-Pad2) -> Net-(C41-Pad2)
- J1 pad 10: (no net) -> /IRQ11
- J1 pad 12: (no net) -> unconnected-(J1-Pad12)
- J1 pad 14: (no net) -> unconnected-(J1-Pad14)
- J1 pad 16: (no net) -> unconnected-(J1-Pad16)
- J1 pad 19: (no net) -> unconnected-(J1-Pad19)
- J1 pad 21: (no net) -> unconnected-(J1-Pad21)
- J1 pad 26: (no net) -> unconnected-(J1-Pad26)
- J1 pad 28: (no net) -> unconnected-(J1-Pad28)
- J1 pad 30: (no net) -> unconnected-(J1-Pad30)
- J1 pad 32: (no net) -> unconnected-(J1-Pad32)
- J1 pad 36: (no net) -> unconnected-(J1-Pad36)
- J1 pad 39: (no net) -> unconnected-(J1-Pad39)
- J1 pad 6: (no net) -> unconnected-(J1-Pad6)
- J3 pad 11: (no net) -> unconnected-(J3-Pad11)
- J3 pad 15: (no net) -> unconnected-(J3-Pad15)
- J3 pad 19: (no net) -> unconnected-(J3-Pad19)
- J3 pad 39: (no net) -> unconnected-(J3-Pad39)
- J3 pad 43: (no net) -> unconnected-(J3-Pad43)
- J3 pad 47: (no net) -> unconnected-(J3-Pad47)
- J3 pad 49: (no net) -> unconnected-(J3-Pad49)
- J3 pad 51: (no net) -> unconnected-(J3-Pad51)
- J3 pad 53: (no net) -> unconnected-(J3-Pad53)
- J3 pad 9: (no net) -> unconnected-(J3-Pad9)
- J5 pad 1: (no net) -> unconnected-(J5-Pad1)
- J5 pad 2: (no net) -> unconnected-(J5-Pad2)
- J5 pad 5: Net-(J5-Pad5) -> unconnected-(J5-Pad5)
- J5 pad 6: Net-(J5-Pad5) -> unconnected-(J5-Pad6)
- J9 pad 15: (no net) -> unconnected-(J9-Pad15)
- J9 pad 6: (no net) -> unconnected-(J9-Pad6)
- R20 pad 1: /MCLK -> Net-(U8-Pad78)
- R20 pad 2: GND -> /OSC
- U1 pad 10: (no net) -> unconnected-(U1-Pad10)
- U1 pad 100: (no net) -> unconnected-(U1-Pad100)
- U1 pad 11: (no net) -> unconnected-(U1-Pad11)
- U1 pad 111: (no net) -> unconnected-(U1-Pad111)
- U1 pad 112: (no net) -> unconnected-(U1-Pad112)
- U1 pad 12: (no net) -> unconnected-(U1-Pad12)
- U1 pad 123: (no net) -> unconnected-(U1-Pad123)
- U1 pad 127: (no net) -> unconnected-(U1-Pad127)
- U1 pad 129: (no net) -> unconnected-(U1-Pad129)
- U1 pad 132: (no net) -> unconnected-(U1-Pad132)
- U1 pad 14: (no net) -> unconnected-(U1-Pad14)
- U1 pad 15: (no net) -> unconnected-(U1-Pad15)
- U1 pad 159: (no net) -> unconnected-(U1-Pad159)
- U1 pad 16: (no net) -> unconnected-(U1-Pad16)
- U1 pad 17: (no net) -> unconnected-(U1-Pad17)
- U1 pad 20: (no net) -> unconnected-(U1-Pad20)
- U1 pad 44: (no net) -> unconnected-(U1-Pad44)
- U1 pad 63: (no net) -> unconnected-(U1-Pad63)
- U1 pad 9: (no net) -> unconnected-(U1-Pad9)
- U1 pad 98: /OSC -> Net-(U1-Pad98)
- U11 pad 10: (no net) -> unconnected-(U11-Pad10)
- U11 pad 11: (no net) -> unconnected-(U11-Pad11)
- U11 pad 12: (no net) -> unconnected-(U11-Pad12)
- U11 pad 13: (no net) -> unconnected-(U11-Pad13)
- U11 pad 14: (no net) -> unconnected-(U11-Pad14)
- U11 pad 7: (no net) -> unconnected-(U11-Pad7)
- U11 pad 9: (no net) -> unconnected-(U11-Pad9)
- U2 pad 1: (no net) -> unconnected-(U2-Pad1)
- U2 pad 12: (no net) -> unconnected-(U2-Pad12)
- U2 pad 17: (no net) -> unconnected-(U2-Pad17)
- U2 pad 26: (no net) -> unconnected-(U2-Pad26)
- U3 pad 5: (no net) -> unconnected-(U3-Pad5)
- U4 pad 5: (no net) -> unconnected-(U4-Pad5)
- U5 pad 5: (no net) -> unconnected-(U5-Pad5)
- U6 pad 5: (no net) -> unconnected-(U6-Pad5)
- U8 pad 27: (no net) -> unconnected-(U8-Pad27)
- U8 pad 28: (no net) -> unconnected-(U8-Pad28)
- U8 pad 29: (no net) -> unconnected-(U8-Pad29)
- U8 pad 30: (no net) -> unconnected-(U8-Pad30)
- U8 pad 31: (no net) -> unconnected-(U8-Pad31)
- U8 pad 32: (no net) -> unconnected-(U8-Pad32)
- U8 pad 33: (no net) -> unconnected-(U8-Pad33)
- U8 pad 34: (no net) -> unconnected-(U8-Pad34)
- U8 pad 40: (no net) -> unconnected-(U8-Pad40)
- U8 pad 53: (no net) -> unconnected-(U8-Pad53)
- U8 pad 54: (no net) -> unconnected-(U8-Pad54)
- U8 pad 55: (no net) -> unconnected-(U8-Pad55)
- U8 pad 56: (no net) -> unconnected-(U8-Pad56)
- U8 pad 59: (no net) -> unconnected-(U8-Pad59)
- U8 pad 69: (no net) -> unconnected-(U8-Pad69)
- U8 pad 70: (no net) -> /IRQ11
- U8 pad 78: Net-(JP8-Pad2) -> Net-(U8-Pad78)
- U8 pad 79: Net-(C41-Pad2) -> unconnected-(U8-Pad79)
- U8 pad 82: (no net) -> unconnected-(U8-Pad82)
- U8 pad 83: (no net) -> unconnected-(U8-Pad83)
- U8 pad 84: (no net) -> unconnected-(U8-Pad84)
- U8 pad 85: (no net) -> unconnected-(U8-Pad85)
- U8 pad 86: (no net) -> unconnected-(U8-Pad86)
- U8 pad 89: (no net) -> unconnected-(U8-Pad89)
- U8 pad 90: /~RSTB -> /~{RSTB}
- U8 pad 91: (no net) -> unconnected-(U8-Pad91)
- U8 pad 93: (no net) -> unconnected-(U8-Pad93)
- U8 pad 94: (no net) -> unconnected-(U8-Pad94)
- U8 pad 95: (no net) -> unconnected-(U8-Pad95)
- U8 pad 96: (no net) -> unconnected-(U8-Pad96)
- Y2 pad 1: Net-(C41-Pad2) -> Net-(C64-Pad2)
- Y2 pad 3: Net-(C42-Pad2) -> Net-(C65-Pad2)
Routing:
- net GND: track 340.1 -> 998.9 mm, vias 13 -> 136
- net +12V: track 0.00 -> 181.6 mm, vias 0 -> 12
- net /OSC: track 0.00 -> 136.9 mm, vias 0 -> 4
- net /~{IOW}: track 0.00 -> 129.4 mm, vias 0 -> 3
- net /RESET: track 0.00 -> 118.3 mm, vias 0 -> 6
- net /IRQ5: track 0.00 -> 112.5 mm, vias 0 -> 2
- net /DRQ5: track 0.00 -> 109.6 mm, vias 0 -> 3
- net /DACK5: track 0.00 -> 109.0 mm, vias 0 -> 3
- net /IRQ7: track 0.00 -> 107.3 mm, vias 0 -> 2
- net /DRQ0: track 0.00 -> 107.2 mm, vias 0 -> 2
- net /IRQ9: track 0.00 -> 103.6 mm, vias 0 -> 2
- net /DACK0: track 0.00 -> 103.3 mm, vias 0 -> 2
- net /DRQ1: track 0.00 -> 98.0 mm, vias 0 -> 2
- net /DACK1: track 0.00 -> 95.3 mm, vias 0 -> 2
- net /IRQ10: track 0.00 -> 95.1 mm, vias 0 -> 2
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- added copper zone on B.Cu, net GND
- added copper zone on F.Cu, net GND
- added copper zone on In1.Cu, net GND
