File: pcb_top/rev.A/charon386_top.kicad_pcb (KiCad board)
At the start: 4 copper layers, 100 x 100 mm, 147 parts, among them J1 PC104_16, J2 Vol. Btns, J3 PC104, J5 ESP, J7 PJ-322, J9 Conn_02x07_Odd_Even, SW1 VGA Config, U1 TVGA9000I, U10 NE5532DR, U11 74HCT138, U12 SAM2695, U13 AMS1117-3.3, U14 74HC4050, U2 27C512PLCC, U3 MT4C4256, U4 MT4C4256, U5 MT4C4256, U6 MT4C4256, U7 AMS1117-5.0, U8 ES1868F, U9 AMS1117-5.0, Y1 40 MHz, Y2 12 MHz

Commit message: wip pcb rev.A
Parts:
- added C51: 1u, Capacitor_SMD:C_0603_1608Metric_Pad1.08x0.95mm_HandSolder, B.Cu at (122.2, 94.4)
- added C52: 1u, Capacitor_SMD:C_0603_1608Metric_Pad1.08x0.95mm_HandSolder, B.Cu at (175.3, 76.2)
- R31: renamed from R20; value 22 -> 33
- R32: renamed from R36; value 22 -> 33
- moved C27 44.8 mm to (138.0, 128.8), turned to -90 degrees
- moved C26 40.3 mm to (141.2, 130.5), turned to 90 degrees
- moved R17 28.7 mm to (170.6, 130.6), turned to -90 degrees
- moved R18 26.3 mm to (170.6, 126.6), turned to -90 degrees
- moved C50 1.66 mm to (173.4, 106.2), turned to 180 degrees
- moved JP1 1.30 mm to (147.2, 94.9)
- moved R31 0.60 mm to (109.4, 105.6)
- renumbered C27 to C1, C1 to C10, C2 to C11, C38 to C12, C37 to C13, C3 to C14, C39 to C15, C4 to C16, C5 to C17, C6 to C18, C7 to C19, C43 to C2, C33 to C20, C40 to C21, C13 to C22, C12 to C23, C11 to C24, C34 to C25, C17 to C26, C18 to C27, C14 to C28, C15 to C29, C29 to C3, C41 to C30, C42 to C31, C16 to C32, C62 to C33, C63 to C34, C64 to C35, C65 to C36, C20 to C37, C60 to C38, C21 to C39, C30 to C4, C22 to C40, C19 to C41, C23 to C42, C24 to C43, C69 to C44, C70 to C45, C66 to C46, C67 to C47, C68 to C48, C71 to C49, C31 to C5, C48 to C50, C61 to C53, C25 to C54, C26 to C55, C35 to C56, C36 to C57, C28 to C58, C44 to C59, C32 to C6, C45 to C60, C46 to C61, C47 to C62, C49 to C63, C50 to C64, C51 to C65, C52 to C66, C53 to C67, C54 to C68, C55 to C69, C8 to C7, C56 to C70, C57 to C71, C58 to C72, C59 to C73, C9 to C8, C10 to C9, FB4 to FB3, FB3 to FB4, J7 to J1, J9 to J3, J5 to J4, J1 to J5, J3 to J6, L5 to L1, L6 to L2, L7 to L3, L9 to L4, L10 to L5, L1 to L6, L2 to L7, L3 to L8, L8 to L9, R2 to R1, R21 to R10, R22 to R11, R23 to R12, R24 to R13, R25 to R14, R26 to R15, R30 to R16, R15 to R17, R16 to R18, R9 to R19, R32 to R2, R7 to R20, R10 to R21, R11 to R22, R12 to R23, R13 to R24, R14 to R25, R33 to R26, R34 to R27, R18 to R28, R35 to R29, R4 to R3, R31 to R30, R19 to R33, R8 to R34, R1 to R35, R17 to R36, R5 to R4, R6 to R5, R27 to R6, R28 to R7, R3 to R8, R29 to R9, U14 to U1, U9 to U10, U3 to U11, U4 to U12, U5 to U13, U6 to U14, U10 to U2, U11 to U3, U8 to U4, U1 to U5, U12 to U6, U2 to U7, U7 to U8, U13 to U9
Connections:
- J4 pad 5: unconnected-(J5-Pad5) -> Net-(J4-Pad5)
- J4 pad 6: unconnected-(J5-Pad6) (its old number) -> Net-(J4-Pad5)
- U3 pad 1: /A13 -> /A15
- U3 pad 3: /A15 -> /A13
- U4 pad 87: /MSD -> unconnected-(U4-Pad87)
- U4 pad 88: /MCLK -> unconnected-(U4-Pad88)
Routing:
- net GND: track 998.9 -> 197.9 mm, vias 136 -> 202
- net +5V: track 56.5 -> 561.1 mm, vias 16 -> 20
- net /~{RAS}: track 76.6 -> 40.9 mm, vias 2 -> 0
- net Net-(R17-Pad1): track 3.85 -> 36.6 mm
- net /~{CAS}: track 72.8 -> 44.0 mm, vias 2 -> 0
- net Net-(R18-Pad1): track 5.02 -> 33.4 mm
- net /LA18: track 37.8 -> 43.1 mm
- net /IOCHRDY: track 66.4 -> 62.5 mm
- net /AVDD_ES: track 21.0 -> 24.8 mm, vias 2 -> 4
- net /~{MEMW}: track 61.0 -> 57.5 mm
- net /MD2: track 91.2 -> 94.6 mm
- net Net-(J2-Pad4): track 90.7 -> 93.4 mm
- net Net-(J2-Pad6): track 91.0 -> 93.7 mm
- net unconnected-(J5-Pad5): track 2.54 -> 0.00 mm
- net Net-(J4-Pad5): track 0.00 -> 2.54 mm
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Other:
- outline, holes or cut-outs redrawn
- board text added: "1"
- board text added: "2"
- board text added: "3"
- board text added: "4"
- board text added: "Charon-386"
- board text added: "Eugene Lozovoy 2022"
- board text added: "Line in"
- board text added: "top board rev.A"

Commit message: wip pcb rev.A
Parts:
- added R37: 4.7k, Resistor_SMD:R_0603_1608Metric_Pad0.98x0.95mm_HandSolder, B.Cu at (146.9, 102.6)
- U7: value 27C512PLCC -> 27C256
- moved R23 0.80 mm to (146.9, 101.0)
- moved R25 0.60 mm to (146.9, 104.2)
Connections:
- U5 pad 97: /ROMA0 -> /ROMBA0
- U7 pad 10: /A1 -> /A2
- U7 pad 11: /A0 -> /A1
- U7 pad 2: /ROMA0 -> +5V
- U7 pad 24: /A10 -> /A11
- U7 pad 27: /A11 -> /A12
- U7 pad 28: /A9 -> /A10
- U7 pad 29: /A8 -> /A9
- U7 pad 3: /A12 -> /A13
- U7 pad 30: /A13 -> /A14
- U7 pad 31: /A14 -> /ROMBA0
- U7 pad 4: /A7 -> /A8
- U7 pad 5: /A6 -> /A7
- U7 pad 6: /A5 -> /A6
- U7 pad 7: /A4 -> /A5
- U7 pad 8: /A3 -> /A4
- U7 pad 9: /A2 -> /A3
Routing:
- net /ROMA0: track 127.0 -> 0.00 mm, vias 2 -> 0
- net /ROMBA0: track 0.00 -> 121.8 mm, vias 0 -> 2
- net /A0: track 144.2 -> 108.0 mm, vias 3 -> 2
- net /A13: track 124.1 -> 130.1 mm
- net +5V: track 561.1 -> 566.9 mm
- net /A10: track 139.9 -> 135.0 mm
- net /RMD5: track 49.7 -> 54.6 mm, vias 0 -> 1
- net /A11: track 135.3 -> 139.7 mm
- net GND: track 197.9 -> 202.3 mm, vias 202 -> 200
- net /~{ROMCS}: track 41.3 -> 44.9 mm
- net /A6: track 127.2 -> 130.4 mm
- net /A8: track 128.7 -> 126.7 mm
- net /A7: track 127.0 -> 128.6 mm
- net /A4: track 131.6 -> 133.0 mm
- net /A5: track 130.5 -> 131.9 mm
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