File: pcb_top/rev.A/charon386_top.kicad_pcb (KiCad board)
At the start: 4 copper layers, 100 x 100 mm, 150 parts, among them J1 PJ-322, J2 Vol. Btns, J3 Conn_02x07_Odd_Even, J4 ESP, J5 PC104_16, J6 PC104, SW1 VGA Config, U1 74HC4050, U10 AMS1117-5.0, U11 MT4C4256, U12 MT4C4256, U13 MT4C4256, U14 MT4C4256, U2 NE5532DR, U3 74HCT138, U4 ES1868F, U5 TVGA9000I, U6 SAM2695, U7 27C256, U8 AMS1117-5.0, U9 AMS1117-3.3, Y1 40 MHz, Y2 12 MHz

Commit message: wip pcb rev.A
Parts:
- added C74: 100u, Capacitor_Tantalum_SMD:CP_EIA-7343-31_Kemet-D_Pad2.25x2.55mm_HandSolder, B.Cu at (179.0, 67.8)
Routing:
- net GND: track 202.3 -> 207.4 mm, vias 200 -> 221

Commit message: wip pcb rev.A
Parts:
- moved C62 0.10 mm to (136.8, 107.0)
Routing:
- net Net-(C10-Pad1): track 9.02 -> 5.79 mm
- net Net-(J2-Pad6): track 93.7 -> 96.0 mm
- net Net-(C14-Pad1): track 3.37 -> 1.38 mm
- net /DRQ5: track 109.7 -> 108.1 mm
- net /RESET: track 118.3 -> 116.9 mm
- net /A1: track 142.7 -> 141.8 mm
- net /ALE: track 77.1 -> 77.7 mm
- net /A14: track 124.7 -> 125.3 mm
- net +5V: track 566.9 -> 567.5 mm
- net /A12: track 129.7 -> 130.3 mm
- net /AEN: track 80.6 -> 80.1 mm
Other:
- board text added: "Layers: 4 Dimensions: 100x100mm Thickness: 1.6mm"
- board text added: "Min clearance: 0.2mm Min track: 0.2mm Min hole: 0.3mm Min annular ring: 0.15mm"

Commit message: wip pcb rev.A
Changed lines of the file:
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@@
     )
   )
+  (gr_rect (start 194.95 61.4) (end 197.5 70.6) (layer "F.Cu") (width 0.2) (fill none))
+  (gr_rect (start 194.95 61.4) (end 197.5 70.6) (layer "In1.Cu") (width 0.2) (fill none))
+  (gr_rect (start 194.95 61.4) (end 197.5 70.6) (layer "In2.Cu") (width 0.2) (fill none))
+  (gr_rect (start 194.95 61.4) (end 197.5 70.6) (layer "B.Cu") (width 0.2) (fill none))
   (gr_line (start 165 62.4) (end 159.8 62.4) (layer "F.SilkS") (width 0.15))
   (gr_line (start 123.2 86) (end 123.2 86.4) (layer "F.SilkS") (width 0.15))
@@
   (gr_line (start 98.75 104.5) (end 107 104.5) (layer "Edge.Cuts") (width 0.1))
   (gr_line (start 121.2 47.7) (end 133.5 47.7) (layer "Edge.Cuts") (width 0.1))
-  (gr_text "1" (at 196.25 62.899654) (layer "F.Cu")
+  (gr_text "1" (at 196.225 62.899654) (layer "F.Cu")
     (effects (font (size 1.5 1.5) (thickness 0.3)))
   )
-  (gr_text "2" (at 196.25 64.999654) (layer "In1.Cu")
+  (gr_text "2" (at 196.225 64.999654) (layer "In1.Cu")
     (effects (font (size 1.5 1.5) (thickness 0.3)))
   )
-  (gr_text "3" (at 196.25 67.099654) (layer "In2.Cu")
+  (gr_text "3" (at 196.225 67.099654) (layer "In2.Cu")
     (effects (font (size 1.5 1.5) (thickness 0.3)))
   )
-  (gr_text "4" (at 196.25 69.199654) (layer "B.Cu")
+  (gr_text "4" (at 196.225 69.199654) (layer "B.Cu")
     (effects (font (size 1.5 1.5) (thickness 0.3)))
   )
@@
       )
     )
-  )
-  (zone (net 0) (net_name "") (layers "F.Cu" "In1.Cu" "In2.Cu" "B.Cu") (hatch edge 0.508)
-    (connect_pads (clearance 0))
-    (min_thickness 0.254)
-    (keepout (tracks allowed) (vias allowed) (pads allowed ) (copperpour not_allowed) (footprints allowed))
-    (fill (thermal_gap 0.508) (thermal_bridge_width 0.508))
-    (polygon
-      (pts
-        (xy 197.4 70.499654)
-        (xy 195 70.499654)
-        (xy 195 61.499654)
-        (xy 197.5 61.499654)
-      )
-    )
