File: pcb_top/rev.A/charon386_top.kicad_sch (KiCad schematic)
At the start: 59 parts, among them J1 PC104_16, J2 AudioJack3, J3 PC104, J4 Jumper for 8-bit bus, J5 DB15_Female_HighDensity_Mount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, SW1 VGA Config, U1 TVGA9000I, U7 27C040, U8 ES1868F, Y1 12 MHz

Commit message: wip pcb rev.A
Parts:
- removed U7: 27C040, Package_LCC:PLCC-32_THT-Socket, symbol Memory_EPROM:27C040
- added U2: 27C512PLCC, my:PLCC-32_11.4x14.0mm_P1.27mm-longpads, symbol Memory_EPROM:27C512PLCC
Connections:
- net +5V: now also U2.32 (VCC)
- net A0: now also U2.11 (A0)
- net A1: now also U2.10 (A1)
- net A10: now also U2.24 (A10)
- net A11: now also U2.27 (A11)
- net A12: now also U2.3 (A12)
- net A13: now also U2.30 (A13)
- net A14: now also U2.31 (A14)
- net A2: now also U2.9 (A2)
- net A3: now also U2.8 (A3)
- net A4: now also U2.7 (A4)
- net A5: now also U2.6 (A5)
- net A6: now also U2.5 (A6)
- net A7: now also U2.4 (A7)
- net A8: now also U2.29 (A8)
- net A9: now also U2.28 (A9)
- net GND: now also U2.16 (GND), U2.23 (~CE)
- net RMD0: now also U2.13 (O0)
- net RMD1: now also U2.14 (O1)
- net RMD2: now also U2.15 (O2)
- net RMD3: now also U2.18 (O3)
- net RMD4: now also U2.19 (O4)
- net RMD5: now also U2.20 (O5)
- net RMD6: now also U2.21 (O6)
- net RMD7: now also U2.22 (O7)
- net ROMA0: now also U2.2 (A15)
- net ~ROMCS: now also U2.25 (~OE~/VPP)
Changed lines of the file:
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@@
   (junction (at 43.18 115.57) (diameter 1.016) (color 0 0 0 0))
   (junction (at 49.53 118.745) (diameter 1.016) (color 0 0 0 0))
-  (junction (at 86.995 227.965) (diameter 1.016) (color 0 0 0 0))
-  (junction (at 86.995 230.505) (diameter 1.016) (color 0 0 0 0))
   (junction (at 94.615 85.09) (diameter 1.016) (color 0 0 0 0))
   (junction (at 158.75 164.465) (diameter 1.016) (color 0 0 0 0))
@@
     (stroke (width 0) (type solid) (color 0 0 0 0))
   )
-  (wire (pts (xy 76.835 240.665) (xy 86.995 240.665))
+  (wire (pts (xy 76.835 227.965) (xy 86.995 227.965))
     (stroke (width 0) (type solid) (color 0 0 0 0))
   )
@@
     (stroke (width 0) (type solid) (color 0 0 0 0))
   )
-  (wire (pts (xy 86.995 225.425) (xy 86.995 227.965))
-    (stroke (width 0) (type solid) (color 0 0 0 0))
-  )
-  (wire (pts (xy 86.995 227.965) (xy 86.995 230.505))
-    (stroke (width 0) (type solid) (color 0 0 0 0))
-  )
   (wire (pts (xy 94.615 82.55) (xy 94.615 85.09))
     (stroke (width 0) (type solid) (color 0 0 0 0))
@@
     (effects (font (size 1 1)) (justify left bottom))
   )
-  (label "~ROMCS" (at 76.835 240.665 0)
+  (label "~ROMCS" (at 76.835 227.965 0)
     (effects (font (size 1 1)) (justify left bottom))
   )
@@
     (pin "1")
   )
-  (symbol (lib_id "power:+5V") (at 86.995 235.585 90) (unit 1)
-    (in_bom yes) (on_board yes)
-    (property "Reference" "#PWR0123" (id 0) (at 90.805 235.585 0)
-      (effects (font (size 1 1)) hide)
-    )
-    (property "Value" "+5V" (id 1) (at 82.1776 235.585 90)
-      (effects (font (size 1 1)))
-    )
-    (property "Footprint" "" (id 2) (at 86.995 235.585 0)
-      (effects (font (size 1.27 1.27)) hide)
-    )
-    (property "Datasheet" "" (id 3) (at 86.995 235.585 0)
-      (effects (font (size 1.27 1.27)) hide)
-    )
-    (pin "1")
-  )
   (symbol (lib_id "power:+5V") (at 94.615 77.47 90) (unit 1)
     (in_bom yes) (on_board yes)
@@
   (symbol (lib_id "power:GND") (at 86.995 230.505 270) (unit 1)
     (in_bom yes) (on_board yes)
-    (property "Reference" "#PWR0125" (id 0) (at 80.645 230.505 0)
+    (property "Reference" "#PWR0124" (id 0) (at 80.645 230.505 0)
       (effects (font (size 1 1)) hide)
     )
@@
     (pin "1")
   )
-  (symbol (lib_id "power:GND") (at 86.995 238.125 270) (unit 1)
-    (in_bom yes) (on_board yes)
-    (property "Reference" "#PWR0124" (id 0) (at 80.645 238.125 0)
-      (effects (font (size 1 1)) hide)
-    )
-    (property "Value" "GND" (id 1) (at 82.55 238.125 90)
-      (effects (font (size 1 1)))
-    )
-    (property "Footprint" "" (id 2) (at 86.995 238.125 0)
-      (effects (font (size 1.27 1.27)) hide)
-    )
-    (property "Datasheet" "" (id 3) (at 86.995 238.125 0)
-      (effects (font (size 1.27 1.27)) hide)
-    )
-    (pin "1")
-  )
   (symbol (lib_id "power:GND") (at 94.615 36.83 270) (unit 1)
     (in_bom yes) (on_board yes)
@@
     (pin "1")
   )
-  (symbol (lib_id "power:GND") (at 97.155 245.745 0) (unit 1)
+  (symbol (lib_id "power:GND") (at 97.155 238.125 0) (unit 1)
     (in_bom yes) (on_board yes)
-    (property "Reference" "#PWR0122" (id 0) (at 97.155 252.095 0)
+    (property "Reference" "#PWR0122" (id 0) (at 97.155 244.475 0)
       (effects (font (size 1 1)) hide)
     )
-    (property "Value" "GND" (id 1) (at 97.155 249.555 0)
+    (property "Value" "GND" (id 1) (at 97.155 241.935 0)
       (effects (font (size 1 1)))
     )
-    (property "Footprint" "" (id 2) (at 97.155 245.745 0)
+    (property "Footprint" "" (id 2) (at 97.155 238.125 0)
       (effects (font (size 1.27 1.27)) hide)
     )
-    (property "Datasheet" "" (id 3) (at 97.155 245.745 0)
+    (property "Datasheet" "" (id 3) (at 97.155 238.125 0)
       (effects (font (size 1.27 1.27)) hide)
     )
@@
     (pin "9")
   )
-  (symbol (lib_id "Memory_EPROM:27C040") (at 97.155 212.725 0) (unit 1)
+  (symbol (lib_id "Memory_EPROM:27C512PLCC") (at 97.155 207.645 0) (unit 1)
     (in_bom yes) (on_board yes)
-    (property "Reference" "U7" (id 0) (at 90.17 180.975 0)
-      (effects (font (size 1 1)))
-    )
-    (property "Value" "27C040" (id 1) (at 102.235 180.975 0)
-      (effects (font (size 1 1)))
-    )
-    (property "Footprint" "Package_LCC:PLCC-32_THT-Socket" (id 2) (at 97.155 212.725 0)
+    (property "Reference" "U2" (id 0) (at 90.17 180.975 0))
+    (property "Value" "27C512PLCC" (id 1) (at 104.14 180.975 0))
+    (property "Footprint" "my:PLCC-32_11.4x14.0mm_P1.27mm-longpads" (id 2) (at 97.155 207.645 0)
       (effects (font (size 1.27 1.27)) hide)
     )
-    (property "Datasheet" "http://ww1.microchip.com/downloads/en/devicedoc/doc0189.pdf" (id 3) (at 97.155 212.725 0)
+    (property "Datasheet" "http://ww1.microchip.com/downloads/en/DeviceDoc/doc0015.pdf" (id 3) (at 97.155 207.645 0)
       (effects (font (size 1.27 1.27)) hide)
     )
@@
       (reference "#PWR0122") (unit 1) (value "GND") (footprint "")
     )
-    (path "/afa051fe-f996-40fc-b318-6aa0774acd5f"
-      (reference "#PWR0123") (unit 1) (value "+5V") (footprint "")
-    )
     (path "/60026849-71b3-46c6-a0b4-8cfea275ea3e"
       (reference "#PWR0124") (unit 1) (value "GND") (footprint "")
     )
-    (path "/701886de-2932-476a-a847-534527e90b18"
-      (reference "#PWR0125") (unit 1) (value "GND") (footprint "")
-    )
     (path "/60931779-8dec-4513-9bd5-63487359f1c1"
       (reference "#PWR0126") (unit 1) (value "+5V") (footprint "")
@@
       (reference "U1") (unit 1) (value "TVGA9000I") (footprint "Package_QFP:PQFP-160_28x28mm_P0.65mm")
     )
-    (path "/b7657fc7-fd18-420c-84cc-275d981edd9a"
-      (reference "U7") (unit 1) (value "27C040") (footprint "Package_LCC:PLCC-32_THT-Socket")
+    (path "/cac7438b-c7a2-4b35-85e0-723b0d42f034"
+      (reference "U2") (unit 1) (value "27C512PLCC") (footprint "my:PLCC-32_11.4x14.0mm_P1.27mm-longpads")
     )
     (path "/3384d8e9-621d-40dd-b676-452c093e7e5a"

Commit message: wip pcb rev.A
Parts:
- Y1: footprint Crystal:Crystal_HC49-U_Vertical -> Crystal:Crystal_SMD_SeikoEpson_TSX3225-4Pin_3.2x2.5mm_HandSoldering
Connections:
- net +5V: no longer R2.1
- net GND: now also Y1.2, Y1.4
- no-connect marks 66 -> 64
Other:
- moved on the sheet: C1, C10, C11, C12, C13, C14, C15, C16, C17, C18, C19, C2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

Commit message: wip pcb rev.A
Parts:
- removed J2: AudioJack3, Connector_Audio:Jack_3.5mm_CUI_SJ1-3535NG_Horizontal, symbol Connector:AudioJack3
- added C21, C23, C25, C38: 10u, Capacitor_SMD:C_0603_1608Metric_Pad1.08x0.95mm_HandSolder, symbol Device:C
- added C22, C24, C26, C36: 100n, Capacitor_SMD:C_0603_1608Metric_Pad1.08x0.95mm_HandSolder, symbol Device:C
- added C27, C28, C29, C30, C31, C32, C33, C34: 220n, Capacitor_SMD:C_0603_1608Metric_Pad1.08x0.95mm_HandSolder, symbol Device:C
- added C35: 100u/16V, Capacitor_Tantalum_SMD:CP_EIA-6032-28_Kemet-C_Pad2.25x2.35mm_HandSolder, symbol Device:CP
- added C37: 10n, Capacitor_SMD:C_0603_1608Metric_Pad1.08x0.95mm_HandSolder, symbol Device:C
- added C39, C40: 47u, Capacitor_Tantalum_SMD:CP_EIA-3216-18_Kemet-A_Pad1.58x1.35mm_HandSolder, symbol Device:CP
- added J2: AUX_A, Connector_PinHeader_2.54mm:PinHeader_1x03_P2.54mm_Vertical, symbol Connector_Generic:Conn_01x03
- added J6: Wavetable, Connector_PinHeader_2.54mm:PinHeader_2x13_P2.54mm_Vertical, symbol Connector_Generic:Conn_02x13_Odd_Even
- added J7, J8: PJ-322, my:PJ-322, symbol Connector:AudioJack4
- added JP2, JP3, JP4, JP5: SolderJumper_2_Open, Jumper:SolderJumper-2_P1.3mm_Open_RoundedPad1.0x1.5mm, symbol Jumper:SolderJumper_2_Open
- added JP6: WTBL. P20, Jumper:SolderJumper-3_P1.3mm_Open_RoundedPad1.0x1.5mm_NumberLabels, symbol Jumper:SolderJumper_3_Open
- added JP7: WTBL. P24, Jumper:SolderJumper-3_P1.3mm_Open_RoundedPad1.0x1.5mm_NumberLabels, symbol Jumper:SolderJumper_3_Open
- added L2, L3, L8: 5.7u, Inductor_SMD:L_1210_3225Metric_Pad1.42x2.65mm_HandSolder, symbol Device:L
- added L4, L5, L6, L7, L? (x2): BLM21PG331BH1D, Inductor_SMD:L_1210_3225Metric_Pad1.42x2.65mm_HandSolder, symbol Device:L
- added R18: 100, Resistor_SMD:R_0603_1608Metric_Pad0.98x0.95mm_HandSolder, symbol Device:R
- added R19, R25, R26, R29, R30: 10k, Resistor_SMD:R_0603_1608Metric_Pad0.98x0.95mm_HandSolder, symbol Device:R
- added R20: 22k, Resistor_SMD:R_0603_1608Metric_Pad0.98x0.95mm_HandSolder, symbol Device:R
- added R21, R23: 15k, Resistor_SMD:R_0603_1608Metric_Pad0.98x0.95mm_HandSolder, symbol Device:R
- added R22, R24: 33k, Resistor_SMD:R_0603_1608Metric_Pad0.98x0.95mm_HandSolder, symbol Device:R
- added R27, R28: 1k, Resistor_SMD:R_0603_1608Metric_Pad0.98x0.95mm_HandSolder, symbol Device:R
- added U10: NE5532DR, Package_SO:SOIC-8_3.9x4.9mm_P1.27mm, symbol Amplifier_Operational:NE5532
- added U11: 74HCT138, Package_SO:TSSOP-16_4.4x5mm_P0.65mm, symbol 74xx:74LS138
- added U3, U4, U5, U6: MT4C4256, Package_DIP:DIP-20_W7.62mm, symbol my:MT4C4256
- added U7, U9: AMS1117-5.0, Package_TO_SOT_SMD:SOT-223-3_TabPin2, symbol Regulator_Linear:AMS1117-5.0
- C11: value 47p -> 1u
- J3: Field4 B A -> A B
- R10, R11, R12, R13, R14, R9: value 1k -> 4.7k
- U1: footprint Package_QFP:PQFP-160_28x28mm_P0.65mm -> my:PQFP-160_28x28mm_P0.65mm_LongPads
- U8: symbol ess:ES1868F -> my:ES1868F
- Y1: value 12 MHz -> 40 MHz
Connections:
- net +5V: now also J6.10 (Pin_10), J6.14 (Pin_14), J6.6 (Pin_6), U11.16 (VCC), U11.6 (E3), U3.10 (VCC), U4.10 (VCC), U5.10 (VCC), U6.10 (VCC), U7.3 (VI), U9.3 (VI)
- net A0: now also U8.99 (A0)
- net A1: now also U8.100 (A1)
- net A10: now also U8.97 (A10)
- net A11: now also U8.98 (A11)
- net A12: now also U11.4 (E1)
- net A13: now also U11.1 (A0)
- net A14: now also U11.2 (A1)
- net A15: now also U11.3 (A2)
- net A2: now also U8.1 (A2)
- net A3: now also U8.2 (A3)
- net A4: now also U8.4 (A4)
- net A5: now also U8.5 (A5)
- net A6: now also U8.6 (A6)
- net A7: now also U8.8 (A7)
- net A8: now also U8.9 (A8)
- net A9: now also U8.10 (A9)
- net AEN: now also U11.5 (E2)
- net D0: now also U8.12 (D0)
- net D1: now also U8.13 (D1)
- net D2: now also U8.14 (D2)
- net D3: now also U8.15 (D3)
- net D4: now also U8.16 (D4)
- net D5: now also U8.17 (D5)
- net D6: now also U8.18 (D6)
- net D7: now also U8.19 (D7)
- net GND: now also J6.1 (Pin_1), J6.11 (Pin_11), J6.3 (Pin_3), J6.5 (Pin_5), J6.7 (Pin_7), J6.9 (Pin_9), R19.2, R20.2, U11.8 (GND), U3.16 (~OE), U3.20 (GND), U4.16 (~OE), U4.20 (GND), U5.16 (~OE), U5.20 (GND), U6.16 (~OE), U6.20 (GND)
- net GNDA: now also C21.1, C22.2, C23.1, C24.2, C25.1, C26.2, C35.2, C36.2, C37.1, C38.1, J2.3 (Pin_3), J6.15 (Pin_15), J6.17 (Pin_17), J6.19 (Pin_19), J6.21 (Pin_21), J6.23 (Pin_23), J6.25 (Pin_25), J7.R2, J7.S, J8.R2, J8.S, R25.2, R26.2, R28.1, U10.4 (V-), U7.1 (GND), U9.1 (GND)
- net MAA0: now also U3.6 (A0), U4.6 (A0)
- net MAA1: now also U3.7 (A1), U4.7 (A1)
- net MAA2: now also U3.8 (A2), U4.8 (A2)
- net MAA3: now also U3.9 (A3), U4.9 (A3)
- net MAA4: now also U3.11 (A4), U4.11 (A4)
- net MAA5: now also U3.12 (A5), U4.12 (A5)
- net MAA6: now also U3.13 (A6), U4.13 (A6)
- net MAA7: now also U3.14 (A7), U4.14 (A7)
- net MAA8: now also U3.15 (A8), U4.15 (A8)
- net MAB0: now also U5.6 (A0), U6.6 (A0)
- net MAB1: now also U5.7 (A1), U6.7 (A1)
- net MAB2: now also U5.8 (A2), U6.8 (A2)
- net MAB3: now also U5.9 (A3), U6.9 (A3)
- net MAB4: now also U5.11 (A4), U6.11 (A4)
- net MAB5: now also U5.12 (A5), U6.12 (A5)
- net MAB6: now also U5.13 (A6), U6.13 (A6)
- net MAB7: now also U5.14 (A7), U6.14 (A7)
- net MAB8: now also U5.15 (A8), U6.15 (A8)
- net MD0: now also U3.1 (DQ1)
- net MD1: now also U3.2 (DQ2)
- net MD16: now also U5.1 (DQ1)
- net MD17: now also U5.2 (DQ2)
- net MD18: now also U5.18 (DQ3)
- net MD19: now also U5.19 (DQ4)
- net MD2: now also U3.18 (DQ3)
- net MD20: now also U6.1 (DQ1)
- net MD21: now also U6.2 (DQ2)
- net MD22: now also U6.18 (DQ3)
- net MD23: now also U6.19 (DQ4)
- net MD3: now also U3.19 (DQ4)
- net MD4: now also U4.1 (DQ1)
- net MD5: now also U4.2 (DQ2)
- net MD6: now also U4.18 (DQ3)
- net MD7: now also U4.19 (DQ4)
- net OSC: now also U8.78 (XI)
- net RESET: now also R17.2, U1.5 (RESET), U8.81 (RESET); no longer J3.3 (Pin_3), R17.1
- net ~CAS: now also U3.17 (~CAS), U4.17 (~CAS), U5.17 (~CAS), U6.17 (~CAS)
- net ~IOR: now also U8.75 (~IORB)
- net ~IOW: now also U8.76 (~IOWB); no longer C14.1
- net ~MEMR: now also R18.2; no longer C15.1, U1.155 (~MEMR)
- net ~RAS: now also U3.4 (~RAS), U4.4 (~RAS), U5.4 (~RAS), U6.4 (~RAS)
- net ~WE0: now also U3.3 (~WE), U4.3 (~WE)
- net ~WE2: now also U5.3 (~WE), U6.3 (~WE)
- net at U8.11 (AEN): now also U11.15 (O0)
- net at U8.35 (AUXB_L): now also C29.1
- net at U8.36 (AUXB_R): now also C30.1
- net at U8.37 (AUXA_L): now also C27.1
- net at U8.38 (AUXA_R): now also C28.1
- net AVDD_ES: now reaches U8.43 (VDDA)
- net AVDD_ES: now also C25.2, C26.1, U9.2 (VO)
- net at U8.48 (LINE_L): now also C31.1
- net at U8.49 (LINE_R): now also C32.1
- net at U8.50 (AOUT_L): now also R23.2
- net at U8.51 (AOUT_R): now also R21.2
- net MSO: now reaches U8.58 (MSO)
- net MSO: now also J6.4 (Pin_4)
- net DRQ3: now reaches U8.63 (DRQC)
- net DRQ3: now also J3.31 (Pin_31)
- net DACK3: now reaches U8.64 (~DACKBC)
- net DACK3: now also J3.29 (Pin_29)
- net DRQ1: now reaches U8.65 (DRQB)
- net DRQ1: now also J3.35 (Pin_35)
- net DACK1: now reaches U8.66 (~DACKBB)
- net DACK1: now also J3.33 (Pin_33)
- net at U8.67 (DRQA): now also JP4.2 (B)
- net at U8.68 (~DACKBA): now also JP5.2 (B)
- net at U8.70 (IRQE): now also JP3.2 (B)
- net at U8.71 (IRQD): now also JP2.2 (B)
- net IRQ7: now reaches U8.72 (IRQC)
- net IRQ7: now also J3.41 (Pin_41)
- net IRQ5: now reaches U8.73 (IRQB)
- net IRQ5: now also J3.45 (Pin_45)
- net IRQ9: now reaches U8.74 (IRQA)
- net IRQ9: now also J3.7 (Pin_7)
- net MSD: now reaches U8.87 (MSD)
- net MSD: now also J6.12 (Pin_12)
- net MCLK: now reaches U8.88 (MCLK)
- net MCLK: now also J6.2 (Pin_2), R20.1
- net ~RSTB: now reaches U8.90 (~RSTB)
- net ~RSTB: now also J6.26 (Pin_26)
- net at U8.92 (GPIRQ): now also R19.1
- net at R7.1, U1.154 (~IOW): now also C14.1
- net -12V: now reaches J3.13 (Pin_13)
- net -12V: now also J6.22 (Pin_22)
- net +12V: now reaches J3.17 (Pin_17)
- net +12V: now also J6.18 (Pin_18), L8.1
- net IRQ4: now reaches J3.47 (Pin_47)
- net IRQ4: now also JP3.1 (A)
- net IRQ3: now reaches J3.49 (Pin_49)
- net IRQ3: now also JP2.1 (A)
- net DACK2: now reaches J3.51 (Pin_51)
- net DACK2: now also JP5.1 (A)
- net +5VA renamed AVDD1
- net AVDD1: now also C21.2, C22.1, L2.2; no longer U1.13 (AVDD2), U1.6 (AVDD2)
- new net: C27.2, L4.1
- new net: R24.1, R30.2, U10.2 (-)
- new net: C34.2, R24.2
- new net: C15.1, R18.1, U1.155 (~MEMR)
- new net: C34.1, R23.1, R25.1
- new net: C39.1, R29.1, U10.7
- new net: R22.1, R29.2, U10.6 (-)
- new net: C40.1, R30.1, U10.1
- new net: C40.2, L?.1
- new net: C19.2, J3.3 (Pin_3), R17.1
- new net: J6.20 (Pin_20), JP6.2 (C)
- new net: J6.24 (Pin_24), JP7.2 (C)
- new net: C37.2, C38.2, R27.1, R28.2, U10.3 (+), U10.5 (+)
- new net: C32.2, L7.1
- new net: C33.1, R21.1, R26.1
- new net: C33.2, R22.2
- new net: L2.1, L3.1, U7.2 (VO)
- new net: C39.2, L?.1
- new net: C28.2, L5.1
- new net: C31.2, L6.1
- new net AOUT_L: J8.T, L?.2
- new net AOUT_R: J8.R1, L?.2
- new net AUXA_L: J2.1 (Pin_1), L4.2
- new net AUXA_R: J2.2 (Pin_2), L5.2
- new net AUXBL: JP6.3 (B), JP7.3 (B)
- new net AUXBR: JP6.1 (A), JP7.1 (A)
- new net AUXB_L: C29.2
- new net AUXB_R: C30.2
- new net AVDD2: C23.2, C24.1, L3.2, U1.13 (AVDD2), U1.6 (AVDD2)
- new net AVDD_OP: C35.1, C36.1, L8.2, R27.2, U10.8 (V+)
- new net DRQ2: JP4.1 (A)
- new net LINE_L: J7.T, L6.2
- new net LINE_R: J7.R1, L7.2
- no-connect marks 64 -> 77
Other:
- moved on the sheet: C1, C14, C15, C19, C2, C20, C3, C4, C5, C6, C7, J3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

Commit message: wip pcb rev.A
Parts:
- removed H1, H2, H3, H4: MountingHole, my:MountingHole_3.2mm_M3_dk5.2mm_Mask, symbol Mechanical:MountingHole
- removed J2: AUX_A, Connector_PinHeader_2.54mm:PinHeader_1x03_P2.54mm_Vertical, symbol Connector_Generic:Conn_01x03
- removed J5: DB15_Female_HighDensity_MountingHoles, Connector_Dsub:DSUB-15-HD_Female_Horizontal_P2.29x1.98mm_EdgePinOffset3.03mm_Housed_MountingHolesOffset4.94mm, symbol Connector:DB15_Female_HighDensity_MountingHoles
- removed J8: PJ-322, my:PJ-322, symbol Connector:AudioJack4
- removed JP2, JP3, JP4, JP5: SolderJumper_2_Open, Jumper:SolderJumper-2_P1.3mm_Open_RoundedPad1.0x1.5mm, symbol Jumper:SolderJumper_2_Open
- removed L4: BLM21PG331BH1D, Inductor_SMD:L_1210_3225Metric_Pad1.42x2.65mm_HandSolder, symbol Device:L
- added C41, C42: 10p, Capacitor_SMD:C_0603_1608Metric_Pad1.08x0.95mm_HandSolder, symbol Device:C
- added C43: 4.7n, Capacitor_SMD:C_0603_1608Metric_Pad1.08x0.95mm_HandSolder, symbol Device:C
- added C44, C45, C46, C47, C49, C50, C51, C52, C53, C54, C55, C56, C57, C58, C59: 100n, Capacitor_SMD:C_0603_1608Metric_Pad1.08x0.95mm_HandSolder, symbol Device:C
- added C48, C60, C61: 1u, Capacitor_SMD:C_0603_1608Metric_Pad1.08x0.95mm_HandSolder, symbol Device:C
- added J2: Vol. Btns, Connector_PinHeader_2.54mm:PinHeader_2x03_P2.54mm_Vertical, symbol Connector_Generic:Conn_02x03_Odd_Even
- added J9: Conn_02x07_Odd_Even, Connector_PinHeader_2.54mm:PinHeader_2x08_P2.54mm_Vertical, symbol Connector_Generic:Conn_02x08_Odd_Even
- added JP8: SolderJumper_3_Bridged12, Jumper:SolderJumper-3_P1.3mm_Bridged12_RoundedPad1.0x1.5mm_NumberLabels, symbol Jumper:SolderJumper_3_Bridged12
- added JP9: SolderJumper_2_Open, Jumper:SolderJumper-2_P1.3mm_Open_RoundedPad1.0x1.5mm, symbol Jumper:SolderJumper_2_Open
- added R31: 10k, Resistor_SMD:R_0603_1608Metric_Pad0.98x0.95mm_HandSolder, symbol Device:R
- added R32: 4.7k, Resistor_SMD:R_0603_1608Metric_Pad0.98x0.95mm_HandSolder, symbol Device:R
- added R33, R34, R35: 1k, Resistor_SMD:R_0603_1608Metric_Pad0.98x0.95mm_HandSolder, symbol Device:R
- added Y2: 14.318 MHz, Crystal:Crystal_SMD_SeikoEpson_TSX3225-4Pin_3.2x2.5mm_HandSoldering, symbol Device:Crystal_GND24
- C21, C23, C25, C38: footprint Capacitor_SMD:C_0603_1608Metric_Pad1.08x0.95mm_HandSolder -> Capacitor_SMD:C_0805_2012Metric_Pad1.18x1.45mm_HandSolder
- C27, C28: value 220n -> 100n
- C39, C40: footprint Capacitor_Tantalum_SMD:CP_EIA-3216-18_Kemet-A_Pad1.58x1.35mm_HandSolder -> Capacitor_Tantalum_SMD:CP_EIA-3528-21_Kemet-B_Pad1.50x2.35mm_HandSolder
- J1: footprint Connector_PinSocket_2.54mm:PinSocket_2x20_P2.54mm_Vertical -> Connector_PinHeader_2.54mm:PinHeader_2x20_P2.54mm_Vertical
- J3: footprint Connector_PinSocket_2.54mm:PinSocket_2x32_P2.54mm_Vertical -> Connector_PinHeader_2.54mm:PinHeader_2x32_P2.54mm_Vertical
- J6: footprint Connector_PinHeader_2.54mm:PinHeader_2x13_P2.54mm_Vertical -> Connector_PinHeader_2.54mm:PinHeader_2x13_P2.54mm_Horizontal
- JP6, JP7: footprint Jumper:SolderJumper-3_P1.3mm_Open_RoundedPad1.0x1.5mm_NumberLabels -> Jumper:SolderJumper-3_P1.3mm_Bridged12_RoundedPad1.0x1.5mm_NumberLabels; symbol Jumper:SolderJumper_3_Open -> Jumper:SolderJumper_3_Bridged12
- L10, L9: renamed from L?; footprint Inductor_SMD:L_1210_3225Metric_Pad1.42x2.65mm_HandSolder -> Inductor_SMD:L_0805_2012Metric_Pad1.15x1.40mm_HandSolder
- L5, L6, L7: footprint Inductor_SMD:L_1210_3225Metric_Pad1.42x2.65mm_HandSolder -> Inductor_SMD:L_0805_2012Metric_Pad1.15x1.40mm_HandSolder
- R2: value 0 -> 47k
- R27, R28: value 1k -> 10k
Connections:
- net GNDA is gone; now on net GND: C1.2, C10.2, C11.2, C12.2, C13.2, C2.2, C21.1, C22.2, C23.1, C24.2, C25.1, C26.2, C3.2, C35.2, C36.2, C37.1, C38.1, C5.2, C7.2, C8.2, C9.2, J6.15 (Pin_15), J6.17 (Pin_17), J6.19 (Pin_19), J6.21 (Pin_21), J6.23 (Pin_23), J6.25 (Pin_25), J7.R2, J7.S, R25.2, R26.2, R28.1, R4.2, R5.2, R6.2, R8.2, U1.1 (AVSS2), U1.126 (AVSS), U10.4 (V-), U7.1 (GND), U8.41 (GNDA), U9.1 (GND)
- net +12V: now also U7.3 (VI), U9.3 (VI), C60.1, C61.1
- net +5V: now also C28.1, C44.1, C45.1, C46.1, C47.1, C48.1, C49.1, C50.1, C51.1, C52.1, C53.1, C54.1, C55.1, C56.1, C57.1, C58.1, C59.1; no longer U7.3 (VI), U9.3 (VI)
- net AOUT_L: now also J9.1 (Pin_1)
- net AOUT_R: now also J9.2 (Pin_2)
- net AUXB_L: now also JP6.1 (A), JP7.3 (B)
- net AUXB_R: now also JP6.3 (B), JP7.1 (A)
- net GND: now also C28.2, U8.25 (PSEL1), C41.1, C42.1, C43.1, C44.2, C45.2, C46.2, C47.2, C48.2, C49.2, C50.2, C51.2, C52.2, C53.2, C54.2, C55.2, C56.2, C57.2, C58.2, C59.2, C60.2, C61.2, J2.1 (Pin_1), J2.3 (Pin_3), J2.5 (Pin_5), J9.11 (Pin_11), J9.12 (Pin_12), J9.3 (Pin_3), J9.4 (Pin_4), J9.7 (Pin_7), R31.2, R32.2, Y2.2, Y2.4
- net HSYNC: now also FB5.1; no longer FB5.2
- net Monitor: now also FB3.1; no longer FB3.2
- net OSC: now also JP8.1 (A); no longer U8.78 (XI)
- net VSYNC: now also FB6.1; no longer FB6.2
- net at C27.1, U8.37 (AUXA_L): now also U8.38 (AUXA_R)
- net at C27.2: now also R2.2, C43.2, R32.1
- net DRQ0: now reaches U8.67 (DRQA)
- net DRQ0: now also J1.20 (Pin_20)
- net DACK0: now reaches J1.18 (Pin_18)
- net DACK0: now also U8.68 (~DACKBA)
- net DACK5: now reaches J1.22 (Pin_22)
- net DACK5: now also U8.62 (~DACKBD)
- net DRQ5: now reaches J1.24 (Pin_24)
- net DRQ5: now also U8.61 (DRQD)
- net IRQ10: now reaches J1.8 (Pin_8)
- net IRQ10: now also U8.71 (IRQD)
- net at R2.1: now also L5.1
- net at R24.1, R30.2: now also U10.6 (-); no longer U10.2 (-)
- net at U8.20 (PSEL0/SECS): now also R31.1
- net at U8.21 (VOLDN/SEDO): now also R35.2
- net at U8.22 (VOLUP/SEDI): now also R34.2
- net at U8.23 (MUTE/SECLK): now also R33.2
- net IRQ11: now reaches U8.70 (IRQE)
- net at U8.79 (XO): now also JP9.2 (B)
- net at C39.1, R29.1: now also U10.1; no longer U10.7
- net at R22.1, R29.2: now also U10.2 (-); no longer U10.6 (-)
- net at C40.1, R30.1: now also U10.7; no longer U10.1
- net AUXA_R renamed SPKR
- net SPKR: now also J9.16 (Pin_16)
- removed net AUXBL: JP6.3 (B), JP7.3 (B)
- removed net AUXBR: JP6.1 (A), JP7.1 (A)
- net DACK2: no longer names the net of J3.51 (Pin_51)
- net IRQ3: no longer names the net of J3.49 (Pin_49)
- net IRQ4: no longer names the net of J3.47 (Pin_47)
- net xB renamed VGA_B
- net VGA_B: now also J9.13 (Pin_13)
- net xG renamed VGA_G
- net VGA_G: now also J9.9 (Pin_9)
- net xHSYNC renamed VGA_HS
- net VGA_HS: now also FB5.2, J9.10 (Pin_10); no longer FB5.1
- net xMonitor renamed VGA_MON
- net VGA_MON: now also FB3.2, J9.8 (Pin_8); no longer FB3.1
- net xR renamed VGA_R
- net VGA_R: now also J9.5 (Pin_5)
- net xVSYNC renamed VGA_VS
- net VGA_VS: now also FB6.2, J9.14 (Pin_14); no longer FB6.1
- new net: JP8.2 (C), U8.78 (XI)
- new net: C42.2, JP8.3 (B), Y2.3
- new net: C41.2, JP9.1 (A), Y2.1
- new net: J2.2 (Pin_2), R33.1
- new net: J2.4 (Pin_4), R34.1
- new net: J2.6 (Pin_6), R35.1
- no-connect marks 77 -> 76
Other:
- note added: "PC/104"
- note added: "Sound"
- note added: "Video"
- moved on the sheet: C1, C10, C11, C12, C13, C14, C15, C16, C17, C18, C19, C2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
