File: pcb_top/rev.A/charon386_top.kicad_sch (KiCad schematic)
At the start: 137 parts, among them J1 PC104_16, J2 Vol. Btns, J3 PC104, J4 Jumper for 8-bit bus, J6 Wavetable, J7 PJ-322, J9 Conn_02x07_Odd_Even, SW1 VGA Config, U1 TVGA9000I, U10 NE5532DR, U11 74HCT138, U2 27C512PLCC, U3 MT4C4256, U4 MT4C4256, U5 MT4C4256, U6 MT4C4256, U7 AMS1117-5.0, U8 ES1868F, U9 AMS1117-5.0, Y1 40 MHz, Y2 14.318 MHz

Commit message: wip pcb rev.A
Parts:
- removed JP9: SolderJumper_2_Open, Jumper:SolderJumper-2_P1.3mm_Open_RoundedPad1.0x1.5mm, symbol Jumper:SolderJumper_2_Open
- added J5: ESP, Connector_PinSocket_2.54mm:PinSocket_2x05_P2.54mm_Vertical, symbol Connector_Generic:Conn_02x05_Odd_Even
Connections:
- net at U8.79 (XO): now also C41.2, Y2.1
- new net: J5.10 (Pin_10), J5.9 (Pin_9)
- new net: J5.3 (Pin_3), J5.4 (Pin_4)
- new net: J5.5 (Pin_5), J5.6 (Pin_6)
- new net: J5.7 (Pin_7), J5.8 (Pin_8)
- no-connect marks 76 -> 78
Changed lines of the file:
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@@
   (no_connect (at 384.81 300.99))
   (no_connect (at 386.715 45.085))
+  (no_connect (at 395.605 109.855))
+  (no_connect (at 408.305 109.855))
   (no_connect (at 434.975 278.765))
   (no_connect (at 447.675 271.145))
@@
     (stroke (width 0) (type solid) (color 0 0 0 0))
   )
-  (wire (pts (xy 336.55 290.83) (xy 339.09 290.83))
+  (wire (pts (xy 336.55 290.83) (xy 346.71 290.83))
     (stroke (width 0) (type solid) (color 0 0 0 0))
   )
@@
     (stroke (width 0) (type solid) (color 0 0 0 0))
   )
+  (wire (pts (xy 395.605 112.395) (xy 408.305 112.395))
+    (stroke (width 0) (type solid) (color 0 0 0 0))
+  )
+  (wire (pts (xy 395.605 114.935) (xy 408.305 114.935))
+    (stroke (width 0) (type solid) (color 0 0 0 0))
+  )
+  (wire (pts (xy 395.605 117.475) (xy 408.305 117.475))
+    (stroke (width 0) (type solid) (color 0 0 0 0))
+  )
+  (wire (pts (xy 395.605 120.015) (xy 408.305 120.015))
+    (stroke (width 0) (type solid) (color 0 0 0 0))
+  )
   (wire (pts (xy 395.605 160.655) (xy 389.255 160.655))
     (stroke (width 0) (type solid) (color 0 0 0 0))
@@
     (pin "8")
   )
-  (symbol (lib_id "Jumper:SolderJumper_2_Open") (at 342.9 290.83 0) (unit 1)
-    (in_bom yes) (on_board yes)
-    (property "Reference" "JP9" (id 0) (at 337.82 289.56 0)
-      (effects (font (size 1 1)))
-    )
-    (property "Value" "SolderJumper_2_Open" (id 1) (at 342.9 288.925 0)
-      (effects (font (size 1 1)) hide)
-    )
-    (property "Footprint" "Jumper:SolderJumper-2_P1.3mm_Open_RoundedPad1.0x1.5mm" (id 2) (at 342.9 290.83 0)
-      (effects (font (size 1.27 1.27)) hide)
-    )
-    (property "Datasheet" "~" (id 3) (at 342.9 290.83 0)
-      (effects (font (size 1.27 1.27)) hide)
-    )
-    (pin "1")
-    (pin "2")
-  )
   (symbol (lib_id "Device:R") (at 52.705 135.89 270) (unit 1)
     (in_bom yes) (on_board yes)
@@
   (symbol (lib_id "Device:Crystal_GND24") (at 314.325 293.37 0) (unit 1)
     (in_bom yes) (on_board yes)
-    (property "Reference" "Y2" (id 0) (at 314.325 283.21 0)
+    (property "Reference" "Y2" (id 0) (at 314.325 284.48 0)
       (effects (font (size 1 1)))
     )
-    (property "Value" "14.318 MHz" (id 1) (at 314.325 285.115 0)
+    (property "Value" "14.318 MHz" (id 1) (at 314.325 286.385 0)
       (effects (font (size 1 1)))
     )
@@
     (pin "7")
   )
+  (symbol (lib_id "Connector_Generic:Conn_02x05_Odd_Even") (at 400.685 114.935 0) (unit 1)
+    (in_bom yes) (on_board yes) (fields_autoplaced)
+    (property "Reference" "J5" (id 0) (at 401.955 104.775 0)
+      (effects (font (size 1 1)))
+    )
+    (property "Value" "ESP" (id 1) (at 401.955 107.315 0)
+      (effects (font (size 1 1)))
+    )
+    (property "Footprint" "Connector_PinSocket_2.54mm:PinSocket_2x05_P2.54mm_Vertical" (id 2) (at 400.685 114.935 0)
+      (effects (font (size 1.27 1.27)) hide)
+    )
+    (property "Datasheet" "~" (id 3) (at 400.685 114.935 0)
+      (effects (font (size 1.27 1.27)) hide)
+    )
+    (pin "1")
+    (pin "10")
+    (pin "2")
+    (pin "3")
+    (pin "4")
+    (pin "5")
+    (pin "6")
+    (pin "7")
+    (pin "8")
+    (pin "9")
+  )
   (symbol (lib_id "Connector_Generic:Conn_02x08_Odd_Even") (at 381.635 34.925 0) (mirror y) (unit 1)
     (in_bom yes) (on_board yes)
@@
       (reference "J4") (unit 1) (value "Jumper for 8-bit bus") (footprint "Connector_PinHeader_2.00mm:PinHeader_2x03_P2.00mm_Vertical")
     )
+    (path "/5864193e-4611-4978-9302-f4aedeaca05c"
+      (reference "J5") (unit 1) (value "ESP") (footprint "Connector_PinSocket_2.54mm:PinSocket_2x05_P2.54mm_Vertical")
+    )
     (path "/5d722216-118f-47f0-915a-b1df49a5981e"
       (reference "J6") (unit 1) (value "Wavetable") (footprint "Connector_PinHeader_2.54mm:PinHeader_2x13_P2.54mm_Horizontal")
@@
       (reference "JP8") (unit 1) (value "SolderJumper_3_Bridged12") (footprint "Jumper:SolderJumper-3_P1.3mm_Bridged12_RoundedPad1.0x1.5mm_NumberLabels")
     )
-    (path "/5e89eaaf-f5c9-42e1-9f0e-a773f1ef457a"
-      (reference "JP9") (unit 1) (value "SolderJumper_2_Open") (footprint "Jumper:SolderJumper-2_P1.3mm_Open_RoundedPad1.0x1.5mm")
-    )
     (path "/62e56801-3f3c-46d3-9b99-f49c6d46c42b"

Commit message: wip pcb rev.A
Parts:
- removed J6: Wavetable, Connector_PinHeader_2.54mm:PinHeader_2x13_P2.54mm_Horizontal, symbol Connector_Generic:Conn_02x13_Odd_Even
- removed JP6: WTBL. P20, Jumper:SolderJumper-3_P1.3mm_Bridged12_RoundedPad1.0x1.5mm_NumberLabels, symbol Jumper:SolderJumper_3_Bridged12
- removed JP7: WTBL. P24, Jumper:SolderJumper-3_P1.3mm_Bridged12_RoundedPad1.0x1.5mm_NumberLabels, symbol Jumper:SolderJumper_3_Bridged12
- removed JP8: SolderJumper_3_Bridged12, Jumper:SolderJumper-3_P1.3mm_Bridged12_RoundedPad1.0x1.5mm_NumberLabels, symbol Jumper:SolderJumper_3_Bridged12
- added C62, C67, C68, C71: 100n, Capacitor_SMD:C_0603_1608Metric_Pad1.08x0.95mm_HandSolder, symbol Device:C
- added C63, C69, C70: 10u, Capacitor_SMD:C_0805_2012Metric_Pad1.18x1.45mm_HandSolder, symbol Device:C
- added C64, C65: 22p, Capacitor_SMD:C_0603_1608Metric_Pad1.08x0.95mm_HandSolder, symbol Device:C
- added C66: 1u, Capacitor_SMD:C_0603_1608Metric_Pad1.08x0.95mm_HandSolder, symbol Device:C
- added LOGO1: graphic, mygraphic:black-mage-12.5x8.6, symbol my:logo
- added R36: 22, Resistor_SMD:R_0603_1608Metric_Pad0.98x0.95mm_HandSolder, symbol Device:R
- added U12: SAM2695, Package_DFN_QFN:QFN-48-1EP_6x6mm_P0.4mm_EP4.2x4.2mm, symbol my:SAM2695
- added U13: AMS1117-3.3, Package_TO_SOT_SMD:SOT-223-3_TabPin2, symbol Regulator_Linear:AMS1117-3.3
- added U14: 74HC4050, Package_SO:SO-16_3.9x9.9mm_P1.27mm, symbol 4xxx:4050
- C1, C35, C39, C40: symbol Device:CP -> Device:C_Polarized
- C41: value 10p -> 100n
- C42: value 10p -> 10u; footprint Capacitor_SMD:C_0603_1608Metric_Pad1.08x0.95mm_HandSolder -> Capacitor_SMD:C_0805_2012Metric_Pad1.18x1.45mm_HandSolder
- FB1, FB2, FB3, FB4, FB5, FB6: symbol Device:Ferrite_Bead -> Device:FerriteBead
- J4: Commend (none) -> Not on PCB
- JP1: now left out of the parts list
- R20: value 22k -> (none)
- Y2: value 14.318 MHz -> 12 MHz
Connections:
- net +5V: now also C69.2, U13.3 (VI)
- net GND: now also C62.1, C63.1, C64.1, C65.1, C66.1, C67.1, C68.1, C69.1, C70.1, C71.1, U12.10 (A0), U12.13 (GND), U12.14 (~{CS}), U12.15 (~{RD}), U12.18 (GND), U12.25 (GND), U12.36 (GND), U12.4 (AGND), U12.45 (GND), U12.48 (GND), U12.49 (GND), U12.7 (MICIN), U12.9 (GND), U13.1 (GND), U14.3, U14.5, U14.7, U14.8 (VSS), U14.9; no longer R20.2
- net IRQ11: now also J1.10 (Pin_10)
- net MCLK: no longer R20.1
- net MSO: now also U14.14
- net OSC: now also R20.2, R36.2; no longer U1.98 (ROMCLK)
- net at U8.78 (XI): now also R20.1
- net at Y2.3: now also C65.2, U12.39 (X1); no longer C42.2
- net at J5.5 (Pin_5): no longer J5.6 (Pin_6)
- net AUXB_L renamed MIDI_L
- net MIDI_L: now also U12.1 (AOUTL)
- net AUXB_R renamed MIDI_R
- net MIDI_R: now also U12.2 (AOUTR)
- net ~CAS renamed ~{CAS}
- net ~IOR renamed ~{IOR}
- net ~IOW renamed ~{IOW}
- net ~MEMCS16 renamed ~{MEMCS16}
- net ~MEMR renamed ~{MEMR}
- net ~MEMW renamed ~{MEMW}
- net ~NMI renamed ~{NMI}
- net ~RAS renamed ~{RAS}
- net ~REFRESH renamed ~{REFRESH}
- net ~ROMCS renamed ~{ROMCS}
- net ~RSTB renamed ~{RSTB}
- net ~{RSTB}: now also U14.11
- net ~SBHE renamed ~{SBHE}
- net ~WE0 renamed ~{WE0}
- net ~WE2 renamed ~{WE2}
- new net: C64.2, U12.40 (X2), Y2.1
- new net: R36.1, U1.98 (ROMCLK)
- new net: C62.2, C63.2, U12.34 (OUTVC12)
- new net: U12.16 (MIDI_IN), U14.15
- new net: U12.38 (~{RST}/~{PD}), U14.12
- new net: C41.2, C42.2, U12.5 (VCM)
- new net +3V3: C66.2, C67.2, C68.2, C70.2, C71.2, U12.11 (VD33), U12.12 (~{WR}), U12.20 (VD33), U12.31 (VD33), U12.35 (VD33), U12.41 (VD33), U12.46 (VD33), U12.47 (XDIV), U12.6 (VA33), U12.8 (VD33), U13.2 (VO), U14.1 (VCC)
- now unconnected: U8.79 (XO)
- no-connect marks 78 -> 90
Other:
- note added: "MIDI"
- moved on the sheet: C1, C19, C2, C21, C22, C23, C24, C25, C26, C27, C28, C29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

Commit message: wip pcb rev.A
Parts:
- added C51, C52: 1u, Capacitor_SMD:C_0603_1608Metric_Pad1.08x0.95mm_HandSolder, symbol Device:C
- R32: renamed from R36; value 22 -> (none); footprint Resistor_SMD:R_0603_1608Metric_Pad0.98x0.95mm_HandSolder -> (none)
- renumbered C27 to C1, C1 to C10, C2 to C11, C38 to C12, C37 to C13, C3 to C14, C39 to C15, C4 to C16, C5 to C17, C6 to C18, C7 to C19, C43 to C2, C33 to C20, C40 to C21, C13 to C22, C12 to C23, C11 to C24, C34 to C25, C17 to C26, C18 to C27, C14 to C28, C15 to C29, C29 to C3, C41 to C30, C42 to C31, C16 to C32, C62 to C33, C63 to C34, C64 to C35, C65 to C36, C20 to C37, C60 to C38, C21 to C39, C30 to C4, C22 to C40, C19 to C41, C23 to C42, C24 to C43, C69 to C44, C70 to C45, C66 to C46, C67 to C47, C68 to C48, C71 to C49, C31 to C5, C48 to C50, C61 to C53, C25 to C54, C26 to C55, C35 to C56, C36 to C57, C28 to C58, C44 to C59, C32 to C6, C45 to C60, C46 to C61, C47 to C62, C49 to C63, C50 to C64, C51 to C65, C52 to C66, C53 to C67, C54 to C68, C55 to C69, C8 to C7, C56 to C70, C57 to C71, C58 to C72, C59 to C73, C9 to C8, C10 to C9, FB4 to FB3, FB3 to FB4, J7 to J1, J9 to J3, J5 to J4, J1 to J5, J3 to J6, J4 to J7, L5 to L1, L6 to L2, L7 to L3, L9 to L4, L10 to L5, L1 to L6, L2 to L7, L3 to L8, L8 to L9, R2 to R1, R21 to R10, R22 to R11, R23 to R12, R24 to R13, R25 to R14, R26 to R15, R30 to R16, R15 to R17, R16 to R18, R9 to R19, R32 to R2, R7 to R20, R10 to R21, R11 to R22, R12 to R23, R13 to R24, R14 to R25, R33 to R26, R34 to R27, R18 to R28, R35 to R29, R4 to R3, R31 to R30, R20 to R31, R19 to R33, R8 to R34, R1 to R35, R17 to R36, R5 to R4, R6 to R5, R27 to R6, R28 to R7, R3 to R8, R29 to R9, U14 to U1, U9 to U10, U3 to U11, U4 to U12, U5 to U13, U6 to U14, U10 to U2, U11 to U3, U8 to U4, U1 to U5, U12 to U6, U2 to U7, U7 to U8, U13 to U9
Connections:
- net +5V: now also C51.1, C52.1
- net A13: now also U3.3 (A2); no longer U3.1 (A0)
- net A15: now also U3.1 (A0); no longer U3.3 (A2)
- net GND: now also C51.2, C52.2
- net at J4.5 (Pin_5): now also J4.6 (Pin_6)
- net MCLK: no longer names the net of U4.88 (MCLK)
- net MSD: no longer names the net of U4.87 (MSD)
- no-connect marks 90 -> 92
Other:
- moved on the sheet: C44, C45, C46, C47, C48, C49, C50, C63, C64, C65, C66, C67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

Commit message: wip pcb rev.A
Parts:
- removed J7: Jumper for 8-bit bus, Connector_PinHeader_2.00mm:PinHeader_2x03_P2.00mm_Vertical, symbol Connector_Generic:Conn_02x03_Odd_Even
- added R37: 4.7k, Resistor_SMD:R_0603_1608Metric_Pad0.98x0.95mm_HandSolder, symbol Device:R
- R31: value (none) -> 33
- R32: value (none) -> 33; footprint (none) -> Resistor_SMD:R_0603_1608Metric_Pad0.98x0.95mm_HandSolder
- U7: value 27C512PLCC -> 27C256
Connections:
- net +5V: now also U7.2 (A15)
- net A0: no longer U7.11 (A0)
- net A1: now also U7.11 (A0); no longer U7.10 (A1)
- net A10: now also U7.28 (A9); no longer U7.24 (A10)
- net A11: now also U7.24 (A10); no longer U7.27 (A11)
- net A12: now also U7.27 (A11); no longer U7.3 (A12)
- net A13: now also U7.3 (A12); no longer U7.30 (A13)
- net A14: now also U7.30 (A13); no longer U7.31 (A14)
- net A2: now also U7.10 (A1); no longer U7.9 (A2)
- net A3: now also U7.9 (A2); no longer U7.8 (A3)
- net A4: now also U7.8 (A3); no longer U7.7 (A4)
- net A5: now also U7.7 (A4); no longer U7.6 (A5)
- net A6: now also U7.6 (A5); no longer U7.5 (A6)
- net A7: now also U7.5 (A6); no longer U7.4 (A7)
- net A8: now also U7.4 (A7); no longer U7.29 (A8)
- net A9: now also U7.29 (A8); no longer U7.28 (A9)
- net GND: now also R37.1
- net RMD5: now also R37.2
- net ROMA0 renamed ROMBA0
- net ROMBA0: now also U7.31 (A14); no longer U7.2 (A15)
Other:
- moved on the sheet: R19, R21, R22, R23, R24, R25, SW1
