File: pcb_top/rev.A/charon386_top.kicad_sch (KiCad schematic)
At the start: 150 parts, among them J1 PJ-322, J2 Vol. Btns, J3 Conn_02x07_Odd_Even, J4 ESP, J5 PC104_16, J6 PC104, SW1 VGA Config, U1 74HC4050, U10 AMS1117-5.0, U11 MT4C4256, U12 MT4C4256, U13 MT4C4256, U14 MT4C4256, U2 NE5532DR, U3 74HCT138, U4 ES1868F, U5 TVGA9000I, U6 SAM2695, U7 27C256, U8 AMS1117-5.0, U9 AMS1117-3.3, Y1 40 MHz, Y2 12 MHz

Commit message: wip pcb rev.A
Parts:
- added C74: 100u, Capacitor_Tantalum_SMD:CP_EIA-7343-31_Kemet-D_Pad2.25x2.55mm_HandSolder, symbol Device:C_Polarized
Connections:
- net +5V: now also C74.1
- net GND: now also C74.2
Other:
- note added: "18mA"
- note added: "195ma"
- note added: "20mA"
- note added: "90mA"
Changed lines of the file:
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@@
   (junction (at 529.59 276.86) (diameter 0) (color 0 0 0 0)
   )
+  (junction (at 570.23 269.24) (diameter 0) (color 0 0 0 0)
+  )
+  (junction (at 570.23 276.86) (diameter 0) (color 0 0 0 0)
+  )
   (junction (at 466.725 73.66) (diameter 1.016) (color 0 0 0 0)
   )
@@
     (stroke (width 0) (type solid) (color 0 0 0 0))
   )
+  (wire (pts (xy 570.23 276.86) (xy 576.58 276.86))
+    (stroke (width 0) (type default) (color 0 0 0 0))
+  )
   (wire (pts (xy 298.45 125.73) (xy 288.29 125.73))
     (stroke (width 0) (type solid) (color 0 0 0 0))
@@
     (stroke (width 0) (type solid) (color 0 0 0 0))
   )
+  (wire (pts (xy 570.23 269.24) (xy 576.58 269.24))
+    (stroke (width 0) (type default) (color 0 0 0 0))
+  )
   (wire (pts (xy 427.355 292.735) (xy 455.93 292.735))
     (stroke (width 0) (type solid) (color 0 0 0 0))
@@
     (effects (font (size 1.524 1.524)) (justify left bottom))
   )
+  (text "90mA" (at 234.95 271.145 0)
+    (effects (font (size 1 1) italic) (justify left bottom))
+  )
+  (text "18mA" (at 494.03 137.16 0)
+    (effects (font (size 1 1) italic) (justify left bottom))
+  )
+  (text "195ma" (at 115.57 36.195 0)
+    (effects (font (size 1 1) italic) (justify left bottom))
+  )
   (text "Sound" (at 291.465 21.59 180)
     (effects (font (size 2 2) italic) (justify right bottom))
@@
     (effects (font (size 2 2) italic) (justify right bottom))
   )
+  (text "90mA" (at 115.57 271.145 0)
+    (effects (font (size 1 1) italic) (justify left bottom))
+  )
+  (text "90mA" (at 55.88 271.145 0)
+    (effects (font (size 1 1) italic) (justify left bottom))
+  )
   (text "MIDI" (at 426.72 133.35 0)
     (effects (font (size 2.0066 2.0066) italic) (justify left bottom))
   )
+  (text "20mA" (at 224.79 176.53 0)
+    (effects (font (size 1 1) italic) (justify left bottom))
+  )
+  (text "90mA" (at 175.26 271.145 0)
+    (effects (font (size 1 1) italic) (justify left bottom))
+  )
   (text "PC/104" (at 294.005 228.6 180)
     (effects (font (size 2 2) italic) (justify right bottom))
@@
     (pin "8")
   )
+  (symbol (lib_id "Device:C_Polarized") (at 576.58 273.05 0) (unit 1)
+    (in_bom yes) (on_board yes)
+    (property "Reference" "C74" (id 0) (at 579.12 270.51 0)
+      (effects (font (size 1 1)))
+    )
+    (property "Value" "100u" (id 1) (at 579.12 275.59 0)
+      (effects (font (size 1 1)))
+    )
+    (property "Footprint" "Capacitor_Tantalum_SMD:CP_EIA-7343-31_Kemet-D_Pad2.25x2.55mm_HandSolder" (id 2) (at 577.5452 276.86 0)
+      (effects (font (size 1.27 1.27)) hide)
+    )
+    (property "Datasheet" "~" (id 3) (at 576.58 273.05 0)
+      (effects (font (size 1.27 1.27)) hide)
+    )
+    (pin "1")
+    (pin "2")
+  )
   (symbol (lib_id "Device:R") (at 346.71 161.29 270) (mirror x) (unit 1)
     (in_bom yes) (on_board yes)
@@
       (reference "C73") (unit 1) (value "100n") (footprint "Capacitor_SMD:C_0603_1608Metric_Pad1.08x0.95mm_HandSolder")
     )
+    (path "/b3b87e50-76ab-48dc-93ed-f701c9ec9a10"
+      (reference "C74") (unit 1) (value "100u") (footprint "Capacitor_Tantalum_SMD:CP_EIA-7343-31_Kemet-D_Pad2.25x2.55mm_HandSolder")
+    )
     (path "/be9d8049-8188-4521-8acb-172c35d5ac92"

Commit message: wip pcb rev.A
Changed lines of the file:
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@@
     (stroke (width 0) (type solid) (color 0 0 0 0))
   )
-  (wire (pts (xy 99.06 309.245) (xy 88.9 309.245))
-    (stroke (width 0) (type solid) (color 0 0 0 0))
-  )
   (wire (pts (xy 516.89 184.15) (xy 516.89 190.5))
     (stroke (width 0) (type solid) (color 0 0 0 0))
@@
     (stroke (width 0) (type solid) (color 0 0 0 0))
   )
-  (wire (pts (xy 39.37 309.245) (xy 29.21 309.245))
-    (stroke (width 0) (type solid) (color 0 0 0 0))
-  )
   (wire (pts (xy 111.125 31.75) (xy 111.125 35.56))
     (stroke (width 0) (type solid) (color 0 0 0 0))
@@
     (stroke (width 0) (type solid) (color 0 0 0 0))
   )
-  (wire (pts (xy 218.44 309.245) (xy 208.28 309.245))
-    (stroke (width 0) (type solid) (color 0 0 0 0))
-  )
   (wire (pts (xy 59.055 158.75) (xy 69.215 158.75))
     (stroke (width 0) (type solid) (color 0 0 0 0))
@@
     (stroke (width 0) (type solid) (color 0 0 0 0))
   )
-  (wire (pts (xy 158.75 309.245) (xy 148.59 309.245))
-    (stroke (width 0) (type solid) (color 0 0 0 0))
-  )
   (wire (pts (xy 59.055 133.35) (xy 69.215 133.35))
     (stroke (width 0) (type solid) (color 0 0 0 0))
@@
     (effects (font (size 1 1)) (justify left bottom))
   )
-  (label "GND" (at 148.59 309.245 0)
-    (effects (font (size 1 1)) (justify left bottom))
-  )
   (label "D6" (at 289.56 245.745 0)
     (effects (font (size 1 1)) (justify left bottom))
@@
     (effects (font (size 1 1)) (justify left bottom))
   )
-  (label "GND" (at 208.28 309.245 0)
-    (effects (font (size 1 1)) (justify left bottom))
-  )
   (label "DRQ0" (at 368.3 263.525 0)
     (effects (font (size 1 1)) (justify left bottom))
   )
-  (label "GND" (at 29.21 309.245 0)
-    (effects (font (size 1 1)) (justify left bottom))
-  )
   (label "~{WE0}" (at 29.21 311.785 0)
     (effects (font (size 1 1)) (justify left bottom))
@@
     (effects (font (size 1 1)) (justify left bottom))
   )
-  (label "GND" (at 88.9 309.245 0)
-    (effects (font (size 1 1)) (justify left bottom))
-  )
   (label "MAB7" (at 208.28 296.545 0)
     (effects (font (size 1 1)) (justify left bottom))
@@
     (effects (font (size 1 1)) (justify left bottom))
   )
+  (symbol (lib_id "power:GND") (at 99.06 309.245 270) (unit 1)
+    (in_bom yes) (on_board yes)
+    (property "Reference" "#PWR?" (id 0) (at 92.71 309.245 0)
+      (effects (font (size 1 1)) hide)
+    )
+    (property "Value" "GND" (id 1) (at 93.98 309.245 90)
+      (effects (font (size 1 1)))
+    )
+    (property "Footprint" "" (id 2) (at 99.06 309.245 0)
+      (effects (font (size 1.27 1.27)) hide)
+    )
+    (property "Datasheet" "" (id 3) (at 99.06 309.245 0)
+      (effects (font (size 1.27 1.27)) hide)
+    )
+    (pin "1")
+  )
   (symbol (lib_id "power:GND") (at 558.8 276.86 0) (unit 1)
     (in_bom yes) (on_board yes)
@@
     (pin "1")
   )
+  (symbol (lib_id "power:GND") (at 39.37 309.245 270) (unit 1)
+    (in_bom yes) (on_board yes)
+    (property "Reference" "#PWR?" (id 0) (at 33.02 309.245 0)
+      (effects (font (size 1 1)) hide)
+    )
+    (property "Value" "GND" (id 1) (at 34.29 309.245 90)
+      (effects (font (size 1 1)))
+    )
+    (property "Footprint" "" (id 2) (at 39.37 309.245 0)
+      (effects (font (size 1.27 1.27)) hide)
+    )
+    (property "Datasheet" "" (id 3) (at 39.37 309.245 0)
+      (effects (font (size 1.27 1.27)) hide)
+    )
+    (pin "1")
+  )
   (symbol (lib_id "power:GNDA") (at 436.88 121.285 0) (unit 1)
     (in_bom yes) (on_board yes)
@@
     (pin "2")
   )
+  (symbol (lib_id "power:GND") (at 158.75 309.245 270) (unit 1)
+    (in_bom yes) (on_board yes)
+    (property "Reference" "#PWR?" (id 0) (at 152.4 309.245 0)
+      (effects (font (size 1 1)) hide)
+    )
+    (property "Value" "GND" (id 1) (at 153.67 309.245 90)
+      (effects (font (size 1 1)))
+    )
+    (property "Footprint" "" (id 2) (at 158.75 309.245 0)
+      (effects (font (size 1.27 1.27)) hide)
+    )
+    (property "Datasheet" "" (id 3) (at 158.75 309.245 0)
+      (effects (font (size 1.27 1.27)) hide)
+    )
+    (pin "1")
+  )
   (symbol (lib_id "Device:C") (at 535.94 296.545 0) (unit 1)
     (in_bom yes) (on_board yes)
@@
     (pin "1")
   )
+  (symbol (lib_id "power:GND") (at 218.44 309.245 270) (unit 1)
+    (in_bom yes) (on_board yes)
+    (property "Reference" "#PWR?" (id 0) (at 212.09 309.245 0)
+      (effects (font (size 1 1)) hide)
+    )
+    (property "Value" "GND" (id 1) (at 213.36 309.245 90)
+      (effects (font (size 1 1)))
+    )
+    (property "Footprint" "" (id 2) (at 218.44 309.245 0)
+      (effects (font (size 1.27 1.27)) hide)
+    )
+    (property "Datasheet" "" (id 3) (at 218.44 309.245 0)
+      (effects (font (size 1.27 1.27)) hide)
+    )
+    (pin "1")
+  )
   (symbol (lib_id "Device:R") (at 236.22 155.575 270) (unit 1)
     (in_bom yes) (on_board yes)
@@
       (reference "#PWR0101") (unit 1) (value "+5V") (footprint "")
     )
+    (path "/0061ae4e-fa6d-4e91-ae74-20d4a542b864"
+      (reference "#PWR?") (unit 1) (value "GND") (footprint "")
+    )
+    (path "/06a4de1e-e0ab-4c45-8360-850367dc2e5b"
+      (reference "#PWR?") (unit 1) (value "GND") (footprint "")
+    )
+    (path "/910c78b1-da80-4349-80d8-c98d670eaa86"
+      (reference "#PWR?") (unit 1) (value "GND") (footprint "")
+    )
+    (path "/ae99a7fb-75ff-4fc6-af63-135b09882e4f"
+      (reference "#PWR?") (unit 1) (value "GND") (footprint "")
+    )
     (path "/02f26204-fab3-4a0e-8b7a-c91ae77181bf"

Commit message: wip pcb rev.A
Other:
- company: (none) -> Eugene Lozovoy
- title: (none) -> PC-CHARON-386-TOP
Changed lines of the file:
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@@
   (paper "User" 599.999 350.012)
   (title_block
+    (title "PC-CHARON-386-TOP")
     (date "2021-12-17")
     (rev "A")
+    (company "Eugene Lozovoy")
+    (comment 1 "VGA & Sound board for Charon-386")
   )
   (junction (at 465.455 292.735) (diameter 1.016) (color 0 0 0 0)

Commit message: wip pcb rev.A (almost done now)
Parts:
- SW1: footprint Button_Switch_THT:SW_DIP_SPSTx02_Slide_9.78x7.26mm_W7.62mm_P2.54mm -> Button_Switch_THT:SW_DIP_SPSTx02_Slide_6.7x6.64mm_W7.62mm_P2.54mm_LowProfile
Changed lines of the file:
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@@
       (effects (font (size 1 1)))
     )
-    (property "Footprint" "Button_Switch_THT:SW_DIP_SPSTx02_Slide_9.78x7.26mm_W7.62mm_P2.54mm" (id 2) (at 214.63 147.955 0)
+    (property "Footprint" "Button_Switch_THT:SW_DIP_SPSTx02_Slide_6.7x6.64mm_W7.62mm_P2.54mm_LowProfile" (id 2) (at 214.63 147.955 0)
       (effects (font (size 1.27 1.27)) hide)
     )
@@
     )
     (path "/46d8c6f2-9c28-4bc8-bf83-68eb4225e4b8"
-      (reference "SW1") (unit 1) (value "VGA Config") (footprint "Button_Switch_THT:SW_DIP_SPSTx02_Slide_9.78x7.26mm_W7.62mm_P2.54mm")
+      (reference "SW1") (unit 1) (value "VGA Config") (footprint "Button_Switch_THT:SW_DIP_SPSTx02_Slide_6.7x6.64mm_W7.62mm_P2.54mm_LowProfile")
     )
     (path "/e9bb9582-e2bc-46cd-b4a2-96539521344a"

Commit message: wip pcb rev.A
Parts:
- removed C39, C42, C45, C54: 10u, Capacitor_SMD:C_0805_2012Metric_Pad1.18x1.45mm_HandSolder, symbol Device:C
- removed C40, C49: 100n, Capacitor_SMD:C_0603_1608Metric_Pad1.08x0.95mm_HandSolder, symbol Device:C
- removed U1: 74HC4050, Package_SO:SO-16_3.9x9.9mm_P1.27mm, symbol 4xxx:4050
- removed U10: AMS1117-5.0, Package_TO_SOT_SMD:SOT-223-3_TabPin2, symbol Regulator_Linear:AMS1117-5.0
- added C39, C40, C42, C45, C49: 10u, Capacitor_Tantalum_SMD:CP_EIA-3216-18_Kemet-A_Pad1.58x1.35mm_HandSolder, symbol Device:CP
- added L10: 5.7u, Inductor_SMD:L_1210_3225Metric_Pad1.42x2.65mm_HandSolder, symbol Device:L
- added R38, R40, R41: 0, Resistor_SMD:R_0805_2012Metric_Pad1.20x1.40mm_HandSolder, symbol Device:R
- added U1: 1117-5.0, Package_TO_SOT_SMD:SOT-223-3_TabPin2, symbol Regulator_Linear:AMS1117-5.0
- U8: value AMS1117-5.0 -> 1117-5.0
- U9: value AMS1117-3.3 -> 1117-3.3
Connections:
- net +12V: now also R41.1, U1.3 (VI); no longer L9.1
- net +3V3: now also C45.1
- net +5V: now also L10.1, R38.1, R40.1
- net AVDD1: now also C39.1
- net AVDD2: now also C42.1
- net AVDD_ES: now also U8.2 (VO), C49.1, L10.2
- net GND: now also C39.2, C40.2, C42.2, C45.2, C49.2, U1.1 (GND)
- net MSO: now also U6.16 (MIDI_IN)
- net ~{RSTB}: now also U6.38 (~{RST}/~{PD})
- net at L7.1, L8.1: now also C40.1, R38.2, U1.2 (VO); no longer U8.2 (VO)
- new net: L9.1, R40.2, R41.2
- no-connect marks 92 -> 88
Other:
- moved on the sheet: C1, C10, C11, C12, C13, C14, C15, C16, C17, C18, C19, C2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

Commit message: wip pcb rev.A
Changed lines of the file:
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@@
   (symbol (lib_id "Device:R") (at 153.67 139.7 90) (unit 1)
     (in_bom yes) (on_board yes)
-    (property "Reference" "R20" (id 0) (at 157.48 138.4258 90)
+    (property "Reference" "R20" (id 0) (at 158.115 138.43 90)
       (effects (font (size 1 1)))
     )
