File: pcb_top/rev.A/kharon386_top.kicad_sch (KiCad schematic)
At the start: 153 parts, among them J1 PJ-322, J2 Vol. Btns, J3 Conn_02x07_Odd_Even, J4 ESP, J5 PC104_16, J6 PC104, SW1 VGA Config, U1 1117-5.0, U11 MT4C4256, U12 MT4C4256, U13 MT4C4256, U14 MT4C4256, U2 NE5532DR, U3 74HCT138, U4 ES1868F, U5 TVGA9000I, U6 SAM2695, U7 27C256, U8 1117-5.0, U9 1117-3.3, Y1 40 MHz, Y2 12 MHz

Commit message: wip pcb rev.A
Parts:
- C39, C40, C42, C45, C49: symbol Device:CP -> Device:C_Polarized
Changed lines of the file:
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@@
     (pin "2")
   )
-  (symbol (lib_id "Device:CP") (at 466.725 250.19 0) (unit 1)
+  (symbol (lib_id "Device:C_Polarized") (at 466.725 250.19 0) (unit 1)
     (in_bom yes) (on_board yes)
     (property "Reference" "C42" (id 0) (at 468.63 248.285 0)
@@
     (pin "1")
   )
-  (symbol (lib_id "Device:CP") (at 440.055 232.41 0) (unit 1)
+  (symbol (lib_id "Device:C_Polarized") (at 440.055 232.41 0) (unit 1)
     (in_bom yes) (on_board yes)
     (property "Reference" "C40" (id 0) (at 441.96 230.505 0)
@@
     (pin "1")
   )
-  (symbol (lib_id "Device:CP") (at 466.725 269.875 0) (unit 1)
+  (symbol (lib_id "Device:C_Polarized") (at 466.725 269.875 0) (unit 1)
     (in_bom yes) (on_board yes)
     (property "Reference" "C49" (id 0) (at 468.63 267.97 0)
@@
     (pin "1")
   )
-  (symbol (lib_id "Device:CP") (at 442.595 313.055 0) (unit 1)
+  (symbol (lib_id "Device:C_Polarized") (at 442.595 313.055 0) (unit 1)
     (in_bom yes) (on_board yes)
     (property "Reference" "C45" (id 0) (at 444.5 311.15 0)
@@
     (pin "9")
   )
-  (symbol (lib_id "Device:CP") (at 466.725 232.41 0) (unit 1)
+  (symbol (lib_id "Device:C_Polarized") (at 466.725 232.41 0) (unit 1)
     (in_bom yes) (on_board yes)
     (property "Reference" "C39" (id 0) (at 468.63 230.505 0)

Commit message: wip pcb rev.A
Other:
- moved on the sheet: C41, J5, J6, R35, R36

Commit message: wip pcb rev.A
Parts:
- removed R28: 100, Resistor_SMD:R_0603_1608Metric_Pad0.98x0.95mm_HandSolder, symbol Device:R
- L10, L7, L8, L9: value 5.7u -> 5.6u
- R20: value 1k -> 100
- R35: value 4.7k -> 10k
- R37: Desc (none) -> Do not install; now left out of the parts list
- U3: value 74HCT138 -> 74HCT138PW
Connections:
- net Monitor: now also R8.2
- net RESET: now also C41.2
- net VGA_MON: no longer R8.2
- net ~{MEMR}: now also C29.1, U5.155 (~{MEMR})
- net at J6.3 (Pin_3), R36.1: no longer C41.2
Other:
- moved on the sheet: C32, C37, C41, J2, JP1, L6, R26, R27, R29, R32, R34, R36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

Commit message: pcb rev.A final version
Parts:
- J1: value PJ-322 -> PJ-320; footprint my:PJ-322 -> my:PJ-320A_D
Changed lines of the file:
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@@
   (symbol (lib_id "Connector:AudioJack4") (at 445.135 55.245 0) (mirror y) (unit 1)
     (in_bom yes) (on_board yes)
-    (property "Reference" "J1" (id 0) (at 445.135 48.26 0)
+    (property "Reference" "J1" (id 0) (at 445.77 48.26 0)
       (effects (font (size 1 1)) (justify right))
     )
-    (property "Value" "PJ-322" (id 1) (at 443.992 49.9364 0)
+    (property "Value" "PJ-320" (id 1) (at 443.992 49.9364 0)
       (effects (font (size 1 1)) (justify right))
     )
-    (property "Footprint" "my:PJ-322" (id 2) (at 445.135 55.245 0)
+    (property "Footprint" "my:PJ-320A_D" (id 2) (at 445.135 55.245 0)
       (effects (font (size 1.27 1.27)) hide)
     )
@@
     )
     (path "/98c1acbb-1c3c-4a60-b114-138db59223a0"
-      (reference "J1") (unit 1) (value "PJ-322") (footprint "my:PJ-322")
+      (reference "J1") (unit 1) (value "PJ-320") (footprint "my:PJ-320A_D")
     )
     (path "/edccd893-c86e-4acc-b4ad-6efa06b3e275"
