File: pcb_main/rev.A/charon386_main.kicad_pcb (KiCad board)
At the start: 2 copper layers, 100 x 100 mm, 86 parts, among them CON1 CF-CARD-cfcard, J1 Mini-DIN-6, J10 COM2, J11 ESP, J2 AudioJack3, J3 USB_B_Micro, J4 Mini-DIN-6, J5 DB15_Female_HighDensity_Mount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, J6 Conn_01x04, J7 PC104_16, J8 PC104, J9 COM1, Q1 BC817, SW1 SW_Push, SW2 Jumper / Pin header 1x2 Pitch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, U1 CH340G, U10 LT1930, U11 TXB0104PW, U12 XC9572XL-VQ64, U2 ESP-12E, U3 MSM5118160F-JS, U4 MSM5118160F-JS, U5 M6117D, U6 GD75232DB, U7 SST39SF040, U8 GD75232DB, U9 AMS1117-3.3, X1 50 MHz, Y1 12 MHz, Y2 32768 Hz

Commit message: wip pcb rev.A
Parts:
- removed C8: 10u, Capacitor_SMD:C_0805_2012Metric_Pad1.18x1.45mm_HandSolder
- added D6: LED_Blue, LED_THT:LED_D3.0mm_Horizontal_O1.27mm_Z6.0mm, F.Cu at (108.8, 141.9)
- added J12: Conn_02x07_Odd_Even, Connector_PinSocket_2.54mm:PinSocket_2x07_P2.54mm_Vertical, F.Cu at (142.5, 58.5)
- added Q2: BC856, Package_TO_SOT_SMD:SOT-23, B.Cu at (108.4, 144.7)
- added R18: 470, Resistor_SMD:R_0603_1608Metric_Pad0.98x0.95mm_HandSolder, B.Cu at (111.2, 144.8)
- added R5: 0, Resistor_SMD:R_0805_2012Metric_Pad1.20x1.40mm_HandSolder, B.Cu at (158.8, 52.7)
- added U13: ST16C554, Package_QFP:LQFP-64_10x10mm_P0.5mm, F.Cu at (124.1, 106.1)
- added U14: 74LS32, Package_SO:TSSOP-14_4.4x5mm_P0.65mm, F.Cu at (145.5, 103.6)
- added U15: 74HCT138, Package_SO:TSSOP-16_4.4x5mm_P0.65mm, F.Cu at (134.3, 103.6)
- added U16: 74HCT138, Package_SO:TSSOP-16_4.4x5mm_P0.65mm, F.Cu at (139.9, 103.6)
- added X2: 14.7456 MHz, Oscillator:Oscillator_SMD_SeikoEpson_SG8002CA-4Pin_7.0x5.0mm, F.Cu at (128.4, 117.8)
- added X3: 80 MHz, Oscillator:Oscillator_SMD_SeikoEpson_SG8002CA-4Pin_7.0x5.0mm, F.Cu at (135.1, 64.7)
- C2, C3, C6, C7, R4, R8, RN1, RN2, RN3, RN4, RN5, RN6, RN7, RN8: moved to B.Cu
- D1: value LED -> LED_Red
- D2: value LED -> LED_Green
- J1, J4: footprint 4x1md:Connector_Mini-DIN_Female_6Pin_2rows -> my:MINI_DIN_6_33PRIMARY
- J2: value AudioJack3 -> PJ-320; footprint Connector_Audio:Jack_3.5mm_CUI_SJ1-3535NG_Horizontal -> my:PJ-322
- U12: value XC9572XL-VQ64 -> MAX823LEUK; footprint Package_QFP:TQFP-64_10x10mm_P0.5mm -> Package_TO_SOT_SMD:SOT-23-5; moved to B.Cu
- U6, U8: value GD75232DB -> GD75232PW; footprint Package_SO:SSOP-20_4.4x6.5mm_P0.65mm -> Package_SO:TSSOP-20_4.4x6.5mm_P0.65mm
- U7: value SST39SF040 -> 27C512PLCC
- X1: value 50 MHz -> 14.318 MHz
- moved R8 97.9 mm to (145.2, 81.1), turned to 180 degrees
- moved C3 89.9 mm to (145.4, 114.0), turned to 180 degrees
- moved Y1 85.8 mm to (145.4, 112.6), turned to -90 degrees
- moved Y2 83.2 mm to (151.7, 100.1)
- moved C7 83.0 mm to (153.6, 104.1), turned to -90 degrees
- moved R4 82.1 mm to (152.7, 101.6)
- moved C2 81.7 mm to (145.4, 111.1), turned to 0 degrees
- moved C6 81.3 mm to (151.8, 104.1), turned to -90 degrees
- moved RN7 78.4 mm to (156.5, 95.5), turned to -90 degrees
- moved U1 78.1 mm to (137.9, 112.6), turned to 90 degrees
- moved C1 76.9 mm to (137.3, 113.1), turned to -90 degrees
- moved RN1 71.6 mm to (168.4, 95.5), turned to 90 degrees
- moved C4 69.3 mm to (133.5, 111.8), turned to -90 degrees
- moved RN6 68.3 mm to (165.6, 71.2), turned to 90 degrees
- moved RN2 66.5 mm to (164.5, 95.5), turned to 90 degrees
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Connections:
- net Net-(U2-Pad21) renamed /ESP_RX
- net Net-(U2-Pad22) renamed /ESP_TX
- net Net-(U2-Pad4) renamed /ESP_RTS
- net Net-(U2-Pad7) renamed /ESP_CTS
- J1 pad 2: (no net) -> unconnected-(J1-Pad2)
- J1 pad 6: (no net) -> unconnected-(J1-Pad6)
- J10 pad 1: (no net) -> /DCD2
- J10 pad 2: (no net) -> /RX2
- J10 pad 3: (no net) -> /TX2
- J10 pad 4: (no net) -> /DTR2
- J10 pad 5: (no net) -> GND
- J10 pad 6: (no net) -> /DSR2
- J10 pad 7: (no net) -> /RTS2
- J10 pad 8: (no net) -> /CTS2
- J10 pad 9: (no net) -> /RI2
- J11 pad 10: Net-(U11-Pad5) -> /CTSD
- J11 pad 4: Net-(U11-Pad2) -> Net-(J11-Pad4)
- J11 pad 6: Net-(U11-Pad3) -> Net-(J11-Pad6)
- J11 pad 8: Net-(U11-Pad4) -> Net-(J11-Pad8)
- J2 pad S: GND -> Net-(J12-Pad6)
- J2 pad T: (no net) -> /SND_L
- J4 pad 2: (no net) -> unconnected-(J4-Pad2)
- J4 pad 6: (no net) -> unconnected-(J4-Pad6)
- J5 pad 1: (no net) -> /VGA_R
- J5 pad 12: (no net) -> /VGA_MON
- J5 pad 13: (no net) -> /VGA_HS
- J5 pad 14: (no net) -> /VGA_VS
- J5 pad 2: (no net) -> /VGA_G
- J5 pad 3: (no net) -> /VGA_B
- J5 pad 9: GND -> Net-(J5-Pad9)
- J7 pad 10: (no net) -> /IRQ11
- J7 pad 14: (no net) -> /IRQ15
- J7 pad 16: (no net) -> /IRQ14
- J7 pad 18: (no net) -> /DACK0
- J7 pad 19: (no net) -> /MEMR
- J7 pad 20: (no net) -> /DRQ0
- J7 pad 21: (no net) -> /MEMW
- J7 pad 22: (no net) -> /DACK5
- J7 pad 23: (no net) -> /SD8
- J7 pad 24: (no net) -> /DRQ5
- J7 pad 25: (no net) -> /SD9
- J7 pad 26: (no net) -> /DACK6
- J7 pad 27: (no net) -> /SD10
- J7 pad 28: (no net) -> /DRQ6
- J7 pad 29: (no net) -> /SD11
- J7 pad 3: (no net) -> /SBHE
- J7 pad 30: (no net) -> /DACK7
- J7 pad 31: (no net) -> /SD12
- J7 pad 32: (no net) -> /DRQ7
- J7 pad 33: (no net) -> /SD13
- J7 pad 35: (no net) -> /SD14
- J7 pad 36: (no net) -> /MASTER
- J7 pad 37: (no net) -> /SD15
- J7 pad 4: (no net) -> /MEMCS16
- J7 pad 6: (no net) -> /IOCS16
- J7 pad 8: (no net) -> /IRQ10
- J8 pad 10: (no net) -> /SD4
- J8 pad 11: (no net) -> /DRQ2
- J8 pad 12: (no net) -> /SD3
- J8 pad 14: (no net) -> /SD2
- J8 pad 15: (no net) -> /NOWS
- J8 pad 16: (no net) -> /SD1
- J8 pad 18: (no net) -> /SD0
- J8 pad 2: (no net) -> /IOCHCK
- J8 pad 21: (no net) -> /SMEMW
- J8 pad 23: (no net) -> /SMEMR
- J8 pad 24: (no net) -> /SA19
- J8 pad 25: (no net) -> /IOW
- J8 pad 26: (no net) -> /SA18
- J8 pad 27: (no net) -> /IOR
- J8 pad 28: (no net) -> /SA17
- J8 pad 29: (no net) -> /DACK3
- J8 pad 3: (no net) -> /RSTDRV
- J8 pad 30: (no net) -> /SA16
- J8 pad 31: (no net) -> /DRQ3
- J8 pad 32: (no net) -> /SA15
- J8 pad 33: (no net) -> /DACK1
- J8 pad 34: (no net) -> /SA14
- J8 pad 35: (no net) -> /DRQ1
- J8 pad 36: (no net) -> /SA13
- J8 pad 37: (no net) -> /REFRESH
- J8 pad 38: (no net) -> /SA12
- J8 pad 39: (no net) -> /SYSCLK
- J8 pad 4: (no net) -> /SD7
- J8 pad 40: (no net) -> /SA11
- J8 pad 41: (no net) -> /IRQ7
- J8 pad 42: (no net) -> /SA10
- J8 pad 43: (no net) -> /IRQ6
- J8 pad 44: (no net) -> /SA9
- J8 pad 45: (no net) -> /IRQ5
- J8 pad 46: (no net) -> /SA8
- J8 pad 47: (no net) -> /IRQ4
- J8 pad 48: (no net) -> /SA7
- J8 pad 49: (no net) -> /IRQ3
- J8 pad 50: (no net) -> /SA6
- J8 pad 51: (no net) -> /DACK2
- J8 pad 52: (no net) -> /SA5
- J8 pad 53: (no net) -> /TC
- J8 pad 54: (no net) -> /SA4
- J8 pad 55: (no net) -> /BALE
- J8 pad 56: (no net) -> /SA3
- J8 pad 58: (no net) -> /SA2
- J8 pad 59: (no net) -> /14MHz
- J8 pad 6: (no net) -> /SD6
- J8 pad 60: (no net) -> /SA1
- J8 pad 62: (no net) -> /SA0
- J8 pad 7: (no net) -> /IRQ9
- J8 pad 8: (no net) -> /SD5
- J9 pad 1: (no net) -> /DCD1
- J9 pad 2: (no net) -> /RX1
- J9 pad 3: (no net) -> /TX1
- J9 pad 4: (no net) -> /DTR1
- J9 pad 5: (no net) -> GND
- J9 pad 6: (no net) -> /DSR1
- J9 pad 7: (no net) -> /RTS1
- J9 pad 8: (no net) -> /CTS1
- J9 pad 9: (no net) -> /RI1
- R10 pad 2: /~RST -> Net-(R10-Pad2)
- R12 pad 1: Net-(D1-Pad2) -> +5V
- R12 pad 2: +5V -> Net-(D1-Pad2)
- R13 pad 1: Net-(D2-Pad2) -> +5V
- R13 pad 2: +5V -> Net-(D2-Pad2)
- RN4 pad 3: /OWS -> /NOWS
- RN7 pad 8: (no net) -> /KBSJ
- RN8 pad 4: /MASTER -> /IOR
- SW1 pad 1: /~RST -> Net-(R10-Pad2)
- U1 pad 10: (no net) -> /DTRC
- U1 pad 11: (no net) -> +5V
- U1 pad 12: (no net) -> /DTRC
- U1 pad 13: (no net) -> /DSRC
- U1 pad 14: (no net) -> /CTSC
- U1 pad 2: (no net) -> /RXC
- U1 pad 3: (no net) -> /TXC
- U1 pad 9: (no net) -> /RTSC
- U11 pad 10: (no net) -> /RTSD
- U11 pad 11: (no net) -> /TXD
- U11 pad 12: (no net) -> /RXD
- U11 pad 13: (no net) -> /RESETL
- U11 pad 2: Net-(U11-Pad2) -> /ESP_RST
- U11 pad 3: Net-(U11-Pad3) -> Net-(J11-Pad4)
- U11 pad 4: Net-(U11-Pad4) -> Net-(J11-Pad6)
- U11 pad 5: Net-(U11-Pad5) -> Net-(J11-Pad8)
- U12 pad 1: (no net) -> /PWG
- U12 pad 2: (no net) -> GND
- U12 pad 3: +3V3 -> Net-(R10-Pad2)
- U12 pad 5: (no net) -> +5V
- U2 pad 1: (no net) -> /ESP_RST
- U5 pad 113: (no net) -> /PWG
- U5 pad 117: (no net) -> /14MHz
- U5 pad 146: (no net) -> /IRQ9
- U5 pad 147: (no net) -> /IRQ7
- U5 pad 148: (no net) -> /IRQ6
- U5 pad 149: (no net) -> /IRQ5
- U5 pad 151: (no net) -> /IRQ4
- U5 pad 152: (no net) -> /IRQ3
- U5 pad 153: (no net) -> /IRQ10
- U5 pad 154: (no net) -> /IRQ11
- U5 pad 159: (no net) -> /IRQ15
- U5 pad 160: (no net) -> /SYSCLK
- U5 pad 162: (no net) -> /RSTDRV
- U5 pad 165: /OWS -> /NOWS
- U5 pad 17: (no net) -> /DRQ0
- U5 pad 173: (no net) -> /BALE
- U5 pad 174: (no net) -> /SA19
- U5 pad 175: (no net) -> /SA18
- U5 pad 176: (no net) -> /SA17
- U5 pad 177: (no net) -> /SA16
- U5 pad 19: (no net) -> /DRQ1
- U5 pad 196: (no net) -> /IOCHCK
- U5 pad 20: (no net) -> /DACK2
- U5 pad 200: (no net) -> /SBHE
- U5 pad 21: (no net) -> /DRQ2
- U5 pad 22: (no net) -> /DACK3
- U5 pad 23: (no net) -> /DRQ3
- U5 pad 25: (no net) -> /DRQ5
- U5 pad 26: (no net) -> /DACK6
- U5 pad 27: (no net) -> /DRQ6
- U5 pad 28: (no net) -> /DACK7
- U5 pad 29: (no net) -> /DRQ7
- U5 pad 39: (no net) -> /CLK2
- U6 pad 12: (no net) -> /RIA
- U6 pad 13: (no net) -> /DTRA
- U6 pad 14: (no net) -> /CTSA
- U6 pad 15: (no net) -> /TXA
- U6 pad 16: (no net) -> /RTSA
- U6 pad 17: (no net) -> /RXA
- U6 pad 18: (no net) -> /DSRA
- U6 pad 19: (no net) -> /CDA
- U6 pad 2: (no net) -> /DCD1
- U6 pad 3: (no net) -> /DSR1
- U6 pad 4: (no net) -> /RX1
- U6 pad 5: (no net) -> /RTS1
- U6 pad 6: (no net) -> /TX1
- U6 pad 7: (no net) -> /CTS1
- U6 pad 8: (no net) -> /DTR1
- U6 pad 9: (no net) -> /RI1
- U7 pad 10: /SA2 -> /SA1
- U7 pad 11: /SA1 -> /SA0
- U7 pad 12: /SA0 -> (no net)
- U7 pad 17: /XD3 -> (no net)
- U7 pad 18: /XD4 -> /XD3
- U7 pad 19: /XD5 -> /XD4
- U7 pad 2: (no net) -> /SA15
- U7 pad 20: /XD6 -> /XD5
- U7 pad 21: /XD7 -> /XD6
- U7 pad 22: /KBSJ -> /XD7
- U7 pad 23: /SA10 -> /KBSJ
- U7 pad 24: /MEMR -> /SA10
- U7 pad 25: /SA11 -> /MEMR
- U7 pad 26: /SA9 -> (no net)
- U7 pad 27: /SA8 -> /SA11
- U7 pad 28: /SA13 -> /SA9
- U7 pad 29: /SA14 -> /SA8
- U7 pad 3: /SA15 -> /SA12
- U7 pad 30: (no net) -> /SA13
- U7 pad 31: (no net) -> /SA14
- U7 pad 4: /SA12 -> /SA7
- U7 pad 5: /SA7 -> /SA6
- U7 pad 6: /SA6 -> /SA5
- U7 pad 7: /SA5 -> /SA4
- U7 pad 8: /SA4 -> /SA3
- U7 pad 9: /SA3 -> /SA2
- U8 pad 12: (no net) -> /RIB
- U8 pad 13: (no net) -> /DTRB
- U8 pad 14: (no net) -> /CTSB
- U8 pad 15: (no net) -> /TXB
- U8 pad 16: (no net) -> /RTSB
- U8 pad 17: (no net) -> /RXB
- U8 pad 18: (no net) -> /DSRB
- U8 pad 19: (no net) -> /CDB
- U8 pad 2: (no net) -> /DCD2
- U8 pad 3: (no net) -> /DSR2
- U8 pad 4: (no net) -> /RX2
- U8 pad 5: (no net) -> /RTS2
- U8 pad 6: (no net) -> /TX2
- U8 pad 7: (no net) -> /CTS2
- U8 pad 8: (no net) -> /DTR2
- U8 pad 9: (no net) -> /RI2
- X1 pad 3: (no net) -> /14MHz

Commit message: wip pcb rev.A
Parts:
- removed RN7: 4.7k, Resistor_SMD:R_Array_Convex_4x0603
- removed X2: 14.7456 MHz, Oscillator:Oscillator_SMD_SeikoEpson_SG8002CA-4Pin_7.0x5.0mm
- added C18: 10u, Capacitor_SMD:C_0805_2012Metric_Pad1.18x1.45mm_HandSolder, B.Cu at (124.2, 123.3)
- added C19: 10u, Capacitor_SMD:C_0805_2012Metric_Pad1.18x1.45mm_HandSolder, B.Cu at (121.9, 123.3)
- added C20: 100n, Capacitor_SMD:C_0603_1608Metric_Pad1.08x0.95mm_HandSolder, B.Cu at (160.4, 95.5)
- added C21: 100n, Capacitor_SMD:C_0603_1608Metric_Pad1.08x0.95mm_HandSolder, B.Cu at (147.7, 74.0)
- added C22: 100n, Capacitor_SMD:C_0603_1608Metric_Pad1.08x0.95mm_HandSolder, B.Cu at (173.4, 96.8)
- added C23: 100n, Capacitor_SMD:C_0603_1608Metric_Pad1.08x0.95mm_HandSolder, B.Cu at (153.2, 69.7)
- added C24: 100n, Capacitor_SMD:C_0603_1608Metric_Pad1.08x0.95mm_HandSolder, B.Cu at (168.5, 69.8)
- added C25: 100n, Capacitor_SMD:C_0603_1608Metric_Pad1.08x0.95mm_HandSolder, B.Cu at (147.7, 94.1)
- added C26: 100n, Capacitor_SMD:C_0603_1608Metric_Pad1.08x0.95mm_HandSolder, B.Cu at (173.4, 81.6)
- added C27: 100n, Capacitor_SMD:C_0603_1608Metric_Pad1.08x0.95mm_HandSolder, B.Cu at (172.8, 74.5)
- added C28: 100n, Capacitor_SMD:C_0603_1608Metric_Pad1.08x0.95mm_HandSolder, B.Cu at (147.7, 84.0)
- added C29: 100n, Capacitor_SMD:C_0603_1608Metric_Pad1.08x0.95mm_HandSolder, B.Cu at (119.3, 95.2)
- added C30: 100n, Capacitor_SMD:C_0603_1608Metric_Pad1.08x0.95mm_HandSolder, B.Cu at (119.3, 69.8)
- added C31: 100n, Capacitor_SMD:C_0603_1608Metric_Pad1.08x0.95mm_HandSolder, B.Cu at (134.7, 69.8)
- added C32: 100n, Capacitor_SMD:C_0603_1608Metric_Pad1.08x0.95mm_HandSolder, B.Cu at (119.3, 76.2)
- added C33: 100n, Capacitor_SMD:C_0603_1608Metric_Pad1.08x0.95mm_HandSolder, B.Cu at (134.7, 95.2)
- added C34: 100n, Capacitor_SMD:C_0603_1608Metric_Pad1.08x0.95mm_HandSolder, B.Cu at (134.7, 76.2)
- added C35: 100n, Capacitor_SMD:C_0603_1608Metric_Pad1.08x0.95mm_HandSolder, B.Cu at (179.9, 113.5)
- added C36: 100n, Capacitor_SMD:C_0603_1608Metric_Pad1.08x0.95mm_HandSolder, B.Cu at (124.1, 102.4)
- added C37: 100n, Capacitor_SMD:C_0603_1608Metric_Pad1.08x0.95mm_HandSolder, B.Cu at (124.1, 110.0)
- added C38: 100n, Capacitor_SMD:C_0603_1608Metric_Pad1.08x0.95mm_HandSolder, B.Cu at (111.9, 98.5)
- added C39: 100n, Capacitor_SMD:C_0603_1608Metric_Pad1.08x0.95mm_HandSolder, B.Cu at (111.9, 105.9)
- added C40: 100n, Capacitor_SMD:C_0603_1608Metric_Pad1.08x0.95mm_HandSolder, B.Cu at (111.9, 107.5)
- added C41: 100n, Capacitor_SMD:C_0603_1608Metric_Pad1.08x0.95mm_HandSolder, B.Cu at (111.9, 100.0)
- added C42: 100n, Capacitor_SMD:C_0603_1608Metric_Pad1.08x0.95mm_HandSolder, B.Cu at (111.9, 111.3)
- added C43: 100n, Capacitor_SMD:C_0603_1608Metric_Pad1.08x0.95mm_HandSolder, B.Cu at (111.9, 104.0)
- added C44: 100n, Capacitor_SMD:C_0603_1608Metric_Pad1.08x0.95mm_HandSolder, B.Cu at (111.9, 113.7)
- added C45: 100n, Capacitor_SMD:C_0603_1608Metric_Pad1.08x0.95mm_HandSolder, B.Cu at (123.0, 135.8)
- added C46: 100n, Capacitor_SMD:C_0603_1608Metric_Pad1.08x0.95mm_HandSolder, B.Cu at (111.9, 115.2)
- added C48: 100n, Capacitor_SMD:C_0603_1608Metric_Pad1.08x0.95mm_HandSolder, B.Cu at (159.4, 107.2)
- added C49: 100n, Capacitor_SMD:C_0603_1608Metric_Pad1.08x0.95mm_HandSolder, B.Cu at (135.1, 64.7)
- added C50: 100n, Capacitor_SMD:C_0603_1608Metric_Pad1.08x0.95mm_HandSolder, B.Cu at (148.7, 124.8)
- added C51: 100n, Capacitor_SMD:C_0603_1608Metric_Pad1.08x0.95mm_HandSolder, B.Cu at (150.2, 124.8)
- added C52: 10u, Capacitor_SMD:C_0805_2012Metric_Pad1.18x1.45mm_HandSolder, B.Cu at (152.1, 124.8)
- added C53: 10u, Capacitor_SMD:C_0805_2012Metric_Pad1.18x1.45mm_HandSolder, B.Cu at (127.2, 95.2)
- added C54: 10u, Capacitor_SMD:C_0805_2012Metric_Pad1.18x1.45mm_HandSolder, B.Cu at (161.2, 71.3)
- added C55: 10u, Capacitor_SMD:C_0805_2012Metric_Pad1.18x1.45mm_HandSolder, B.Cu at (177.3, 128.4)
- added C56: 100n, Capacitor_SMD:C_0603_1608Metric_Pad1.08x0.95mm_HandSolder, B.Cu at (181.3, 138.6)
- added C57: 22p, Capacitor_SMD:C_0603_1608Metric_Pad1.08x0.95mm_HandSolder, B.Cu at (123.1, 116.0)
- added C58: 22p, Capacitor_SMD:C_0603_1608Metric_Pad1.08x0.95mm_HandSolder, B.Cu at (126.1, 116.0)
- added C8: 47u, Capacitor_SMD:CP_Elec_5x5.9, F.Cu at (163.6, 59.9)
- added D7: BZV55C5V6, Diode_SMD:D_MiniMELF, B.Cu at (164.8, 56.2)
- added D8: BT168GW, Package_TO_SOT_SMD:SOT-223-3_TabPin2, B.Cu at (163.8, 62.0)
- added R16: 22, Resistor_SMD:R_0603_1608Metric_Pad0.98x0.95mm_HandSolder, B.Cu at (186.4, 67.9)
- added R17: 22, Resistor_SMD:R_0603_1608Metric_Pad0.98x0.95mm_HandSolder, F.Cu at (157.3, 101.3)
- added R19: 22, Resistor_SMD:R_0603_1608Metric_Pad0.98x0.95mm_HandSolder, F.Cu at (154.6, 64.8)
- added R20: 4.7k, Resistor_SMD:R_0603_1608Metric_Pad0.98x0.95mm_HandSolder, B.Cu at (155.1, 94.6)
- added R21: 1k, Resistor_SMD:R_0603_1608Metric_Pad0.98x0.95mm_HandSolder, B.Cu at (166.6, 53.2)
- added Y3: 14.7456 MHz, Crystal:Crystal_SMD_SeikoEpson_TSX3225-4Pin_3.2x2.5mm_HandSoldering, F.Cu at (124.6, 116.0)
- J2: value PJ-320 -> PJ-322
- U14: value 74LS32 -> 74HCT32
- moved R18 5.90 mm to (111.2, 138.9)
- moved Q2 5.90 mm to (108.4, 138.8)
- moved F1 4.24 mm to (169.8, 60.8)
- moved R12 4.18 mm to (116.8, 139.8)
- moved R13 4.08 mm to (103.3, 139.8)
- moved U9 3.50 mm to (121.9, 129.9)
- moved C15 3.36 mm to (178.9, 64.8)
- moved D3 3.36 mm to (176.9, 65.5)
- moved U10 3.36 mm to (173.9, 59.9)
- moved C13 3.36 mm to (177.8, 59.0)
- moved C14 3.36 mm to (173.7, 67.0)
- moved C16 3.36 mm to (181.9, 62.0)
- moved D4 3.36 mm to (181.7, 65.0)
- moved L1 3.36 mm to (177.9, 62.0)
- moved R14 3.36 mm to (174.7, 64.2)
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Connections:
- J1 pad 2: unconnected-(J1-Pad2) -> (no net)
- J1 pad 6: unconnected-(J1-Pad6) -> (no net)
- J4 pad 2: unconnected-(J4-Pad2) -> (no net)
- J4 pad 6: unconnected-(J4-Pad6) -> (no net)
- J6 pad 3: GND -> (no net)
- J8 pad 59: /14MHz -> Net-(J8-Pad59)
- RN3 pad 1: /MEMW -> (no net)
- RN3 pad 2: /MEMR -> (no net)
- RN3 pad 3: (no net) -> /MEMW
- RN3 pad 4: (no net) -> /MEMR
- RN4 pad 1: /REFRESH -> /NOWS
- RN4 pad 3: /NOWS -> /REFRESH
- RN6 pad 5: /TC -> /DACK5
- RN6 pad 6: /DACK5 -> /DACK1
- RN6 pad 7: /DACK1 -> /DACK0
- RN6 pad 8: /DACK0 -> /TC
- U13 pad 26: (no net) -> Net-(U13-Pad26)
- U13 pad 46: +5V -> Net-(U13-Pad46)
- U13 pad 48: +5V -> Net-(U13-Pad46)
- U13 pad 49: +5V -> Net-(U13-Pad46)
- U5 pad 117: /14MHz -> Net-(R17-Pad1)
- U5 pad 39: /CLK2 -> Net-(R19-Pad1)
- X1 pad 1: +3V3 -> +5V
- X1 pad 4: +3V3 -> +5V
- X3 pad 1: +3V3 -> +5V
- X3 pad 4: +3V3 -> +5V
Other:
- copper layers 2 -> 4

Commit message: wip pcb rev.A
Parts:
- J12: footprint Connector_PinSocket_2.54mm:PinSocket_2x07_P2.54mm_Vertical -> Connector_PinSocket_2.54mm:PinSocket_2x08_P2.54mm_Vertical
- moved J9 4.48 mm to (101.8, 70.9)
- moved J10 2.00 mm to (101.8, 89.1)
- moved J12 1.28 mm to (141.2, 58.5)
- moved C8 0.80 mm to (164.4, 59.9)
Connections:
- C57 pad 1: Net-(U13-Pad25) -> (no net)
- C58 pad 1: Net-(U13-Pad26) -> (no net)
- U13 pad 25: Net-(U13-Pad25) -> (no net)
- U13 pad 26: Net-(U13-Pad26) -> (no net)
- Y3 pad 1: Net-(U13-Pad26) -> (no net)
- Y3 pad 3: Net-(U13-Pad25) -> (no net)

Commit message: wip pcb rev.A
Parts:
- added D9: MBR0520, Diode_SMD:D_SOD-123, B.Cu at (181.4, 65.8)
- added R22: 51k, Resistor_SMD:R_0603_1608Metric_Pad0.98x0.95mm_HandSolder, F.Cu at (174.0, 59.9)
- C15: footprint Capacitor_SMD:C_0603_1608Metric_Pad1.08x0.95mm_HandSolder -> Capacitor_SMD:C_0805_2012Metric_Pad1.18x1.45mm_HandSolder
- D4: value BAT54S -> MBR0520; footprint Package_TO_SOT_SMD:SOT-23 -> Diode_SMD:D_SOD-123
- L1: value L -> 10u; footprint Inductor_SMD:L_0805_2012Metric_Pad1.15x1.40mm_HandSolder -> Inductor_THT:L_Radial_D9.5mm_P5.00mm_Fastron_07HVP; moved to F.Cu
- R14: value R -> 113k
- R15: value R -> 13.3k
- moved L1 4.52 mm to (173.4, 62.5), turned to 0 degrees
- moved D4 2.14 mm to (183.8, 65.8)
- moved D7 0.92 mm to (163.9, 56.2)
- moved R21 0.80 mm to (165.8, 53.2)
- moved C16 0.68 mm to (182.6, 62.2)
- moved C8 0.30 mm to (164.1, 59.9)
- moved C15 0.28 mm to (179.1, 65.1)
- moved SW2 0.23 mm to (171.4, 56.0)
- moved D8 0.07 mm to (163.7, 62.0)
Connections:
- C57 pad 1: (no net) -> Net-(C57-Pad1)
- C58 pad 1: (no net) -> Net-(C58-Pad1)
- D4 pad 1: -12V -> GND
- D4 pad 2: GND -> Net-(C15-Pad2)
- J12 pad 15: unconnected-(J12-Pad15) -> (no net)
- U10 pad 4: +5V -> Net-(U10-Pad4)
- U13 pad 25: (no net) -> Net-(C57-Pad1)
- U13 pad 26: (no net) -> Net-(C58-Pad1)
- U14 pad 4: (no net) -> GND
- U14 pad 5: (no net) -> GND
- Y3 pad 1: (no net) -> Net-(C58-Pad1)
- Y3 pad 3: (no net) -> Net-(C57-Pad1)

Commit message: wip pcb rev.A
Parts:
- removed H5, H6, H7, H8: MountingHole, my:MountingHole_3.2mm_M3_dk5.2mm_Mask
- added C47: 10p, Capacitor_SMD:C_0603_1608Metric_Pad1.08x0.95mm_HandSolder, B.Cu at (174.7, 42.8)
- added LOGO1: graphic, mygraphic:black-mage-12.5x8.6, F.Cu at (160.8, 82.8)
- H1, H2, H3, H4: value MountingHole -> Screw M3 dk=5mm L=4mm
- moved C49 0.45 mm to (134.7, 64.7), turned to 180 degrees
- moved X3 0.45 mm to (134.7, 64.7), turned to 0 degrees
- turned R19 to 180 degrees
Connections:
- net /~CF_BUSY renamed /~{CF_BUSY}
- CON1 pad 25: (no net) -> unconnected-(CON1-Pad25)
- CON1 pad 26: (no net) -> unconnected-(CON1-Pad26)
- CON1 pad 33: (no net) -> unconnected-(CON1-Pad33)
- CON1 pad 40: (no net) -> unconnected-(CON1-Pad40)
- CON1 pad 43: (no net) -> unconnected-(CON1-Pad43)
- J1 pad 2: (no net) -> unconnected-(J1-Pad2)
- J1 pad 6: (no net) -> unconnected-(J1-Pad6)
- J10 pad 10: (no net) -> unconnected-(J10-Pad10)
- J12 pad 15: (no net) -> unconnected-(J12-Pad15)
- J3 pad 4: (no net) -> unconnected-(J3-Pad4)
- J4 pad 2: (no net) -> unconnected-(J4-Pad2)
- J4 pad 6: (no net) -> unconnected-(J4-Pad6)
- J5 pad 11: (no net) -> unconnected-(J5-Pad11)
- J5 pad 15: (no net) -> unconnected-(J5-Pad15)
- J5 pad 4: (no net) -> unconnected-(J5-Pad4)
- J6 pad 3: (no net) -> unconnected-(J6-Pad3)
- J7 pad 12: (no net) -> unconnected-(J7-Pad12)
- J7 pad 39: (no net) -> unconnected-(J7-Pad39)
- J8 pad 19: (no net) -> unconnected-(J8-Pad19)
- J8 pad 9: (no net) -> unconnected-(J8-Pad9)
- J9 pad 10: (no net) -> unconnected-(J9-Pad10)
- RN3 pad 1: (no net) -> unconnected-(RN3-Pad1)
- RN3 pad 2: (no net) -> unconnected-(RN3-Pad2)
- RN4 pad 4: (no net) -> unconnected-(RN4-Pad4)
- RN5 pad 3: (no net) -> /IOCHK
- U1 pad 15: (no net) -> unconnected-(U1-Pad15)
- U11 pad 6: (no net) -> unconnected-(U11-Pad6)
- U11 pad 9: (no net) -> unconnected-(U11-Pad9)
- U12 pad 4: (no net) -> unconnected-(U12-Pad4)
- U14 pad 3: (no net) -> unconnected-(U14-Pad3)
- U14 pad 6: (no net) -> unconnected-(U14-Pad6)
- U15 pad 10: (no net) -> unconnected-(U15-Pad10)
- U15 pad 11: (no net) -> unconnected-(U15-Pad11)
- U15 pad 12: (no net) -> unconnected-(U15-Pad12)
- U15 pad 13: (no net) -> unconnected-(U15-Pad13)
- U15 pad 14: (no net) -> unconnected-(U15-Pad14)
- U15 pad 15: (no net) -> unconnected-(U15-Pad15)
- U15 pad 9: (no net) -> unconnected-(U15-Pad9)
- U16 pad 12: (no net) -> unconnected-(U16-Pad12)
- U16 pad 13: (no net) -> unconnected-(U16-Pad13)
- U16 pad 14: (no net) -> unconnected-(U16-Pad14)
- U16 pad 15: (no net) -> unconnected-(U16-Pad15)
- U2 pad 10: (no net) -> unconnected-(U2-Pad10)
- U2 pad 11: (no net) -> unconnected-(U2-Pad11)
- U2 pad 12: (no net) -> unconnected-(U2-Pad12)
- U2 pad 13: (no net) -> unconnected-(U2-Pad13)
- U2 pad 14: (no net) -> unconnected-(U2-Pad14)
- U2 pad 19: (no net) -> unconnected-(U2-Pad19)
- U2 pad 2: (no net) -> unconnected-(U2-Pad2)
- U2 pad 20: (no net) -> unconnected-(U2-Pad20)
- U2 pad 5: (no net) -> unconnected-(U2-Pad5)
- U2 pad 6: (no net) -> unconnected-(U2-Pad6)
- U2 pad 9: (no net) -> unconnected-(U2-Pad9)
- U3 pad 11: (no net) -> unconnected-(U3-Pad11)
- U3 pad 12: (no net) -> unconnected-(U3-Pad12)
- U3 pad 15: (no net) -> unconnected-(U3-Pad15)
- U3 pad 16: (no net) -> unconnected-(U3-Pad16)
- U3 pad 32: (no net) -> unconnected-(U3-Pad32)
- U4 pad 11: (no net) -> unconnected-(U4-Pad11)
- U4 pad 12: (no net) -> unconnected-(U4-Pad12)
- U4 pad 15: (no net) -> unconnected-(U4-Pad15)
- U4 pad 16: (no net) -> unconnected-(U4-Pad16)
- U4 pad 32: (no net) -> unconnected-(U4-Pad32)
- U5 pad 109: (no net) -> unconnected-(U5-Pad109)
- U5 pad 114: (no net) -> unconnected-(U5-Pad114)
- U5 pad 115: (no net) -> unconnected-(U5-Pad115)
- U5 pad 116: (no net) -> unconnected-(U5-Pad116)
- U5 pad 124: (no net) -> unconnected-(U5-Pad124)
- U5 pad 126: (no net) -> unconnected-(U5-Pad126)
- U5 pad 127: (no net) -> unconnected-(U5-Pad127)
- U5 pad 2: (no net) -> unconnected-(U5-Pad2)
- U5 pad 30: (no net) -> unconnected-(U5-Pad30)
- U5 pad 33: (no net) -> unconnected-(U5-Pad33)
- U5 pad 35: (no net) -> unconnected-(U5-Pad35)
- U5 pad 36: (no net) -> unconnected-(U5-Pad36)
- U5 pad 37: (no net) -> unconnected-(U5-Pad37)
- U5 pad 41: (no net) -> unconnected-(U5-Pad41)
- U5 pad 42: (no net) -> unconnected-(U5-Pad42)
- U5 pad 43: (no net) -> unconnected-(U5-Pad43)
- U5 pad 44: (no net) -> unconnected-(U5-Pad44)
- U5 pad 45: (no net) -> unconnected-(U5-Pad45)
- U5 pad 47: (no net) -> unconnected-(U5-Pad47)
- U5 pad 48: (no net) -> unconnected-(U5-Pad48)
- U5 pad 49: (no net) -> unconnected-(U5-Pad49)
- U5 pad 51: (no net) -> /GPCS0
- U5 pad 55: (no net) -> unconnected-(U5-Pad55)
- U5 pad 56: (no net) -> unconnected-(U5-Pad56)
- U5 pad 57: (no net) -> unconnected-(U5-Pad57)
- U5 pad 77: (no net) -> unconnected-(U5-Pad77)
- U5 pad 78: (no net) -> unconnected-(U5-Pad78)
- U5 pad 80: (no net) -> unconnected-(U5-Pad80)
- U5 pad 82: (no net) -> unconnected-(U5-Pad82)
- U5 pad 86: (no net) -> unconnected-(U5-Pad86)
- U5 pad 87: (no net) -> unconnected-(U5-Pad87)
- U5 pad 88: (no net) -> unconnected-(U5-Pad88)
- U5 pad 89: (no net) -> unconnected-(U5-Pad89)
- U5 pad 95: (no net) -> unconnected-(U5-Pad95)
- U5 pad 96: (no net) -> unconnected-(U5-Pad96)
- U7 pad 1: (no net) -> unconnected-(U7-Pad1)
- U7 pad 12: (no net) -> unconnected-(U7-Pad12)
- U7 pad 17: (no net) -> unconnected-(U7-Pad17)
- U7 pad 26: (no net) -> unconnected-(U7-Pad26)
