File: pcb_main/rev.A/charon386_main.kicad_pcb (KiCad board)
At the start: 4 copper layers, 100 x 100 mm, 143 parts, among them CON1 CF-CARD-cfcard, J1 Mini-DIN-6, J10 COM2, J11 ESP, J12 Conn_02x07_Odd_Even, J2 PJ-322, J3 USB_B_Micro, J4 Mini-DIN-6, J5 DB15_Female_HighDensity_Mount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, J6 Conn_01x04, J7 PC104_16, J8 PC104, J9 COM1, Q1 BC817, Q2 BC856, SW1 SW_Push, SW2 Jumper / Pin header 1x2 Pitch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, U1 CH340G, U10 LT1930, U11 TXB0104PW, U12 MAX823LEUK, U13 ST16C554, U14 74HCT32, U15 74HCT138, U16 74HCT138, U2 ESP-12E, U3 MSM5118160F-JS, U4 MSM5118160F-JS, U5 M6117D, U6 GD75232PW, U7 27C512PLCC, U8 GD75232PW, U9 AMS1117-3.3, X1 14.318 MHz, X3 80 MHz, Y1 12 MHz, Y2 32768 Hz, Y3 14.7456 MHz

Commit message: wip pcb rev.A
Parts:
- removed Y3: 14.7456 MHz, Crystal:Crystal_SMD_SeikoEpson_TSX3225-4Pin_3.2x2.5mm_HandSoldering
- added C59: 1u, Capacitor_SMD:C_0603_1608Metric_Pad1.08x0.95mm_HandSolder, B.Cu at (160.4, 94.2)
- added C60: 1u, Capacitor_SMD:C_0603_1608Metric_Pad1.08x0.95mm_HandSolder, B.Cu at (172.1, 77.0)
- added C61: 1u, Capacitor_SMD:C_0603_1608Metric_Pad1.08x0.95mm_HandSolder, B.Cu at (147.2, 94.2)
- added C62: 1u, Capacitor_SMD:C_0603_1608Metric_Pad1.08x0.95mm_HandSolder, B.Cu at (171.9, 69.7)
- added C63: 1u, Capacitor_SMD:C_0603_1608Metric_Pad1.08x0.95mm_HandSolder, B.Cu at (173.4, 98.5)
- added C64: 1u, Capacitor_SMD:C_0603_1608Metric_Pad1.08x0.95mm_HandSolder, B.Cu at (149.2, 74.0)
- added C65: 1u, Capacitor_SMD:C_0603_1608Metric_Pad1.08x0.95mm_HandSolder, B.Cu at (149.2, 84.0)
- added C66: 1u, Capacitor_SMD:C_0603_1608Metric_Pad1.08x0.95mm_HandSolder, B.Cu at (153.2, 71.2)
- added C67: 1u, Capacitor_SMD:C_0603_1608Metric_Pad1.08x0.95mm_HandSolder, B.Cu at (115.5, 77.8)
- added C68: 1u, Capacitor_SMD:C_0603_1608Metric_Pad1.08x0.95mm_HandSolder, B.Cu at (132.8, 77.8)
- added C69: 100n, Capacitor_SMD:C_0603_1608Metric_Pad1.08x0.95mm_HandSolder, B.Cu at (136.5, 103.6)
- added C70: 100n, Capacitor_SMD:C_0603_1608Metric_Pad1.08x0.95mm_HandSolder, B.Cu at (142.2, 103.6)
- added C71: 100n, Capacitor_SMD:C_0603_1608Metric_Pad1.08x0.95mm_HandSolder, B.Cu at (147.6, 103.6)
- added C72: 100n, Capacitor_SMD:C_0603_1608Metric_Pad1.08x0.95mm_HandSolder, B.Cu at (127.0, 108.8)
- added C73: 100n, Capacitor_SMD:C_0603_1608Metric_Pad1.08x0.95mm_HandSolder, B.Cu at (126.3, 103.2)
- added X2: 1.8432 Mhz, Oscillator:Oscillator_SMD_SeikoEpson_SG8002CA-4Pin_7.0x5.0mm, F.Cu at (128.5, 117.2)
- C57: value 22p -> 100n
- C58: value 22p -> 1u
- C6, C7, R16, R4: moved to F.Cu
- C8: value 47u -> 100u; footprint Capacitor_SMD:CP_Elec_5x5.9 -> Capacitor_Tantalum_SMD:CP_EIA-7343-31_Kemet-D_Pad2.25x2.55mm_HandSolder
- L1: footprint Inductor_THT:L_Radial_D9.5mm_P5.00mm_Fastron_07HVP -> Inductor_SMD:L_Taiyo-Yuden_NR-60xx_HandSoldering
- R5: footprint Resistor_SMD:R_0805_2012Metric_Pad1.20x1.40mm_HandSolder -> Resistor_SMD:R_0603_1608Metric_Pad0.98x0.95mm_HandSolder
- U7: value 27C512PLCC -> 27C512
- Y2: footprint Crystal:Crystal_C38-LF_D3.0mm_L8.0mm_Horizontal_1EP_style2 -> Crystal:Crystal_SMD_SeikoEpson_MC306-4Pin_8.0x3.2mm_HandSoldering
- moved C58 57.4 mm to (172.1, 81.6)
- moved D5 43.1 mm to (120.5, 64.9)
- moved C47 21.6 mm to (175.5, 64.4), turned to 90 degrees
- moved R2 8.08 mm to (192.2, 52.2), turned to -90 degrees
- moved R7 7.99 mm to (115.7, 52.2), turned to -90 degrees
- moved C11 5.86 mm to (190.6, 52.2), turned to 90 degrees
- moved C9 5.78 mm to (114.1, 52.2), turned to 90 degrees
- moved Y2 5.64 mm to (152.4, 105.7), turned to -90 degrees
- moved C57 5.53 mm to (128.5, 117.2)
- moved C15 5.32 mm to (182.9, 61.3), turned to 0 degrees
- moved R6 5.11 mm to (108.2, 52.2)
- moved C10 5.11 mm to (106.6, 52.2)
- moved C12 4.92 mm to (184.7, 52.2)
- moved R1 4.92 mm to (183.1, 52.2)
- moved C14 4.35 mm to (177.3, 64.6), turned to -90 degrees
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Connections:
- C57 pad 1: Net-(C57-Pad1) -> +5V
- C58 pad 1: Net-(C58-Pad1) -> GND
- C58 pad 2: GND -> +5V
- D5 pad 1: Net-(BT1-Pad1) -> +3V3
- D5 pad 2: +3V3 -> Net-(BT1-Pad1)
- J11 pad 10: /CTSD -> /CTSC
- J8 pad 2: /IOCHCK -> /IOCHK
- RN3 pad 1: unconnected-(RN3-Pad1) -> /AEN
- RN5 pad 1: /MEMCS16 -> /IOCS16
- RN5 pad 2: /IOCS16 -> /MEMCS16
- RN5 pad 3: /IOCHK -> /MASTER
- RN5 pad 4: /MASTER -> /IOCHK
- U1 pad 10: /DTRC -> /DTRD
- U1 pad 12: /DTRC -> /DTRD
- U1 pad 13: /DSRC -> /DSRD
- U1 pad 14: /CTSC -> /CTSD
- U1 pad 2: /RXC -> /RXD
- U1 pad 3: /TXC -> /TXD
- U1 pad 9: /RTSC -> /RTSD
- U11 pad 10: /RTSD -> /RTSC
- U11 pad 11: /TXD -> /TXC
- U11 pad 12: /RXD -> /RXC
- U13 pad 25: Net-(C57-Pad1) -> Net-(U13-Pad25)
- U13 pad 26: Net-(C58-Pad1) -> unconnected-(U13-Pad26)
- U13 pad 31: /DSRC -> Net-(U13-Pad32)
- U13 pad 32: /DSRC -> Net-(U13-Pad32)
- U13 pad 34: /DTRC -> Net-(U13-Pad32)
- U13 pad 46: Net-(U13-Pad46) -> /DTRD
- U13 pad 48: Net-(U13-Pad46) -> /DSRD
- U13 pad 49: Net-(U13-Pad46) -> /DSRD
- U5 pad 196: /IOCHCK -> /IOCHK
- U6 pad 12: /RIA -> /CTSA
- U6 pad 13: /DTRA -> /TXA
- U6 pad 14: /CTSA -> /DSRA
- U6 pad 15: /TXA -> /RTSA
- U6 pad 16: /RTSA -> /DTRA
- U6 pad 17: /RXA -> /CDA
- U6 pad 18: /DSRA -> /RIA
- U6 pad 19: /CDA -> /RXA
- U6 pad 2: /DCD1 -> /RX1
- U6 pad 3: /DSR1 -> /RI1
- U6 pad 4: /RX1 -> /DCD1
- U6 pad 5: /RTS1 -> /DTR1
- U6 pad 6: /TX1 -> /RTS1
- U6 pad 7: /CTS1 -> /DSR1
- U6 pad 8: /DTR1 -> /TX1
- U6 pad 9: /RI1 -> /CTS1
- U8 pad 12: /RIB -> /RXB
- U8 pad 14: /CTSB -> /RIB
- U8 pad 15: /TXB -> /RTSB
- U8 pad 16: /RTSB -> /TXB
- U8 pad 17: /RXB -> /CDB
- U8 pad 19: /CDB -> /CTSB
- U8 pad 2: /DCD2 -> /CTS2
- U8 pad 4: /RX2 -> /DCD2
- U8 pad 5: /RTS2 -> /TX2
- U8 pad 6: /TX2 -> /RTS2
- U8 pad 7: /CTS2 -> /RI2
- U8 pad 9: /RI2 -> /RX2
- Y2 pad 2: Net-(C7-Pad1) -> GND
Routing:
- added copper zone on F.Cu, net GND
- added copper zone on In1.Cu, net GND
Other:
- board text added: "1"
- board text added: "2"
- board text added: "3"
- board text added: "4"

Commit message: wip pcb rev.A
Parts:
- removed C50: 100n, Capacitor_SMD:C_0603_1608Metric_Pad1.08x0.95mm_HandSolder
- removed R9: 4.7k, Resistor_SMD:R_0603_1608Metric_Pad0.98x0.95mm_HandSolder
- J1, J4: footprint my:MINI_DIN_6_33PRIMARY -> my:minidin-6
- moved J6 7.60 mm to (176.6, 123.7), turned to 90 degrees
- moved LS1 7.60 mm to (184.2, 131.8), turned to 180 degrees
- moved R11 6.27 mm to (177.6, 126.6), turned to 0 degrees
- moved C5 6.20 mm to (183.2, 126.6), turned to 0 degrees
- moved R3 5.92 mm to (177.6, 128.8), turned to 0 degrees
- moved C55 5.91 mm to (183.2, 128.8), turned to 180 degrees
- moved C52 3.78 mm to (148.6, 126.2), turned to 180 degrees
- moved Q1 3.33 mm to (180.4, 131.8)
- moved R19 1.76 mm to (152.8, 65.0)
- moved C51 1.71 mm to (148.6, 124.4), turned to 0 degrees
- moved C10 1.60 mm to (108.2, 52.2)
- moved R6 1.60 mm to (106.6, 52.2)
- moved C48 0.90 mm to (159.7, 107.1)
- moved R17 0.90 mm to (156.6, 101.5)
- moved R4 0.90 mm to (152.4, 101.5)
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Connections:
- C2 pad 1: Net-(C2-Pad1) -> Net-(U1-Pad7)
- CON1 pad 46: Net-(CON1-Pad46) -> unconnected-(CON1-Pad46)
- CON1 pad S1: (no net) -> unconnected-(CON1-PadS1)
- CON1 pad S2: (no net) -> unconnected-(CON1-PadS2)
- D1 pad 1: /~{CF_BUSY} -> Net-(D1-Pad1)
- D1 pad 2: Net-(D1-Pad2) -> +5V
- D2 pad 1: GND -> Net-(D2-Pad1)
- D2 pad 2: Net-(D2-Pad2) -> +5V
- D6 pad 2: Net-(D6-Pad2) -> +5V
- Q2 pad 2: Net-(D6-Pad1) -> Net-(Q2-Pad2)
- R12 pad 1: +5V -> Net-(D1-Pad1)
- R12 pad 2: Net-(D1-Pad2) -> /~{CF_BUSY}
- R13 pad 1: +5V -> Net-(D2-Pad1)
- R13 pad 2: Net-(D2-Pad2) -> GND
- R18 pad 1: +5V -> Net-(D6-Pad1)
- R18 pad 2: Net-(D6-Pad2) -> Net-(Q2-Pad2)
- U1 pad 7: Net-(C3-Pad1) -> Net-(U1-Pad7)
- U1 pad 8: Net-(C2-Pad1) -> Net-(C3-Pad1)
- U11 pad 10: /RTSC -> /RESETL
- U11 pad 11: /TXC -> /RTSC
- U11 pad 12: /RXC -> /TXC
- U11 pad 13: /RESETL -> /RXC
- U11 pad 2: /ESP_RST -> Net-(J11-Pad4)
- U11 pad 3: Net-(J11-Pad4) -> Net-(J11-Pad6)
- U11 pad 4: Net-(J11-Pad6) -> Net-(J11-Pad8)
- U11 pad 5: Net-(J11-Pad8) -> /ESP_RST
- U3 pad 10: /BD7 -> /BD0
- U3 pad 2: /BD0 -> /BD7
- U3 pad 3: /BD1 -> /BD6
- U3 pad 4: /BD2 -> /BD5
- U3 pad 5: /BD3 -> /BD4
- U3 pad 7: /BD4 -> /BD3
- U3 pad 8: /BD5 -> /BD2
- U3 pad 9: /BD6 -> /BD1
- U4 pad 10: /BD7 -> /BD0
- U4 pad 2: /BD0 -> /BD7
- U4 pad 3: /BD1 -> /BD6
- U4 pad 4: /BD2 -> /BD5
- U4 pad 5: /BD3 -> /BD4
- U4 pad 7: /BD4 -> /BD3
- U4 pad 8: /BD5 -> /BD2
- U4 pad 9: /BD6 -> /BD1
- Y1 pad 1: Net-(C2-Pad1) -> Net-(U1-Pad7)
Routing:
- net +5V: track 0.00 -> 333.1 mm, vias 0 -> 43
- net GND: track 0.00 -> 241.4 mm, vias 0 -> 135
- net /SD7: track 0.00 -> 96.2 mm, vias 0 -> 4
- net /SD6: track 0.00 -> 95.9 mm, vias 0 -> 4
- net /SD5: track 0.00 -> 95.4 mm, vias 0 -> 4
- net /SD4: track 0.00 -> 94.8 mm, vias 0 -> 4
- net /SD3: track 0.00 -> 94.6 mm, vias 0 -> 4
- net /SD2: track 0.00 -> 70.3 mm, vias 0 -> 4
- net /SD1: track 0.00 -> 70.2 mm, vias 0 -> 4
- net /SD0: track 0.00 -> 68.1 mm, vias 0 -> 4
- net /~{CF_BUSY}: track 0.00 -> 54.4 mm, vias 0 -> 1
- net /MA0: track 0.00 -> 49.4 mm, vias 0 -> 2
- net /MA1: track 0.00 -> 45.6 mm, vias 0 -> 2
- net +3V3: track 0.00 -> 42.8 mm, vias 0 -> 5
- net /MA2: track 0.00 -> 41.8 mm, vias 0 -> 2
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- added copper zone on B.Cu, net +5V
- added copper zone on F.Cu, net +5V

Commit message: wip pcb rev.A
Parts:
- moved C57 17.6 mm to (124.1, 100.1), turned to 180 degrees
- moved X2 17.6 mm to (124.1, 100.1), turned to 180 degrees
- moved C73 12.2 mm to (121.9, 114.5), turned to 90 degrees
- moved C71 11.9 mm to (135.7, 103.5)
- moved U14 11.9 mm to (133.7, 103.5)
- moved C36 11.6 mm to (127.1, 113.8), turned to 0 degrees
- moved C72 5.77 mm to (121.2, 108.8), turned to 0 degrees
- moved U13 5.42 mm to (124.1, 111.5), turned to 180 degrees
- moved C70 5.23 mm to (147.4, 103.5)
- moved U15 5.23 mm to (139.4, 103.5)
- moved C69 5.23 mm to (141.7, 103.5)
- moved U16 5.23 mm to (145.1, 103.5)
- moved C37 3.56 mm to (125.9, 108.6), turned to 90 degrees
- moved C35 3.07 mm to (181.2, 110.2), turned to -90 degrees
- moved C54 2.50 mm to (158.7, 71.0), turned to 0 degrees
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Connections:
- net /USB_DM renamed /USB_DN
- CON1 pad S1: unconnected-(CON1-PadS1) -> GND
- CON1 pad S2: unconnected-(CON1-PadS2) -> GND
- J11 pad 10: /CTSC -> /CTS_ESP
- U1 pad 10: /DTRD -> /DTR_USB
- U1 pad 12: /DTRD -> /DTR_USB
- U1 pad 13: /DSRD -> /DSR_USB
- U1 pad 14: /CTSD -> /CTS_USB
- U1 pad 2: /RXD -> /RX_USB
- U1 pad 3: /TXD -> /TX_USB
- U1 pad 9: /RTSD -> /RTS_USB
- U11 pad 11: /RTSC -> /RTS_ESP
- U11 pad 12: /TXC -> /TX_ESP
- U11 pad 13: /RXC -> /RX_ESP
- U13 pad 1: /DSRA -> Net-(U13-Pad1)
- U13 pad 10: /TXB -> /TX_USB
- U13 pad 11: /0x2F8 -> /0x3E8
- U13 pad 13: /RTSB -> /RTS_USB
- U13 pad 15: /DTRB -> /DTR_USB
- U13 pad 16: /CTSB -> /CTS_USB
- U13 pad 17: /DSRB -> /DSR_USB
- U13 pad 18: /CDB -> /DSR_USB
- U13 pad 19: /RIB -> +5V
- U13 pad 2: /CTSA -> /CTS_ESP
- U13 pad 20: /RXB -> /RX_USB
- U13 pad 29: /RXC -> /RX_COM1
- U13 pad 3: /DTRA -> Net-(U13-Pad1)
- U13 pad 30: +5V -> /RI_COM1
- U13 pad 31: Net-(U13-Pad31) -> /CD_COM1
- U13 pad 32: Net-(U13-Pad31) -> /DSR_COM1
- U13 pad 33: /CTSC -> /CTS_COM1
- U13 pad 34: Net-(U13-Pad31) -> /DTR_COM1
- U13 pad 36: /RTSC -> /RTS_COM1
- U13 pad 38: /0x3E8 -> /0x3F8
- U13 pad 39: /TXC -> /TX_COM1
- U13 pad 41: /TXD -> /TX_COM2
- U13 pad 42: /0x2E8 -> /0x2F8
- U13 pad 44: /RTSD -> /RTS_COM2
- U13 pad 46: /DTRD -> /DTR_COM2
- U13 pad 47: /CTSD -> /CTS_COM2
- U13 pad 48: /DSRD -> /DSR_COM2
- U13 pad 49: /DSRD -> /CD_COM2
- U13 pad 5: /RTSA -> /RTS_ESP
- U13 pad 50: +5V -> /RI_COM2
- U13 pad 51: /RXD -> /RX_COM2
- U13 pad 62: /RXA -> /RX_ESP
- U13 pad 63: /RIA -> +5V
- U13 pad 64: /CDA -> Net-(U13-Pad1)
- U13 pad 7: /0x3F8 -> /0x2E8
- U13 pad 8: /TXA -> /TX_ESP
- U15 pad 1: /SA6 -> /SA8
- U15 pad 10: unconnected-(U15-Pad10) -> /0x3E8
- U15 pad 11: unconnected-(U15-Pad11) -> /0x2E8
- U15 pad 2: /SA7 -> /SA4
- U15 pad 3: /SA9 -> /SA3
- U15 pad 4: GND -> Net-(U15-Pad4)
- U15 pad 7: Net-(U15-Pad7) -> /0x3F8
- U15 pad 9: unconnected-(U15-Pad9) -> /0x2F8
- U16 pad 1: /SA8 -> /SA6
- U16 pad 10: /0x3E8 -> unconnected-(U16-Pad10)
- U16 pad 11: /0x2E8 -> unconnected-(U16-Pad11)
- U16 pad 2: /SA4 -> /SA7
- U16 pad 3: /SA3 -> /SA9
- U16 pad 4: Net-(U15-Pad7) -> GND
- U16 pad 7: /0x3F8 -> Net-(U15-Pad4)
- U16 pad 9: /0x2F8 -> unconnected-(U16-Pad9)
- U6 pad 12: /CTSA -> /CTS_COM1
- U6 pad 13: /TXA -> /TX_COM1
- U6 pad 14: /DSRA -> /DSR_COM1
- U6 pad 15: /RTSA -> /RTS_COM1
- U6 pad 16: /DTRA -> /DTR_COM1
- U6 pad 17: /CDA -> /CD_COM1
- U6 pad 18: /RIA -> /RI_COM1
- U6 pad 19: /RXA -> /RX_COM1
- U8 pad 12: /RXB -> /RX_COM2
- U8 pad 13: /DTRB -> /DTR_COM2
- U8 pad 14: /RIB -> /RI_COM2
- U8 pad 15: /RTSB -> /RTS_COM2
- U8 pad 16: /TXB -> /TX_COM2
- U8 pad 17: /CDB -> /CD_COM2
- U8 pad 18: /DSRB -> /DSR_COM2
- U8 pad 19: /CTSB -> /CTS_COM2
Routing:
- net +5V: track 333.1 -> 501.9 mm, vias 43 -> 44
- net /USB_DN: track 0.00 -> 116.5 mm, vias 0 -> 2
- net /USB_DP: track 0.00 -> 114.2 mm, vias 0 -> 2
- net /DRQ2: track 0.00 -> 87.1 mm, vias 0 -> 1
- net /MEMCS16: track 0.00 -> 77.1 mm, vias 0 -> 3
- net /IOCS16: track 2.71 -> 79.0 mm, vias 1 -> 4
- net /14MHz: track 3.07 -> 76.3 mm, vias 0 -> 2
- net /HDCS0: track 2.87 -> 73.9 mm, vias 1 -> 2
- net /PWG: track 0.00 -> 70.0 mm, vias 0 -> 3
- net /SD11: track 2.47 -> 71.6 mm, vias 1 -> 4
- net /SD12: track 2.47 -> 69.7 mm, vias 1 -> 4
- net /SD13: track 2.49 -> 67.7 mm, vias 1 -> 4
- net /RESETL: track 2.42 -> 67.3 mm, vias 1 -> 4
- net /HDCS1: track 2.46 -> 66.6 mm, vias 1 -> 2
- net /DRQ0: track 0.00 -> 63.8 mm, vias 0 -> 3
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