File: pcb_main/rev.A/charon386_main.kicad_pcb (KiCad board)
At the start: 4 copper layers, 100 x 100 mm, 156 parts, among them CON1 CF-CARD-cfcard, J1 Mini-DIN-6, J10 COM2, J11 ESP, J12 Conn_02x07_Odd_Even, J2 PJ-322, J3 USB_B_Micro, J4 Mini-DIN-6, J5 DB15_Female_HighDensity_Mount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, J6 Conn_01x04, J7 PC104_16, J8 PC104, J9 COM1, Q1 BC817, Q2 BC856, SW1 SW_Push, SW2 Jumper / Pin header 1x2 Pitch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, U1 CH340G, U10 LT1930, U11 TXB0104PW, U12 MAX823LEUK, U13 ST16C554, U14 74HCT32, U15 74HCT138, U16 74HCT138, U2 ESP-12E, U3 MSM5118160F-JS, U4 MSM5118160F-JS, U5 M6117D, U6 GD75232PW, U7 27C512, U8 GD75232PW, U9 AMS1117-3.3, X1 14.318 MHz, X2 1.8432 Mhz, X3 80 MHz, Y1 12 MHz, Y2 32768 Hz

Commit message: wip pcb rev.A
Routing:
- net /RSTDRV: track 1.15 -> 56.8 mm, vias 1 -> 2
- net /SA19: track 0.00 -> 44.2 mm, vias 0 -> 2
- net /NOWS: track 4.06 -> 47.6 mm, vias 1 -> 3
- net /IOCHRDY: track 20.8 -> 59.8 mm, vias 2 -> 3
- net /SMEMW: track 4.03 -> 42.3 mm, vias 1 -> 3
- net /SMEMR: track 4.11 -> 40.2 mm, vias 1 -> 3
- net /IOW: track 57.1 -> 88.4 mm, vias 3 -> 5
- net /BALE: track 0.00 -> 30.7 mm, vias 0 -> 2
- net /IOR: track 61.7 -> 90.6 mm, vias 3 -> 5
- net /MEMR: track 4.40 -> 32.9 mm, vias 1 -> 3
- net /IRQ15: track 0.00 -> 27.3 mm, vias 0 -> 2
- net /MEMW: track 4.53 -> 31.0 mm, vias 1 -> 3
- net /IRQ14: track 19.4 -> 44.1 mm
- net /SA3: track 1.15 -> 19.4 mm
- net /SA4: track 1.52 -> 19.1 mm
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
Commit message: wip pcb rev.A
Routing:
- net GND: track 256.8 -> 254.3 mm, vias 132 -> 131
- net /HDCS1: track 66.6 -> 67.4 mm
- net /HDCS0: track 73.9 -> 74.5 mm
Other:
- board text added: "Layers: 4 Dimensions: 100x100mm Thickness: 1.6mm"
- board text added: "Min clearance: 0.2mm Min track: 0.2mm Min hole: 0.3mm Min annular ring: 0.15mm"

Commit message: wip pcb rev.A
Parts:
- moved RN1 46.6 mm to (196.9, 131.8), turned to 0 degrees
- moved RN2 46.2 mm to (196.9, 127.9), turned to 0 degrees
- moved C35 4.56 mm to (183.7, 114.1), turned to 90 degrees
- moved Q2 0.72 mm to (109.1, 138.9), turned to 180 degrees
- moved R18 0.71 mm to (111.9, 139.0)
- moved R16 0.62 mm to (185.2, 67.8)
- moved C23 0.50 mm to (153.7, 69.7)
- moved C66 0.50 mm to (153.7, 71.2)
- moved C53 0.20 mm to (126.2, 95.2)
- moved D8 0.15 mm to (163.7, 61.8)
Connections:
- RN1 pad 1: /SD0 -> /SD7
- RN1 pad 2: /SD1 -> /SD6
- RN1 pad 3: /SD2 -> /SD5
- RN1 pad 4: /SD3 -> /SD4
- RN2 pad 1: /SD4 -> /SD3
- RN2 pad 2: /SD5 -> /SD2
- RN2 pad 3: /SD6 -> /SD1
- RN2 pad 4: /SD7 -> /SD0
- RN3 pad 3: /MEMW -> /MEMR
- RN3 pad 4: /MEMR -> /MEMW
- RN5 pad 1: /IOCS16 -> /MASTER
- RN5 pad 2: /MEMCS16 -> /IOCS16
- RN5 pad 3: /MASTER -> /MEMCS16
Routing:
- net +5V: track 501.9 -> 831.9 mm, vias 44 -> 59
- net /SPKR: track 7.18 -> 216.8 mm, vias 0 -> 2
- net /SA1: track 4.24 -> 142.6 mm, vias 2 -> 7
- net /SA0: track 4.23 -> 141.4 mm, vias 2 -> 6
- net /SA2: track 4.78 -> 141.6 mm, vias 2 -> 6
- net +12V: track 21.6 -> 118.6 mm, vias 2 -> 3
- net -12V: track 16.9 -> 111.1 mm, vias 2 -> 3
- net /LA23: track 0.00 -> 74.7 mm, vias 0 -> 2
- net +3V3: track 40.1 -> 112.3 mm
- net /LA20: track 0.00 -> 70.3 mm, vias 0 -> 2
- net /LA22: track 0.00 -> 70.3 mm, vias 0 -> 2
- net /LA19: track 0.00 -> 64.6 mm
- net /LA21: track 0.00 -> 64.0 mm, vias 0 -> 1
- net /KBDAT: track 6.79 -> 68.1 mm, vias 0 -> 1
- net /KBCLK: track 7.33 -> 67.0 mm, vias 0 -> 1
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- added copper zone on In2.Cu, net +5V
