File: pcb_main/rev.A/charon386_main.kicad_sch (KiCad schematic)
At the start: 86 parts, among them CON1 CF-CARD-cfcard, J1 Mini-DIN-6, J10 COM2, J11 ESP, J2 AudioJack3, J3 USB_B_Micro, J4 Mini-DIN-6, J5 DB15_Female_HighDensity_Mount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, J6 Conn_01x04, J7 PC104_16, J8 PC104, J9 COM1, Q1 BC817, SW1 SW_Push, SW2 Jumper / Pin header 1x2 Pitch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, U1 CH340G, U10 LT1930, U11 TXB0104PW, U12 XC9572XL-VQ64, U2 ESP-12E, U3 MSM5118160F-JS, U4 MSM5118160F-JS, U5 M6117D, U6 GD75232DB, U7 SST39SF040, U8 GD75232DB, U9 AMS1117-3.3, X1 50 MHz, Y1 12 MHz, Y2 32768 Hz

Commit message: wip pcb rev.A
Parts:
- removed C8: 10u, Capacitor_SMD:C_0805_2012Metric_Pad1.18x1.45mm_HandSolder, symbol Device:C
- removed J2: AudioJack3, Connector_Audio:Jack_3.5mm_CUI_SJ1-3535NG_Horizontal, symbol Connector:AudioJack3
- removed U12: XC9572XL-VQ64, Package_QFP:TQFP-64_10x10mm_P0.5mm, symbol CPLD_Xilinx:XC9572XL-VQ64
- removed U6, U8: GD75232DB, Package_SO:SSOP-20_4.4x6.5mm_P0.65mm, symbol Interface_UART:GD75232DB
- removed U7: SST39SF040, my:PLCC-32_11.4x14.0mm_P1.27mm-longpads, symbol Memory_Flash:SST39SF040
- added D6: LED_Blue, LED_THT:LED_D3.0mm_Horizontal_O1.27mm_Z6.0mm, symbol Device:LED
- added J12: Conn_02x07_Odd_Even, Connector_PinSocket_2.54mm:PinSocket_2x07_P2.54mm_Vertical, symbol Connector_Generic:Conn_02x07_Odd_Even
- added J2: PJ-320, my:PJ-322, symbol Connector:AudioJack4
- added Q2: BC856, Package_TO_SOT_SMD:SOT-23, symbol Transistor_BJT:BC856
- added R18: 470, Resistor_SMD:R_0603_1608Metric_Pad0.98x0.95mm_HandSolder, symbol Device:R
- added R5: 0, Resistor_SMD:R_0805_2012Metric_Pad1.20x1.40mm_HandSolder, symbol Device:R
- added U12: MAX823LEUK, Package_TO_SOT_SMD:SOT-23-5, symbol my:MAX823
- added U13: ST16C554, Package_QFP:LQFP-64_10x10mm_P0.5mm, symbol my:ST16C554-LQFP
- added U14: 74LS32, Package_SO:TSSOP-14_4.4x5mm_P0.65mm, symbol 74xx:74LS32
- added U15, U16: 74HCT138, Package_SO:TSSOP-16_4.4x5mm_P0.65mm, symbol 74xx:74LS138
- added U6, U8: GD75232PW, Package_SO:TSSOP-20_4.4x6.5mm_P0.65mm, symbol Interface_UART:GD75232PW
- added U7: 27C512PLCC, my:PLCC-32_11.4x14.0mm_P1.27mm-longpads, symbol Memory_EPROM:27C512PLCC
- added X2: 14.7456 MHz, Oscillator:Oscillator_SMD_SeikoEpson_SG8002CA-4Pin_7.0x5.0mm, symbol Oscillator:XO91
- added X3: 80 MHz, Oscillator:Oscillator_SMD_SeikoEpson_SG8002CA-4Pin_7.0x5.0mm, symbol Oscillator:XO91
- D1: value LED -> LED_Red
- D2: value LED -> LED_Green
- J1, J4: footprint 4x1md:Connector_Mini-DIN_Female_6Pin_2rows -> my:MINI_DIN_6_33PRIMARY
- J8: Field4 B A -> A B
- U5: symbol M6117D:M6117D -> my:M6117D
- X1: value 50 MHz -> 14.318 MHz
Connections:
- net A0 is gone; now on net SA0: J8.62 (Pin_62)
- net A1 is gone; now on net SA1: J8.60 (Pin_60)
- net A10 is gone; now on net SA10: J8.42 (Pin_42)
- net A11 is gone; now on net SA11: J8.40 (Pin_40)
- net A12 is gone; now on net SA12: J8.38 (Pin_38)
- net A13 is gone; now on net SA13: J8.36 (Pin_36)
- net A14 is gone; now on net SA14: J8.34 (Pin_34)
- net A15 is gone; now on net SA15: J8.32 (Pin_32)
- net A16 is gone; now on net SA16: J8.30 (Pin_30)
- net A17 is gone; now on net SA17: J8.28 (Pin_28)
- net A18 is gone; now on net SA18: J8.26 (Pin_26)
- net A19 is gone; now on net SA19: J8.24 (Pin_24)
- net A2 is gone; now on net SA2: J8.58 (Pin_58)
- net A3 is gone; now on net SA3: J8.56 (Pin_56)
- net A4 is gone; now on net SA4: J8.54 (Pin_54)
- net A5 is gone; now on net SA5: J8.52 (Pin_52)
- net A6 is gone; now on net SA6: J8.50 (Pin_50)
- net A7 is gone; now on net SA7: J8.48 (Pin_48)
- net A8 is gone; now on net SA8: J8.46 (Pin_46)
- net A9 is gone; now on net SA9: J8.44 (Pin_44)
- net ALE is gone; now on net BALE: J8.55 (Pin_55)
- net CLK is gone; now on net 14MHz: X1.3 (OUT)
- net D0 is gone; now on net SD0: J8.18 (Pin_18)
- net D1 is gone; now on net SD1: J8.16 (Pin_16)
- net D10 is gone; now on net SD10: J7.27 (Pin_27)
- net D11 is gone; now on net SD11: J7.29 (Pin_29)
- net D12 is gone; now on net SD12: J7.31 (Pin_31)
- net D13 is gone; now on net SD13: J7.33 (Pin_33)
- net D14 is gone; now on net SD14: J7.35 (Pin_35)
- net D15 is gone; now on net SD15: J7.37 (Pin_37)
- net D2 is gone; now on net SD2: J8.14 (Pin_14)
- net D3 is gone; now on net SD3: J8.12 (Pin_12)
- net D4 is gone; now on net SD4: J8.10 (Pin_10)
- net D5 is gone; now on net SD5: J8.8 (Pin_8)
- net D6 is gone; now on net SD6: J8.6 (Pin_6)
- net D7 is gone; now on net SD7: J8.4 (Pin_4)
- net D8 is gone; now on net SD8: J7.23 (Pin_23)
- net D9 is gone; now on net SD9: J7.25 (Pin_25)
- net OSC is gone; now on net 14MHz: J8.59 (Pin_59)
- net OWS is gone; now on net NOWS: RN4.3 (R3.1), U5.165 (NOWSJ)
- net RESET is gone; now on net RSTDRV: J8.3 (Pin_3)
- net ~IOR is gone; now on net IOR: J8.27 (Pin_27)
- net ~IOW is gone; now on net IOW: J8.25 (Pin_25)
- net ~MEMCS16 is gone; now on net MEMCS16: J7.4 (Pin_4)
- net ~MEMR is gone; now on net SMEMR: J8.23 (Pin_23)
- net ~MEMW is gone; now on net SMEMW: J8.21 (Pin_21)
- net ~NMI is gone; now on net IOCHCK: J8.2 (Pin_2)
- net ~REFRESH is gone; now on net REFRESH: J8.37 (Pin_37)
- net +12V: now also U6.1 (VDD), U8.1 (VDD)
- net +3V3: now also X3.1 (EN), X3.4 (V+)
- net +5V: now also R12.1, R13.1, U1.11 (~RI), R18.1, R5.1, U12.5 (VCC), U13.21 (VCC), U13.30 (RIC#), U13.35 (VCC), U13.4 (VCC), U13.46 (DTRD#), U13.48 (DSRD#), U13.49 (CDD#), U13.50 (RID#), U13.52 (VCC), U14.14 (VCC), U15.16 (VCC), U15.6 (E3), U16.16 (VCC), U6.20 (VCC), U7.32 (VCC), U8.20 (VCC), X2.1 (EN), X2.4 (V+); no longer R12.2, R13.2
- net -12V: now also U6.10 (VSS), U8.10 (VSS)
- net AEN: now also U16.5 (E2)
- net CLK2: now also X3.3 (OUT)
- net DACK0: now also J7.18 (Pin_18)
- net DACK1: now also J8.33 (Pin_33)
- net DACK5: now also J7.22 (Pin_22)
- net ESP_CTS: now also J11.7 (Pin_7), U2.7 (GPIO13); no longer U11.11 (B3)
- net ESP_RTS: now also J11.9 (Pin_9), U2.4 (GPIO16); no longer U11.10 (B4)
- net ESP_RX: now also J11.5 (Pin_5), U2.21 (GPIO3/RXD); no longer U11.12 (B2)
- net ESP_TX: now also J11.3 (Pin_3), U2.22 (GPIO1/TXD), Q2.1 (B); no longer U11.13 (B1)
- net GND: now also J10.5 (Pin_5), J9.5 (Pin_5), J12.11 (Pin_11), J12.12 (Pin_12), J12.3 (Pin_3), J12.4 (Pin_4), J12.7 (Pin_7), J2.R2, Q2.3 (C), U12.2 (GND), U13.14 (GND), U13.28 (GND), U13.45 (GND), U13.61 (GND), U14.1, U14.2, U14.7 (GND), U15.4 (E1), U15.5 (E2), U15.8 (GND), U16.8 (GND), U6.11 (GND), U7.16 (GND), U8.11 (GND), X2.2 (GND), X3.2 (GND); no longer J5.9
- net IOCS16: now also J7.6 (Pin_6)
- net IOR: now also RN8.4 (R4.1), U13.40 (IOR#)
- net IOW: now also U13.9 (IOW#)
- net IRQ10: now also J7.8 (Pin_8)
- net IRQ11: now also J7.10 (Pin_10)
- net IRQ14: now also J7.16 (Pin_16)
- net IRQ15: now also J7.14 (Pin_14)
- net IRQ3: now also J8.49 (Pin_49), U14.11
- net IRQ4: now also J8.47 (Pin_47), U14.8
- net IRQ5: now also J8.45 (Pin_45)
- net IRQ6: now also J8.43 (Pin_43)
- net IRQ7: now also J8.41 (Pin_41)
- net IRQ9: now also J8.7 (Pin_7)
- net KBSJ: now also RN7.8 (R1.2), U7.23 (~CE)
- net MASTER: now also J7.36 (Pin_36); no longer RN8.4 (R4.1)
- net MEMR: now also J7.19 (Pin_19), U7.25 (~OE~/VPP)
- net MEMW: now also J7.21 (Pin_21)
- net PWG: now also U12.1 (~RST)
- net RESETL: now also U11.13 (B1)
- net RSTDRV: now also U13.27 (RESET)
- net SA0: now also U13.24 (A0), U7.11 (A0)
- net SA1: now also U13.23 (A1), U7.10 (A1)
- net SA10: now also U7.24 (A10)
- net SA11: now also U7.27 (A11)
- net SA12: now also U7.3 (A12)
- net SA13: now also U7.30 (A13)
- net SA14: now also U7.31 (A14)
- net SA15: now also U7.2 (A15)
- net SA2: now also U13.22 (A2), U7.9 (A2)
- net SA3: now also U16.3 (A2), U7.8 (A3)
- net SA4: now also U16.2 (A1), U7.7 (A4)
- net SA5: now also U16.6 (E3), U7.6 (A5)
- net SA6: now also U15.1 (A0), U7.5 (A6)
- net SA7: now also U15.2 (A1), U7.4 (A7)
- net SA8: now also U16.1 (A0), U7.29 (A8)
- net SA9: now also U15.3 (A2), U7.28 (A9)
- net SD0: now also U13.53 (D0)
- net SD1: now also U13.54 (D1)
- net SD2: now also U13.55 (D2)
- net SD3: now also U13.56 (D3)
- net SD4: now also U13.57 (D4)
- net SD5: now also U13.58 (D5)
- net SD6: now also U13.59 (D6)
- net SD7: now also U13.60 (D7)
- net SYSCLK: now also J8.39 (Pin_39)
- net TC: now also J8.53 (Pin_53)
- net XD0: now also U7.13 (O0)
- net XD1: now also U7.14 (O1)
- net XD2: now also U7.15 (O2)
- net XD3: now also U7.18 (O3)
- net XD4: now also U7.19 (O4)
- net XD5: now also U7.20 (O5)
- net XD6: now also U7.21 (O6)
- net XD7: now also U7.22 (O7)
- net DTRC: now reaches U1.10 (~DSR)
- net DTRC: now also U1.12 (~DCD), U13.34 (DTRC#)
- net DSRC: now reaches U1.13 (~DTR)
- net DSRC: now also U13.31 (CDC#), U13.32 (DSRC#)
- net at U11.5 (A4): now also J11.8 (Pin_8); no longer J11.10 (Pin_10)
- net at J11.4 (Pin_4): now also U11.3 (A2); no longer U11.2 (A1)
- net at J11.6 (Pin_6): now also U11.4 (A3); no longer U11.3 (A2)
- net DCD2: now reaches J10.1 (Pin_1)
- net DCD2: now also U8.2 (RA1)
- net RX2: now reaches J10.2 (Pin_2)
- net RX2: now also U8.4 (RA3)
- net TX2: now reaches J10.3 (Pin_3)
- net TX2: now also U8.6 (DY2)
- net DTR2: now reaches J10.4 (Pin_4)
- net DTR2: now also U8.8 (DY3)
- net DSR2: now reaches J10.6 (Pin_6)
- net DSR2: now also U8.3 (RA2)
- net RTS2: now reaches J10.7 (Pin_7)
- net RTS2: now also U8.5 (DY1)
- net CTS2: now reaches J10.8 (Pin_8)
- net CTS2: now also U8.7 (RA4)
- net RI2: now reaches J10.9 (Pin_9)
- net RI2: now also U8.9 (RA5)
- net at D2.2 (A): now also R13.2; no longer R13.1
- net DRQ0: now reaches J7.20 (Pin_20)
- net DRQ0: now also U5.17 (DRQ0)
- net DRQ5: now reaches J7.24 (Pin_24)
- net DRQ5: now also U5.25 (DRQ5)
- net DACK6: now reaches J7.26 (Pin_26)
- net DACK6: now also U5.26 (DACK6J)
- net DRQ6: now reaches J7.28 (Pin_28)
- net DRQ6: now also U5.27 (DRQ6)
- net DACK7: now reaches J7.30 (Pin_30)
- net DACK7: now also U5.28 (DACK7J)
- net DRQ7: now reaches J7.32 (Pin_32)
- net DRQ7: now also U5.29 (DRQ7)
- net DRQ2: now reaches J8.11 (Pin_11)
- net DRQ2: now also U5.21 (DRQ2)
- net NOWS: now reaches J8.15 (Pin_15)
- net DACK3: now reaches J8.29 (Pin_29)
- net DACK3: now also U5.22 (DACK3J)
- net DRQ3: now reaches J8.31 (Pin_31)
- net DRQ3: now also U5.23 (DRQ3)
- net DRQ1: now reaches J8.35 (Pin_35)
- net DRQ1: now also U5.19 (DRQ1)
- net DACK2: now reaches J8.51 (Pin_51)
- net DACK2: now also U5.20 (DACK2J)
- net at D1.2 (A): now also R12.2; no longer R12.1
- net VGA_R: now reaches J5.1
- net VGA_R: now also J12.5 (Pin_5)
- net VGA_MON: now reaches J5.12
- net VGA_MON: now also J12.8 (Pin_8)
- net VGA_HS: now reaches J5.13
- net VGA_HS: now also J12.10 (Pin_10)
- net VGA_VS: now reaches J5.14
- net VGA_VS: now also J12.14 (Pin_14)
- net VGA_G: now reaches J5.2
- net VGA_G: now also J12.9 (Pin_9)
- net VGA_B: now reaches J5.3
- net VGA_B: now also J12.13 (Pin_13)
- net DCD1: now reaches J9.1 (Pin_1)
- net DCD1: now also U6.2 (RA1)
- net RX1: now reaches J9.2 (Pin_2)
- net RX1: now also U6.4 (RA3)
- net TX1: now reaches J9.3 (Pin_3)
- net TX1: now also U6.6 (DY2)
- net DTR1: now reaches J9.4 (Pin_4)
- net DTR1: now also U6.8 (DY3)
- net DSR1: now reaches J9.6 (Pin_6)
- net DSR1: now also U6.3 (RA2)
- net RTS1: now reaches J9.7 (Pin_7)
- net RTS1: now also U6.5 (DY1)
- net CTS1: now reaches J9.8 (Pin_8)
- net CTS1: now also U6.7 (RA4)
- net RI1: now reaches J9.9 (Pin_9)
- net RI1: now also U6.9 (RA5)
- net SER0_CTS renamed RTSC
- net RTSC: now also U13.36 (RTSC#)
- net SER0_RTS renamed CTSC
- net CTSC: now also U13.33 (CTSC#)
- net SER0_RX renamed RXC
- net RXC: now also U13.29 (RXC)
- net SER0_TX renamed TXC
- net TXC: now also U13.39 (TXC)
- net ~RESET renamed ESP_RST
- net ESP_RST: now also U11.2 (A1)
- net ~RST: no longer names the net of R10.2, SW1.1
- net ~RST: now also U12.3 (~MR)
- new net: J12.6 (Pin_6), J2.S
- new net: U15.7 (O7), U16.4 (E1)
- new net: J5.9, R5.2
- new net: U13.25 (XTAL1), X2.3 (OUT)
- new net: D6.1 (K), Q2.2 (E)
- new net: D6.2 (A), R18.2
- new net 0x2E8: U13.42 (CSD#), U16.11 (O4)
- new net 0x2F8: U13.11 (CSB#), U16.9 (O6)
- new net 0x3E8: U13.38 (CSC#), U16.10 (O5)
- new net 0x3F8: U13.7 (CSA#), U16.7 (O7)
- new net CDA: U13.64 (CDA#), U6.19 (RY1)
- new net CDB: U13.18 (CDB#), U8.19 (RY1)
- new net CTSA: U13.2 (CTSA#), U6.14 (RY4)
- new net CTSB: U13.16 (CTSB#), U8.14 (RY4)
- new net CTSD: J11.10 (Pin_10), U13.47 (CTSD#)
- new net DSRA: U13.1 (DSRA#), U6.18 (RY2)
- new net DSRB: U13.17 (DSRB#), U8.18 (RY2)
- new net DTRA: U13.3 (DTRA#), U6.13 (DA3)
- new net DTRB: U13.15 (DTRB#), U8.13 (DA3)
- new net RIA: U13.63 (RIA#), U6.12 (RY5)
- new net RIB: U13.19 (RIB#), U8.12 (RY5)
- new net RTSA: U13.5 (RTSA#), U6.16 (DA1)
- new net RTSB: U13.13 (RTSB#), U8.16 (DA1)
- new net RTSD: U11.10 (B4), U13.44 (RTSD#)
- new net RXA: U13.62 (RXA), U6.17 (RY3)
- new net RXB: U13.20 (RXB), U8.17 (RY3)
- new net RXD: U11.12 (B2), U13.51 (RXD)
- new net SND_L: J12.1 (Pin_1), J2.T
- new net SND_R: J12.2 (Pin_2), J2.R1
- new net TXA: U13.8 (TXA), U6.15 (DA2)
- new net TXB: U13.10 (TXB), U8.15 (DA2)
- new net TXD: U11.11 (B3), U13.41 (TXD)
- new net UART_INTA: U13.6 (INTA), U14.9
- new net UART_INTB: U13.12 (INTB), U14.12
- new net UART_INTC: U13.37 (INTC), U14.10
- new net UART_INTD: U13.43 (INTD), U14.13
- no-connect marks 109 -> 90
Other:
- note added: "COM (UART)"
- note added: "Compact Flash"
- note added: "PC/104"
- note added: "RAM 2Mb"
- note added: "ROM"
- moved on the sheet: BT1, C1, C10, C11, C12, C13, C14, C15, C16, C17, C2, C3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

Commit message: wip pcb rev.A
Parts:
- removed RN7: 4.7k, Resistor_SMD:R_Array_Convex_4x0603, symbol Device:R_Pack04
- removed X2: 14.7456 MHz, Oscillator:Oscillator_SMD_SeikoEpson_SG8002CA-4Pin_7.0x5.0mm, symbol Oscillator:XO91
- added C18, C19, C52, C53, C54, C55: 10u, Capacitor_SMD:C_0805_2012Metric_Pad1.18x1.45mm_HandSolder, symbol Device:C
- added C20, C21, C22, C23, C24, C25, C26, C27, C28, C29, C30, C31, C32, C33, C34, C35, C36, C37, C38, C39, C40, C41, C42, C43, C44, C45, C46, C48, C49, C50, C51, C56: 100n, Capacitor_SMD:C_0603_1608Metric_Pad1.08x0.95mm_HandSolder, symbol Device:C
- added C57, C58: 22p, Capacitor_SMD:C_0603_1608Metric_Pad1.08x0.95mm_HandSolder, symbol Device:C
- added C8: 47u, Capacitor_SMD:CP_Elec_5x5.9, symbol Device:CP
- added D7: BZV55C5V6, Diode_SMD:D_MiniMELF, symbol Device:D_Zener
- added D8: BT168GW, Package_TO_SOT_SMD:SOT-223-3_TabPin2, symbol Device:Q_SCR_KAG
- added R16, R17, R19: 22, Resistor_SMD:R_0603_1608Metric_Pad0.98x0.95mm_HandSolder, symbol Device:R
- added R20: 4.7k, Resistor_SMD:R_0603_1608Metric_Pad0.98x0.95mm_HandSolder, symbol Device:R
- added R21: 1k, Resistor_SMD:R_0603_1608Metric_Pad0.98x0.95mm_HandSolder, symbol Device:R
- added Y3: 14.7456 MHz, Crystal:Crystal_SMD_SeikoEpson_TSX3225-4Pin_3.2x2.5mm_HandSoldering, symbol Device:Crystal_GND24
- J2: value PJ-320 -> PJ-322
- U14: value 74LS32 -> 74HCT32
Connections:
- net +12V: now also C40.2, C41.2
- net +3V3: now also C19.2, C45.2, C46.2; no longer X1.1 (EN), X1.4 (V+), X3.1 (EN), X3.4 (V+)
- net +5V: now also X1.1 (EN), X1.4 (V+), X3.1 (EN), X3.4 (V+), C18.2, C20.2, C21.2, C22.2, C23.2, C24.2, C25.2, C26.2, C27.2, C28.2, C29.2, C30.2, C31.2, C32.2, C33.2, C34.2, C35.2, C36.2, C37.2, C38.2, C39.2, C44.2, C48.2, C49.2, C50.2, C51.2, C52.1, C53.1, C54.1, C55.1, C56.1, C8.1, D7.1 (K), D8.2 (A); no longer U13.46 (DTRD#), U13.48 (DSRD#), U13.49 (CDD#)
- net -12V: now also C42.2, C43.2
- net 14MHz: now also R16.2, R17.2; no longer J8.59 (Pin_59), U5.117 (OSC14M)
- net CLK2: now also R19.2; no longer U5.39 (BCLK2)
- net DACK0: now also RN6.7 (R2.2); no longer RN6.8 (R1.2)
- net DACK1: now also RN6.6 (R3.2); no longer RN6.7 (R2.2)
- net DACK5: now also RN6.5 (R4.2); no longer RN6.6 (R3.2)
- net GND: now also C18.1, C19.1, C20.1, C21.1, C22.1, C23.1, C24.1, C25.1, C26.1, C27.1, C28.1, C29.1, C30.1, C31.1, C32.1, C33.1, C34.1, C35.1, C36.1, C37.1, C38.1, C39.1, C40.1, C41.1, C42.1, C43.1, C44.1, C45.1, C46.1, C48.1, C49.1, C50.1, C51.1, C52.2, C53.2, C54.2, C55.2, C56.2, C57.2, C58.2, C8.2, D8.1 (K), R20.1, R21.2, Y3.2, Y3.4; no longer J6.3 (Pin_3)
- net KBSJ: now also R20.2
- net MEMR: now also RN3.4 (R4.1); no longer RN3.2 (R2.1)
- net MEMW: now also RN3.3 (R3.1); no longer RN3.1 (R1.1)
- net NOWS: now also RN4.1 (R1.1); no longer RN4.3 (R3.1)
- net REFRESH: now also RN4.3 (R3.1); no longer RN4.1 (R1.1)
- net TC: now also RN6.8 (R1.2); no longer RN6.5 (R4.2)
- net at U13.25 (XTAL1): now also C57.1, Y3.3
- net at U13.26 (XTAL2): now also C58.1, Y3.1
- new net: R17.1, U5.117 (OSC14M)
- new net: J8.59 (Pin_59), R16.1
- new net: U13.46 (DTRD#), U13.48 (DSRD#), U13.49 (CDD#)
- new net: D7.2 (A), D8.3 (G), R21.1
- new net: R19.1, U5.39 (BCLK2)
- no-connect marks 90 -> 92
Other:
- note added: "LED"
- note added: "Power"
- moved on the sheet: BT1, C10, C11, C12, C13, C14, C15, C16, C17, C2, C3, C4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

Commit message: wip pcb rev.A
Parts:
- J12: footprint Connector_PinSocket_2.54mm:PinSocket_2x07_P2.54mm_Vertical -> Connector_PinSocket_2.54mm:PinSocket_2x08_P2.54mm_Vertical; symbol Connector_Generic:Conn_02x07_Odd_Even -> Connector_Generic:Conn_02x08_Odd_Even
Connections:
- net GND: now also U14.4, U14.5
- net SPKR: now also J12.16 (Pin_16)
- no-connect marks 92 -> 84
Other:
- moved on the sheet: C1, C2, C3, C57, C58, J10, J11, J9, R8, U1, U11, U13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

Commit message: wip pcb rev.A
Parts:
- removed D4: BAT54S, Package_TO_SOT_SMD:SOT-23, symbol Diode:BAT54S
- added C?: 10p, Capacitor_SMD:C_0805_2012Metric_Pad1.18x1.45mm_HandSolder, symbol Device:C
- added D4, D9: MBR0520, Diode_SMD:D_SOD-123, symbol Diode:MBR0520
- added R22: 51k, Resistor_SMD:R_0603_1608Metric_Pad0.98x0.95mm_HandSolder, symbol Device:R
- C15: footprint Capacitor_SMD:C_0603_1608Metric_Pad1.08x0.95mm_HandSolder -> Capacitor_SMD:C_0805_2012Metric_Pad1.18x1.45mm_HandSolder
- L1: value L -> 10u; footprint Inductor_SMD:L_0805_2012Metric_Pad1.15x1.40mm_HandSolder -> Inductor_THT:L_Radial_D9.5mm_P5.00mm_Fastron_07HVP
- R14: value R -> 113k
- R15: value R -> 13.3k
Connections:
- net +12V: now also C?.1
- net +5V: now also R22.1; no longer U10.4 (~SHDN)
- net -12V: now also D9.2 (A)
- net GND: now also D4.1 (K)
- net at R14.2, R15.1, U10.3 (FB): now also C?.2
- net at C15.2: now also D4.2 (A), D9.1 (K)
- new net: R22.2, U10.4 (~SHDN)
Other:
- note added: "1.1A"
- note added: "19mA"
- note added: "20mA"
- note added: "215mA"
- note added: "290mA"
- note added: "2A"
- note added: "300mA"
- note added: "30mA"
- note added: "40mA"
- note added: "6mA"
- note added: "800mA"
- moved on the sheet: BT1, C13, C14, C16, C17, C18, C19, D5, R14, R15, U9

Commit message: wip pcb rev.A
Parts:
- removed H5, H6, H7, H8: MountingHole, my:MountingHole_3.2mm_M3_dk5.2mm_Mask, symbol Mechanical:MountingHole
- added LOGO1: (no value), symbol my:logo
- added N1: G738 or G706, symbol Mechanical:Housing
- C47: renamed from C?; footprint Capacitor_SMD:C_0805_2012Metric_Pad1.18x1.45mm_HandSolder -> Capacitor_SMD:C_0603_1608Metric_Pad1.08x0.95mm_HandSolder
- C8: symbol Device:CP -> Device:C_Polarized
- H1, H2, H3, H4: value MountingHole -> Screw M3 dk=5mm L=4mm
Connections:
- net ~CF_BUSY renamed ~{CF_BUSY}
Other:
- moved on the sheet: H1, H2, H3, H4

Commit message: wip pcb rev.A
Parts:
- removed Y2: 32768 Hz, Crystal:Crystal_C38-LF_D3.0mm_L8.0mm_Horizontal_1EP_style2, symbol Device:Crystal_GND3
- removed Y3: 14.7456 MHz, Crystal:Crystal_SMD_SeikoEpson_TSX3225-4Pin_3.2x2.5mm_HandSoldering, symbol Device:Crystal_GND24
- added C59, C60, C61, C62, C63, C64, C65, C66, C67, C68: 1u, Capacitor_SMD:C_0603_1608Metric_Pad1.08x0.95mm_HandSolder, symbol Device:C
- added C69, C70, C71, C72, C73: 100n, Capacitor_SMD:C_0603_1608Metric_Pad1.08x0.95mm_HandSolder, symbol Device:C
- added X2: 1.8432 Mhz, Oscillator:Oscillator_SMD_SeikoEpson_SG8002CA-4Pin_7.0x5.0mm, symbol Oscillator:XO91
- added Y2: 32768 Hz, Crystal:Crystal_SMD_SeikoEpson_MC306-4Pin_8.0x3.2mm_HandSoldering, symbol Device:Crystal_GND23
- C57: value 22p -> 100n
- C58: value 22p -> 1u
- C8: value 47u -> 100u; footprint Capacitor_SMD:CP_Elec_5x5.9 -> Capacitor_Tantalum_SMD:CP_EIA-7343-31_Kemet-D_Pad2.25x2.55mm_HandSolder
- L1: footprint Inductor_THT:L_Radial_D9.5mm_P5.00mm_Fastron_07HVP -> Inductor_SMD:L_Taiyo-Yuden_NR-60xx_HandSoldering
- LOGO1: value (none) -> graphic; footprint (none) -> mygraphic:black-mage-12.5x8.6
- R5: footprint Resistor_SMD:R_0805_2012Metric_Pad1.20x1.40mm_HandSolder -> Resistor_SMD:R_0603_1608Metric_Pad0.98x0.95mm_HandSolder
- U7: value 27C512PLCC -> 27C512
Connections:
- net IOCHCK is gone; now on net IOCHK: J8.2 (Pin_2), U5.196 (IOCHKJ)
- net +3V3: now also D5.1; no longer D5.2
- net +5V: now also C57.1, C58.2, C59.2, C60.2, C61.2, C62.2, C63.2, C64.1, C65.1, C66.1, C67.1, C68.1, C69.1, C70.1, C71.1, C72.1, C73.1, X2.1 (EN), X2.4 (V+)
- net AEN: now also RN3.1 (R1.1)
- net CDA: now also U6.17 (RY3); no longer U6.19 (RY1)
- net CDB: now also U8.17 (RY3); no longer U8.19 (RY1)
- net CTS1: now also U6.9 (RA5); no longer U6.7 (RA4)
- net CTS2: now also U8.2 (RA1); no longer U8.7 (RA4)
- net CTSA: now also U6.12 (RY5); no longer U6.14 (RY4)
- net CTSB: now also U8.19 (RY1); no longer U8.14 (RY4)
- net CTSC: now also J11.10 (Pin_10); no longer U1.14 (~{RTS})
- net CTSD: now also U1.14 (~{RTS}); no longer J11.10 (Pin_10)
- net DCD1: now also U6.4 (RA3); no longer U6.2 (RA1)
- net DCD2: now also U8.4 (RA3); no longer U8.2 (RA1)
- net DSR1: now also U6.7 (RA4); no longer U6.3 (RA2)
- net DSRA: now also U6.14 (RY4); no longer U6.18 (RY2)
- net DTR1: now also U6.5 (DY1); no longer U6.8 (DY3)
- net DTRA: now also U6.16 (DA1); no longer U6.13 (DA3)
- net GND: now also C58.1, C59.1, C60.1, C61.1, C62.1, C63.1, C64.2, C65.2, C66.2, C67.2, C68.2, C69.2, C70.2, C71.2, C72.2, C73.2, X2.2 (GND), Y2.2, Y2.3; no longer C58.2
- net IOCHK: now also RN5.4 (R4.1); no longer RN5.3 (R3.1)
- net IOCS16: now also RN5.1 (R1.1); no longer RN5.2 (R2.1)
- net MASTER: now also RN5.3 (R3.1); no longer RN5.4 (R4.1)
- net MEMCS16: now also RN5.2 (R2.1); no longer RN5.1 (R1.1)
- net RI1: now also U6.3 (RA2); no longer U6.9 (RA5)
- net RI2: now also U8.7 (RA4); no longer U8.9 (RA5)
- net RIA: now also U6.18 (RY2); no longer U6.12 (RY5)
- net RIB: now also U8.14 (RY4); no longer U8.12 (RY5)
- net RTS1: now also U6.6 (DY2); no longer U6.5 (DY1)
- net RTS2: now also U8.6 (DY2); no longer U8.5 (DY1)
- net RTSA: now also U6.15 (DA2); no longer U6.16 (DA1)
- net RTSB: now also U8.15 (DA2); no longer U8.16 (DA1)
- net RTSC: now also U11.10 (B4); no longer U1.9 (~{CTS})
- net RTSD: now also U1.9 (~{CTS}); no longer U11.10 (B4)
- net RX1: now also U6.2 (RA1); no longer U6.4 (RA3)
- net RX2: now also U8.9 (RA5); no longer U8.4 (RA3)
- net RXA: now also U6.19 (RY1); no longer U6.17 (RY3)
- net RXB: now also U8.12 (RY5); no longer U8.17 (RY3)
- net RXC: now also U11.12 (B2); no longer U1.2 (TXD)
- net RXD: now also U1.2 (TXD); no longer U11.12 (B2)
- net TX1: now also U6.8 (DY3); no longer U6.6 (DY2)
- net TX2: now also U8.5 (DY1); no longer U8.6 (DY2)
- net TXA: now also U6.13 (DA3); no longer U6.15 (DA2)
- net TXB: now also U8.16 (DA1); no longer U8.15 (DA2)
- net TXC: now also U11.11 (B3); no longer U1.3 (RXD)
- net TXD: now also U1.3 (RXD); no longer U11.11 (B3)
- net at BT1.1 (+): now also D5.2; no longer D5.1
- net at U13.25 (XTAL1): now also X2.3 (OUT); no longer C57.1
- net at U13.26 (XTAL2): no longer C58.1
- net DSRD: now reaches U13.48 (DSRD#), U13.49 (CDD#)
- net DSRD: now also U1.13 (~{DTR}); no longer U13.46 (DTRD#)
- net at C6.1, R4.1, U5.111 (XTAL1): now also Y2.1
- net at C7.1, R4.2, U5.112 (XTAL2): now also Y2.4
- net DSRC: no longer names the net of U13.31 (CDC#), U13.32 (DSRC#)
- net DSRC: now also U13.34 (DTRC#); no longer U1.13 (~{DTR})
- net DTRC renamed DTRD
- net DTRD: now also U13.46 (DTRD#); no longer U13.34 (DTRC#)
Other:
- moved on the sheet: C6, C7, D5

Commit message: wip pcb rev.A
Parts:
- removed C50: 100n, Capacitor_SMD:C_0603_1608Metric_Pad1.08x0.95mm_HandSolder, symbol Device:C
- removed R9: 4.7k, Resistor_SMD:R_0603_1608Metric_Pad0.98x0.95mm_HandSolder, symbol Device:R
- J1, J4: footprint my:MINI_DIN_6_33PRIMARY -> my:minidin-6; symbol Connector:Mini-DIN-6 -> my:Mini-DIN-6
Connections:
- net +5V: now also D1.2 (A), D2.2 (A), D6.2 (A); no longer R12.1, R13.1, R18.1
- net BD0: now also U3.10 (DQ7), U4.10 (DQ7); no longer U3.2 (DQ0), U4.2 (DQ0)
- net BD1: now also U3.9 (DQ6), U4.9 (DQ6); no longer U3.3 (DQ1), U4.3 (DQ1)
- net BD2: now also U3.8 (DQ5), U4.8 (DQ5); no longer U3.4 (DQ2), U4.4 (DQ2)
- net BD3: now also U3.7 (DQ4), U4.7 (DQ4); no longer U3.5 (DQ3), U4.5 (DQ3)
- net BD4: now also U3.5 (DQ3), U4.5 (DQ3); no longer U3.7 (DQ4), U4.7 (DQ4)
- net BD5: now also U3.4 (DQ2), U4.4 (DQ2); no longer U3.8 (DQ5), U4.8 (DQ5)
- net BD6: now also U3.3 (DQ1), U4.3 (DQ1); no longer U3.9 (DQ6), U4.9 (DQ6)
- net BD7: now also U3.2 (DQ0), U4.2 (DQ0); no longer U3.10 (DQ7), U4.10 (DQ7)
- net ESP_RST: now also U11.5 (A4); no longer U11.2 (A1)
- net GND: now also J1.0, J4.0, R13.2; no longer D2.1 (K)
- net RESETL: now also U11.10 (B4); no longer U11.13 (B1)
- net RTSC: now also U11.11 (B3); no longer U11.10 (B4)
- net RXC: now also U11.13 (B1); no longer U11.12 (B2)
- net TXC: now also U11.12 (B2); no longer U11.11 (B3)
- net ~{CF_BUSY}: now also R12.2; no longer D1.1 (K)
- net at C3.1, Y1.3: now also U1.8 (XO); no longer U1.7 (XI)
- net at C2.1, Y1.1: now also U1.7 (XI); no longer U1.8 (XO)
- net at J11.4 (Pin_4): now also U11.2 (A1); no longer U11.3 (A2)
- net at J11.6 (Pin_6): now also U11.3 (A2); no longer U11.4 (A3)
- net at J11.8 (Pin_8): now also U11.4 (A3); no longer U11.5 (A4)
- net at Q2.2 (E): now also R18.2; no longer D6.1 (K)
- new net: D2.1 (K), R13.1
- new net: D1.1 (K), R12.1
- new net: D6.1 (K), R18.1
- no-connect marks 84 -> 87
Other:
- moved on the sheet: C2, C3, D1, D2, D6, R12, R13, R18

Commit message: wip pcb rev.A
Connections:
- net +5V: now also U13.19 (RIB#), U13.63 (RIA#); no longer U13.30 (RIC#), U13.50 (RID#)
- net 0x2E8: now also U13.7 (CSA#), U15.11 (O4); no longer U13.42 (CSD#), U16.11 (O4)
- net 0x2F8: now also U13.42 (CSD#), U15.9 (O6); no longer U13.11 (CSB#), U16.9 (O6)
- net 0x3E8: now also U13.11 (CSB#), U15.10 (O5); no longer U13.38 (CSC#), U16.10 (O5)
- net 0x3F8: now also U13.38 (CSC#), U15.7 (O7); no longer U13.7 (CSA#), U16.7 (O7)
- net GND: now also CON1.S1 (Shield), CON1.S2 (Shield), U16.4 (E1); no longer U15.4 (E1)
- net SA3: now also U15.3 (A2); no longer U16.3 (A2)
- net SA4: now also U15.2 (A1); no longer U16.2 (A1)
- net SA6: now also U16.1 (A0); no longer U15.1 (A0)
- net SA7: now also U16.2 (A1); no longer U15.2 (A1)
- net SA8: now also U15.1 (A0); no longer U16.1 (A0)
- net SA9: now also U16.3 (A2); no longer U15.3 (A2)
- net CDA: no longer names the net of U13.64 (CDA#)
- net CDA: now also U13.1 (DSRA#), U13.3 (DTRA#); no longer U6.17 (RY3)
- net CDB renamed CD_COM2
- net CD_COM2: now also U13.49 (CDD#); no longer U13.18 (CDB#)
- net CTSA renamed CTS_COM1
- net CTS_COM1: now also U13.33 (CTSC#); no longer U13.2 (CTSA#)
- net CTSB renamed CTS_COM2
- net CTS_COM2: now also U13.47 (CTSD#); no longer U13.16 (CTSB#)
- net CTSC renamed CTS_ESP
- net CTS_ESP: now also U13.2 (CTSA#); no longer U13.33 (CTSC#)
- net CTSD renamed CTS_USB
- net CTS_USB: now also U13.16 (CTSB#); no longer U13.47 (CTSD#)
- net DSRA renamed DSR_COM1
- net DSR_COM1: now also U13.32 (DSRC#); no longer U13.1 (DSRA#)
- net DSRB renamed DSR_COM2
- net DSR_COM2: now also U13.48 (DSRD#); no longer U13.17 (DSRB#)
- removed net DSRD: U1.13 (~{DTR}), U13.48 (DSRD#), U13.49 (CDD#)
- net DTRA renamed DTR_COM1
- net DTR_COM1: now also U13.34 (DTRC#); no longer U13.3 (DTRA#)
- net DTRB renamed DTR_COM2
- net DTR_COM2: now also U13.46 (DTRD#); no longer U13.15 (DTRB#)
- net DTRD renamed DTR_USB
- net DTR_USB: now also U13.15 (DTRB#); no longer U13.46 (DTRD#)
- net RIA renamed RI_COM1
- net RI_COM1: now also U13.30 (RIC#); no longer U13.63 (RIA#)
- net RIB renamed RI_COM2
- net RI_COM2: now also U13.50 (RID#); no longer U13.19 (RIB#)
- net RTSA renamed RTS_COM1
- net RTS_COM1: now also U13.36 (RTSC#); no longer U13.5 (RTSA#)
- net RTSB renamed RTS_COM2
- net RTS_COM2: now also U13.44 (RTSD#); no longer U13.13 (RTSB#)
- net RTSC renamed RTS_ESP
- net RTS_ESP: now also U13.5 (RTSA#); no longer U13.36 (RTSC#)
- net RTSD renamed RTS_USB
- net RTS_USB: now also U13.13 (RTSB#); no longer U13.44 (RTSD#)
- net RXA renamed RX_COM1
- net RX_COM1: now also U13.29 (RXC); no longer U13.62 (RXA)
- net RXB renamed RX_COM2
- net RX_COM2: now also U13.51 (RXD); no longer U13.20 (RXB)
- net RXC renamed RX_ESP
- net RX_ESP: now also U13.62 (RXA); no longer U13.29 (RXC)
- net RXD renamed RX_USB
- net RX_USB: now also U13.20 (RXB); no longer U13.51 (RXD)
- net TXA renamed TX_COM1
- net TX_COM1: now also U13.39 (TXC); no longer U13.8 (TXA)
- net TXB renamed TX_COM2
- net TX_COM2: now also U13.41 (TXD); no longer U13.10 (TXB)
- net TXC renamed TX_ESP
- net TX_ESP: now also U13.8 (TXA); no longer U13.39 (TXC)
- net TXD renamed TX_USB
- net TX_USB: now also U13.10 (TXB); no longer U13.41 (TXD)
- net USB_DM renamed USB_DN
- new net: U15.4 (E1), U16.7 (O7)
- new net CD_COM1: U13.31 (CDC#), U6.17 (RY3)
- new net DSR_USB: U1.13 (~{DTR}), U13.17 (DSRB#), U13.18 (CDB#)
- no-connect marks 87 -> 85
Other:
- note added: "COM1: I/O port 0x3F8, IRQ 4 COM2: I/O port 0x2F8, IRQ 3 COM3: I/O port 0x3E8, IRQ 4 - USB COM4: I/O port 0x2E8, IRQ 3 - WiFi"
- moved on the sheet: U15, U16
