File: pcb_main/rev.A/charon386_main.kicad_sch (KiCad schematic)
At the start: 157 parts, among them CON1 CF-CARD-cfcard, J1 Mini-DIN-6, J10 COM2, J11 ESP, J12 Conn_02x07_Odd_Even, J2 PJ-322, J3 USB_B_Micro, J4 Mini-DIN-6, J5 DB15_Female_HighDensity_Mount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, J6 Conn_01x04, J7 PC104_16, J8 PC104, J9 COM1, Q1 BC817, Q2 BC856, SW1 SW_Push, SW2 Jumper / Pin header 1x2 Pitch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, U1 CH340G, U10 LT1930, U11 TXB0104PW, U12 MAX823LEUK, U13 ST16C554, U14 74HCT32, U15 74HCT138, U16 74HCT138, U2 ESP-12E, U3 MSM5118160F-JS, U4 MSM5118160F-JS, U5 M6117D, U6 GD75232PW, U7 27C512, U8 GD75232PW, U9 AMS1117-3.3, X1 14.318 MHz, X2 1.8432 Mhz, X3 80 MHz, Y1 12 MHz, Y2 32768 Hz

Commit message: wip pcb rev.A
Other:
- company: (none) -> Eugene Lozovoy
- title: (none) -> PC-CHARON-386-MAIN
Changed lines of the file:
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@@
   (paper "A2")
   (title_block
+    (title "PC-CHARON-386-MAIN")
     (date "2021-12-17")
     (rev "A")
+    (company "Eugene Lozovoy")
+    (comment 1 "Miniature 386 IBMPC-compatible computer")
   )
   (junction (at 565.785 36.83) (diameter 1.016) (color 0 0 0 0)
@@
     (effects (font (size 1 1)) (justify left bottom))
   )
-  (label "ESP_RST" (at 318.77 349.25 180)
+  (label "ESP_RST" (at 319.405 349.25 180)
     (effects (font (size 1 1)) (justify right bottom))
   )

Commit message: wip pcb rev.A
Connections:
- net IOCS16: now also RN5.2 (R2.1); no longer RN5.1 (R1.1)
- net MASTER: now also RN5.1 (R1.1); no longer RN5.3 (R3.1)
- net MEMCS16: now also RN5.3 (R3.1); no longer RN5.2 (R2.1)
- net MEMR: now also RN3.3 (R3.1); no longer RN3.4 (R4.1)
- net MEMW: now also RN3.4 (R4.1); no longer RN3.3 (R3.1)
- net SD0: now also RN2.4 (R4.1); no longer RN1.1 (R1.1)
- net SD1: now also RN2.3 (R3.1); no longer RN1.2 (R2.1)
- net SD2: now also RN2.2 (R2.1); no longer RN1.3 (R3.1)
- net SD3: now also RN2.1 (R1.1); no longer RN1.4 (R4.1)
- net SD4: now also RN1.4 (R4.1); no longer RN2.1 (R1.1)
- net SD5: now also RN1.3 (R3.1); no longer RN2.2 (R2.1)
- net SD6: now also RN1.2 (R2.1); no longer RN2.3 (R3.1)
- net SD7: now also RN1.1 (R1.1); no longer RN2.4 (R4.1)
Changed lines of the file:
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@@
     (stroke (width 0) (type solid) (color 0 0 0 0))
   )
-  (wire (pts (xy 146.685 69.85) (xy 140.335 69.85))
+  (wire (pts (xy 146.685 52.07) (xy 140.335 52.07))
     (stroke (width 0) (type solid) (color 0 0 0 0))
   )
@@
     (stroke (width 0) (type solid) (color 0 0 0 0))
   )
-  (wire (pts (xy 146.685 49.53) (xy 140.335 49.53))
+  (wire (pts (xy 146.685 72.39) (xy 140.335 72.39))
     (stroke (width 0) (type solid) (color 0 0 0 0))
   )
@@
     (stroke (width 0) (type solid) (color 0 0 0 0))
   )
-  (wire (pts (xy 146.685 57.15) (xy 140.335 57.15))
+  (wire (pts (xy 146.685 64.77) (xy 140.335 64.77))
     (stroke (width 0) (type solid) (color 0 0 0 0))
   )
@@
     (stroke (width 0) (type solid) (color 0 0 0 0))
   )
-  (wire (pts (xy 146.685 52.07) (xy 140.335 52.07))
+  (wire (pts (xy 146.685 69.85) (xy 140.335 69.85))
     (stroke (width 0) (type solid) (color 0 0 0 0))
   )
@@
     (stroke (width 0) (type solid) (color 0 0 0 0))
   )
-  (wire (pts (xy 146.685 64.77) (xy 140.335 64.77))
+  (wire (pts (xy 146.685 57.15) (xy 140.335 57.15))
     (stroke (width 0) (type solid) (color 0 0 0 0))
   )
@@
     (stroke (width 0) (type solid) (color 0 0 0 0))
   )
-  (wire (pts (xy 139.065 153.67) (xy 146.685 153.67))
+  (wire (pts (xy 140.335 153.67) (xy 146.685 153.67))
     (stroke (width 0) (type default) (color 0 0 0 0))
   )
@@
     (stroke (width 0) (type solid) (color 0 0 0 0))
   )
-  (wire (pts (xy 146.685 54.61) (xy 140.335 54.61))
+  (wire (pts (xy 146.685 67.31) (xy 140.335 67.31))
     (stroke (width 0) (type solid) (color 0 0 0 0))
   )
@@
     (stroke (width 0) (type solid) (color 0 0 0 0))
   )
-  (wire (pts (xy 146.685 67.31) (xy 140.335 67.31))
+  (wire (pts (xy 146.685 54.61) (xy 140.335 54.61))
     (stroke (width 0) (type solid) (color 0 0 0 0))
   )
@@
     (stroke (width 0) (type solid) (color 0 0 0 0))
   )
-  (wire (pts (xy 146.685 72.39) (xy 140.335 72.39))
+  (wire (pts (xy 146.685 49.53) (xy 140.335 49.53))
     (stroke (width 0) (type solid) (color 0 0 0 0))
   )
@@
     (effects (font (size 1 1)) (justify right bottom))
   )
-  (label "MEMR" (at 140.335 161.29 0)
+  (label "MEMR" (at 140.335 158.75 0)
     (effects (font (size 1 1)) (justify left bottom))
   )
@@
     (effects (font (size 1 1)) (justify left bottom))
   )
-  (label "SD5" (at 140.335 67.31 0)
+  (label "SD5" (at 140.335 54.61 0)
     (effects (font (size 1 1)) (justify left bottom))
   )
@@
     (effects (font (size 1 1)) (justify right bottom))
   )
-  (label "SD4" (at 140.335 64.77 0)
+  (label "SD4" (at 140.335 57.15 0)
     (effects (font (size 1 1)) (justify left bottom))
   )
@@
     (effects (font (size 1 1)) (justify right bottom))
   )
-  (label "MASTER" (at 140.335 189.23 0)
+  (label "MASTER" (at 140.335 184.15 0)
     (effects (font (size 1 1)) (justify left bottom))
   )
@@
     (effects (font (size 1 1)) (justify left bottom))
   )
-  (label "IOCS16" (at 140.335 184.15 0)
+  (label "IOCS16" (at 140.335 186.69 0)
     (effects (font (size 1 1)) (justify left bottom))
   )
@@
     (effects (font (size 1 1)) (justify left bottom))
   )
-  (label "SD3" (at 140.335 57.15 0)
+  (label "SD3" (at 140.335 64.77 0)
     (effects (font (size 1 1)) (justify left bottom))
   )
@@
     (effects (font (size 1 1)) (justify left bottom))
   )
-  (label "SD1" (at 140.335 52.07 0)
+  (label "SD1" (at 140.335 69.85 0)
     (effects (font (size 1 1)) (justify left bottom))
   )
@@
     (effects (font (size 1.27 1.27)) (justify right bottom))
   )
-  (label "SD2" (at 140.335 54.61 0)
+  (label "SD2" (at 140.335 67.31 0)
     (effects (font (size 1 1)) (justify left bottom))
   )
@@
     (effects (font (size 1 1)) (justify left bottom))
   )
-  (label "AEN" (at 139.065 153.67 0)
+  (label "AEN" (at 140.335 153.67 0)
     (effects (font (size 1 1)) (justify left bottom))
   )
@@
     (effects (font (size 1 1)) (justify right bottom))
   )
-  (label "MEMCS16" (at 140.335 186.69 0)
+  (label "MEMCS16" (at 140.335 189.23 0)
     (effects (font (size 1 1)) (justify left bottom))
   )
@@
     (effects (font (size 1 1)) (justify right bottom))
   )
-  (label "MEMW" (at 140.335 158.75 0)
+  (label "MEMW" (at 140.335 161.29 0)
     (effects (font (size 1 1)) (justify left bottom))
   )
@@
     (effects (font (size 1 1)) (justify left bottom))
   )
-  (label "SD7" (at 140.335 72.39 0)
+  (label "SD7" (at 140.335 49.53 0)
     (effects (font (size 1 1)) (justify left bottom))
   )
@@
     (effects (font (size 1 1)) (justify left bottom))
   )
-  (label "SD6" (at 140.335 69.85 0)
+  (label "SD6" (at 140.335 52.07 0)
     (effects (font (size 1 1)) (justify left bottom))
   )
@@
     (effects (font (size 1.27 1.27)) (justify right bottom))
   )
-  (label "SD0" (at 140.335 49.53 0)
+  (label "SD0" (at 140.335 72.39 0)
     (effects (font (size 1 1)) (justify left bottom))
   )

Commit message: wip pcb rev.A
Parts:
- removed C19: 10u, Capacitor_SMD:C_0805_2012Metric_Pad1.18x1.45mm_HandSolder, symbol Device:C
- added C19: 10u, Capacitor_Tantalum_SMD:CP_EIA-3216-18_Kemet-A_Pad1.58x1.35mm_HandSolder, symbol Device:CP
Connections:
- net +3V3: now also C19.1
- net GND: now also C19.2
Changed lines of the file:
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@@
   (junction (at 536.575 203.2) (diameter 1.016) (color 0 0 0 0)
   )
+  (junction (at 539.75 31.115) (diameter 0) (color 0 0 0 0)
+  )
   (junction (at 399.415 84.455) (diameter 1.016) (color 0 0 0 0)
   )
@@
   (junction (at 512.445 144.78) (diameter 1.016) (color 0 0 0 0)
   )
-  (junction (at 539.75 31.115) (diameter 1.016) (color 0 0 0 0)
-  )
   (junction (at 392.43 76.835) (diameter 1.016) (color 0 0 0 0)
   )
@@
     (pin "1")
   )
-  (symbol (lib_id "Device:C") (at 539.75 34.925 180) (unit 1)
-    (in_bom yes) (on_board yes)
-    (property "Reference" "C19" (id 0) (at 542.8742 32.385 0)
-      (effects (font (size 1 1)))
-    )
-    (property "Value" "10u" (id 1) (at 543.2806 37.465 0)
-      (effects (font (size 1 1)))
-    )
-    (property "Footprint" "Capacitor_SMD:C_0805_2012Metric_Pad1.18x1.45mm_HandSolder" (id 2) (at 538.7848 31.115 0)
-      (effects (font (size 1.27 1.27)) hide)
-    )
-    (property "Datasheet" "~" (id 3) (at 539.75 34.925 0)
-      (effects (font (size 1.27 1.27)) hide)
-    )
-    (pin "1")
-    (pin "2")
-  )
   (symbol (lib_id "power:GND") (at 276.86 28.575 90) (mirror x) (unit 1)
     (in_bom yes) (on_board yes)
@@
     (pin "1")
   )
+  (symbol (lib_id "Device:CP") (at 539.75 34.925 0) (unit 1)
+    (in_bom yes) (on_board yes)
+    (property "Reference" "C19" (id 0) (at 541.655 33.02 0)
+      (effects (font (size 0.9906 0.9906)))
+    )
+    (property "Value" "10u" (id 1) (at 541.655 36.83 0)
+      (effects (font (size 0.9906 0.9906)))
+    )
+    (property "Footprint" "Capacitor_Tantalum_SMD:CP_EIA-3216-18_Kemet-A_Pad1.58x1.35mm_HandSolder" (id 2) (at 540.7152 38.735 0)
+      (effects (font (size 1.27 1.27)) hide)
+    )
+    (property "Datasheet" "~" (id 3) (at 539.75 34.925 0)
+      (effects (font (size 1.27 1.27)) hide)
+    )
+    (pin "1")
+    (pin "2")
+  )
   (symbol (lib_id "power:+5V") (at 276.86 33.655 270) (mirror x) (unit 1)
     (in_bom yes) (on_board yes)
@@
       (reference "C18") (unit 1) (value "10u") (footprint "Capacitor_SMD:C_0805_2012Metric_Pad1.18x1.45mm_HandSolder")
     )
-    (path "/5e0b7f0e-7035-4d80-8114-eb1ed1aef2b9"
-      (reference "C19") (unit 1) (value "10u") (footprint "Capacitor_SMD:C_0805_2012Metric_Pad1.18x1.45mm_HandSolder")
+    (path "/a8538d46-c82e-4842-aed3-ce20334e1494"
+      (reference "C19") (unit 1) (value "10u") (footprint "Capacitor_Tantalum_SMD:CP_EIA-3216-18_Kemet-A_Pad1.58x1.35mm_HandSolder")
     )
     (path "/33708f24-5925-4541-a2e8-8fb92e3c2e55"

Commit message: wip pcb rev.A
Parts:
- C6: renamed from C8; value 100u -> 220u
- U1: renamed from U9; value AMS1117-3.3 -> 1117-3.3
- U14: renamed from U7; value 27C512 -> 39SF010; symbol Memory_EPROM:27C512PLCC -> my:29C040
- renumbered C18 to C1, C20 to C10, C21 to C11, C22 to C12, C23 to C13, C24 to C14, C25 to C15, C26 to C16, C27 to C17, C28 to C18, C29 to C19, C19 to C2, C30 to C20, C31 to C21, C32 to C22, C33 to C23, C34 to C24, C35 to C25, C36 to C26, C37 to C27, C38 to C28, C39 to C29, C47 to C3, C44 to C30, C48 to C31, C49 to C32, C51 to C33, C4 to C34, C56 to C35, C57 to C36, C69 to C37, C70 to C38, C71 to C39, C13 to C4, C72 to C40, C73 to C41, C40 to C42, C41 to C43, C42 to C44, C43 to C45, C45 to C46, C46 to C47, C58 to C48, C59 to C49, C14 to C5, C60 to C50, C61 to C51, C62 to C52, C63 to C53, C64 to C54, C65 to C55, C66 to C56, C67 to C57, C68 to C58, C52 to C59, C53 to C60, C54 to C61, C55 to C62, C9 to C63, C10 to C64, C11 to C65, C12 to C66, C1 to C67, C6 to C68, C7 to C69, C17 to C7, C3 to C70, C2 to C71, C5 to C72, C15 to C8, C16 to C9, D3 to D1, D5 to D2, D7 to D3, D8 to D4, D4 to D5, D9 to D6, D6 to D7, D1 to D8, D2 to D9, H4 to H3, H3 to H4, J3 to J1, J6 to J11, J11 to J12, J7 to J2, J8 to J3, J2 to J4, J12 to J5, J5 to J6, J4 to J7, J9 to J8, J1 to J9, Q2 to Q1, Q1 to Q2, R14 to R1, R6 to R10, R17 to R11, R19 to R12, R20 to R13, R2 to R14, R1 to R15, R4 to R16, R18 to R17, R12 to R18, R13 to R19, R8 to R2, R3 to R20, R11 to R21, R22 to R3, R21 to R4, R15 to R5, R16 to R6, R10 to R7, R5 to R8, R7 to R9, RN8 to RN7, SW2 to SW1, SW1 to SW2, U13 to U10, U8 to U11, U3 to U12, U4 to U13, U11 to U15, U2 to U16, U10 to U2, U12 to U3, U5 to U4, U14 to U5, U16 to U6, U15 to U7, U6 to U8, U1 to U9, X3 to X2, X2 to X3, Y2 to Y1, Y1 to Y2
Connections:
- net +5V: now also U14.1 (A18), U14.30 (A17)
- net GND: now also R5.1; no longer R5.2
- net KBSJ: now also U14.22 (~{CE}); no longer U14.23 (~{CE})
- net MEMR: now also U14.24 (~{OE}); no longer U14.25 (~{OE}/VPP)
- net SA0: now also U14.12 (A0); no longer U14.11 (A0)
- net SA1: now also U14.11 (A1); no longer U14.10 (A1)
- net SA10: now also U14.23 (A10); no longer U14.24 (A10)
- net SA11: now also U14.25 (A11); no longer U14.27 (A11)
- net SA12: now also U14.4 (A12); no longer U14.3 (A12)
- net SA13: now also U14.28 (A13); no longer U14.30 (A13)
- net SA14: now also U14.29 (A14); no longer U14.31 (A14)
- net SA15: now also U14.3 (A15); no longer U14.2 (A15)
- net SA16: now also U14.2 (A16)
- net SA2: now also U14.10 (A2); no longer U14.9 (A2)
- net SA3: now also U14.9 (A3); no longer U14.8 (A3)
- net SA4: now also U14.8 (A4); no longer U14.7 (A4)
- net SA5: now also U14.7 (A5); no longer U14.6 (A5)
- net SA6: now also U14.6 (A6); no longer U14.5 (A6)
- net SA7: now also U14.5 (A7); no longer U14.4 (A7)
- net SA8: now also U14.27 (A8); no longer U14.29 (A8)
- net SA9: now also U14.26 (A9); no longer U14.28 (A9)
- net SMEMW: now also U14.31 (~{WE})
- net XD3: now also U14.17 (D3); no longer U14.18 (O3)
- net XD4: now also U14.18 (D4); no longer U14.19 (O4)
- net XD5: now also U14.19 (D5); no longer U14.20 (O5)
- net XD6: now also U14.20 (D6); no longer U14.21 (O6)
- net XD7: now also U14.21 (D7); no longer U14.22 (O7)
- net at C3.2, R1.2, U2.3 (FB): now also R5.2; no longer R5.1
- net ESP_BOOT: now reaches J12.1 (Pin_1), U16.18 (GPIO0)
Other:
- note added: "Pull ESP_BOOT to GND to enter programming mode."
- moved on the sheet: C10, C11, C12, C13, C14, C15, C16, C17, C18, C19, C20, C21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
