File: pcb_main/rev.A/kharon386_main.kicad_sch (KiCad schematic)
At the start: 157 parts, among them CON1 CF-CARD-cfcard, J1 USB_B_Micro, J10 COM2, J11 Conn_01x04, J12 ESP, J2 PC104_16, J3 PC104, J4 PJ-322, J5 Conn_02x07_Odd_Even, J6 DB15_Female_HighDensity_Mount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, J7 Mini-DIN-6, J8 COM1, J9 Mini-DIN-6, Q1 BC856, Q2 BC817, SW1 Jumper / Pin header 1x2 Pitch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, SW2 SW_Push, U1 1117-3.3, U10 ST16C554, U11 GD75232PW, U12 MSM5118160F-JS, U13 MSM5118160F-JS, U14 39SF010, U15 TXB0104PW, U16 ESP-12E, U2 LT1930, U3 MAX823LEUK, U4 M6117D, U5 74HCT32, U6 74HCT138, U7 74HCT138, U8 GD75232PW, U9 CH340G, X1 14.318 MHz, X2 80 MHz, X3 1.8432 Mhz, Y1 32768 Hz, Y2 12 MHz

Commit message: wip pcb rev.A
Parts:
- removed U3: MAX823LEUK, Package_TO_SOT_SMD:SOT-23-5, symbol my:MAX823
- added C73, C74: 10u, Capacitor_Tantalum_SMD:CP_EIA-3528-21_Kemet-B_Pad1.50x2.35mm_HandSolder, symbol Device:C_Polarized
- added R23: 10k, Resistor_SMD:R_0603_1608Metric_Pad0.98x0.95mm_HandSolder, symbol Device:R
- added U17: ICL7660A, Package_SO:SOIC-8_3.9x4.9mm_P1.27mm, symbol Regulator_SwitchedCapacitor:ICL7660
- added U3: MAX809LEUR, Package_TO_SOT_SMD:SOT-23, symbol my:MAX809
- C2: symbol Device:CP -> Device:C_Polarized
- R1: value 113k -> 117k
- R7: value 10k -> 1k
- U2: value LT1930 -> LMR62014
Connections:
- net +12V: now also U17.8 (V+)
- net +5V: no longer C35.1
- net -12V: now also C74.2, U17.5 (VOUT)
- net GND: now also C74.1, R23.2, U17.3 (GND), U3.1 (GND)
- net PWG: now also R23.1, U3.2 (~{RST})
- net at R7.2, SW2.1: now also C35.1, U3.3 (VCC)
- new net: C73.1, U17.2 (CAP+)
- new net: C73.2, U17.4 (CAP-)
- no-connect marks 85 -> 86
Other:
- note added: "100 Ohm"
- note added: "Alternative -12V DC converter If used - do not install D5, D6, C8, C9"
- moved on the sheet: C35, C36, C37, C38, C39, C40, C41, C63, C64, C65, C66, C72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

Commit message: wip pcb rev.A
Parts:
- J5: value Conn_02x07_Odd_Even -> Conn_02x08_Odd_Even
Other:
- moved on the sheet: J2, J3, R6

Commit message: wip pcb rev.A
Parts:
- added R22: 5.6k, Resistor_SMD:R_0603_1608Metric_Pad0.98x0.95mm_HandSolder, symbol Device:R
- U10: value ST16C554 -> ST16C554D
- U5: value 74HCT32 -> 74HCT32PW
- U6, U7: value 74HCT138 -> 74HCT138PW
- X1, X2, X3: footprint Oscillator:Oscillator_SMD_SeikoEpson_SG8002CA-4Pin_7.0x5.0mm -> my:Oscillator_SMD_7050_7.0x5.0mm
Connections:
- net GND: now also R22.2
- net at CON1.43 (~{INPACK}): now also R22.1
- net GPCS0: no longer names the net of U4.51 (GPCS0J)
Other:
- moved on the sheet: BT1, C1, C10, C11, C12, C13, C14, C15, C16, C17, C18, C19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

Commit message: pcb rev.A final version
Parts:
- added U18, U19: IP4220CZ6, Package_SO:TSOP-6_1.65x3.05mm_P0.95mm, symbol my:IP4220CZ6
- C2: value 10u -> 47u; footprint Capacitor_Tantalum_SMD:CP_EIA-3216-18_Kemet-A_Pad1.58x1.35mm_HandSolder -> Capacitor_Tantalum_SMD:CP_EIA-3528-21_Kemet-B_Pad1.50x2.35mm_HandSolder
- C3: value 10p -> 220p
- J4: value PJ-322 -> PJ-320; footprint my:PJ-322 -> my:PJ-320A_D
- SW2: Desc (none) -> Reset
Connections:
- net +5V: now also U18.5 (+), U19.5 (+)
- net GND: now also U18.2 (-), U19.2 (-)
- net KBCLK: now also U18.1
- net KBDAT: now also U18.4
- net MSCLK: now also U19.1
- net MSDAT: now also U19.4
- no-connect marks 86 -> 90
Other:
- note added: "PS/2"
- note added: "VGA & Sound"
- moved on the sheet: C3, C63, C64, C65, C66, C67, C70, C71, C72, CON1, D7, D8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
