File: pcb_covers/rev.A/charon386_covers.kicad_pcb (KiCad board)
At the start: 2 copper layers, 134.6 x 64 mm, 1 part

Commit message: wip pcb rev.A (almost done now)
Parts:
- removed G***: LOGO, mygraphic:zxuno_30x7.5
Other:
- board size 134.6 x 64 mm -> 134.6 x 63 mm
- board text added: "5.1V 2.5A"
- board text added: "CF Card"
- board text added: "COM1"
- board text added: "COM2"
- board text added: "Charon-386"
- board text added: "Charon-386 Back cover Rev.A"
- board text added: "Charon-386 Front cover Rev.A"
- board text added: "Line In"
- board text added: "Line Out"
- board text added: "WiFi"
- board text removed: "1010"
- board text removed: "5V 1A"
- board text removed: "Gamepad 1"
- board text removed: "Gamepad 2"
- board text removed: "NMI"
- board text removed: "SD Card"
- board text removed: "Service"
- board text removed: "Sound"
- board text removed: "Tape"
- board text removed: "WiFI"
- board text removed: "ZXUNO.1010 Back cover Rev.A"
- board text removed: "ZXUNO.1010 Front cover Rev.A"
