File: pcb_main/rev.A1/kharon386_main.kicad_sch (KiCad schematic)
At the start: 169 parts, among them CON1 CF-CARD-cfcard, J1 USB_B_Micro, J10 COM2, J11 Conn_01x04, J12 ESP, J2 PC104_16, J3 PC104, J4 PJ-320, J5 Conn_02x08_Odd_Even, J6 DB15_Female_HighDensity_Mount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, J7 Mini-DIN-6, J8 COM1, J9 Mini-DIN-6, Q1 BC856, Q2 BC817, Q3 BC856, SW1 Jumper / Pin header 1x2 Pitch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, SW2 SW_Push, SW3 SW_DIP_x01, U1 1117-3.3, U10 ST16C554D, U11 GD75232PW, U12 MSM5118160F-JS, U13 MSM5118160F-JS, U14 39SF040, U15 TXS0104PW, U16 ESP-12F, U17 ICL7660A, U18 IP4220CZ6, U19 IP4220CZ6, U2 LMR62014, U3 MAX809LEUR, U4 M6117D, U5 74HCT32PW, U6 74HCT138PW, U7 74HCT138PW, U8 GD75232PW, U9 CH340G, X1 14.318 MHz, X2 80 MHz, X3 1.8432 Mhz, Y1 32768 Hz, Y2 12 MHz

Commit message: update pcb files for kicad 7.0 and grid 1.27
Parts:
- J4: symbol Connector:AudioJack4 -> Connector_Audio:AudioJack4
Other:
- moved on the sheet: BT1, C1, C10, C11, C12, C13, C14, C15, C16, C17, C18, C19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

Commit message: wip pcb rev.A1
Parts:
- added R27: 10k, Resistor_SMD:R_0603_1608Metric_Pad0.98x0.95mm_HandSolder, symbol Device:R
Connections:
- net +3V3: now also R27.2; no longer U16.17 (GPIO2)
- new net: R27.1, U16.17 (GPIO2)
Other:
- moved on the sheet: C67, C70, C71, C72, J10, J11, J8, LS1, Q2, R20, R21, U10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

Commit message: update all pcb rev.A1 files - minor changes
Parts:
- N1: footprint (none) -> my:G738
Other:
- note added: "RAM 4Mb"
- note added: "Reset"
- note removed: "RAM 2Mb"
- moved on the sheet: C35, C42, C43, C44, C45, C46, C47, C59, C60, C61, C62, C72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
