File: pcb_top/rev.A1/kharon386_top.kicad_sch (KiCad schematic)
At the start: 150 parts, among them J1 PJ-320, J2 Vol. Btns, J3 Conn_02x07_Odd_Even, J4 ESP, J5 PC104_16, J6 PC104, SW1 VGA Config, U1 1117-5.0, U10 93C66A, U11 MT4C4256, U12 MT4C4256, U13 MT4C4256, U14 MT4C4256, U2 NE5532DR, U3 74HCT138PW, U4 ES1868F, U5 TVGA9000I, U6 SAM2695, U7 27C512, U8 1117-5.0, U9 1117-3.3, Y1 40 MHz, Y2 12 MHz

Commit message: update pcb files for kicad 7.0 and grid 1.27
Parts:
- J1: symbol Connector:AudioJack4 -> Connector_Audio:AudioJack4
Other:
- moved on the sheet: C1, C10, C11, C12, C13, C14, C15, C16, C17, C18, C19, C2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

Commit message: wip pcb rev.A1
Parts:
- added C54: 100n, Capacitor_SMD:C_0603_1608Metric_Pad1.08x0.95mm_HandSolder, symbol Device:C
- added R10, R12: 47k, Resistor_SMD:R_0603_1608Metric_Pad0.98x0.95mm_HandSolder, symbol Device:R
- U10: now not fitted; now left out of the parts list
Connections:
- net +5V: now also JP2.3 (B), C54.1; no longer JP2.1 (A)
- net AOUT_L: now also R12.2
- net AOUT_R: now also R10.2
- net GND: now also JP2.1 (A), C54.2, R10.1, R12.1; no longer JP2.3 (B)
Other:
- note added: "10-20ma"
- note added: "Install R40 or R41 R41 recommended"
- note added: "Install U1 or R38 R38 recommended"
- note added: "Install U8 or L10 U8 recommended"
- note added: "JP 1-2: Internal ROM used JP 2-3: EEPROM used for PnP"
- note removed: "Install R40 or R41"
- note removed: "Install U1 or R38"
- note removed: "Install U8 or L10"
- note removed: "JP 1-2: EEPROM used for PnP JP 2-3: Internal ROM used"
- moved on the sheet: C46, C47, C48, C50, C51, C52, C58, C59, C60, C61, C62, C63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

Commit message: update all pcb rev.A1 files - minor changes
Parts:
- R37: Desc Do not install -> (none); now not fitted
Other:
- moved on the sheet: C56, C57, L9, R40, R41
